File: tolt/tolt.kicad_pcb (KiCad board)
At the start: 2 copper layers, 0 parts

Commit message: revert the mess
i am stupid
Parts:
- added Q1: NMOS, Library:HDSOP-16-2, B.Cu at (58.2, 74.8)
- added Q10: NMOS, Library:HDSOP-16-2, B.Cu at (93.7, 99.2)
- added Q11: NMOS, Library:HDSOP-16-2, B.Cu at (105.3, 99.2)
- added Q12: NMOS, Library:HDSOP-16-2, B.Cu at (117.0, 99.2)
- added Q13: NMOS, Library:HDSOP-16-2, B.Cu at (140.9, 74.8)
- added Q14: NMOS, Library:HDSOP-16-2, B.Cu at (152.5, 74.8)
- added Q15: NMOS, Library:HDSOP-16-2, B.Cu at (129.2, 74.8)
- added Q16: NMOS, Library:HDSOP-16-2, B.Cu at (129.2, 99.2)
- added Q17: NMOS, Library:HDSOP-16-2, B.Cu at (140.9, 99.2)
- added Q18: NMOS, Library:HDSOP-16-2, B.Cu at (152.5, 99.2)
- added Q2: NMOS, Library:HDSOP-16-2, B.Cu at (69.8, 74.8)
- added Q3: NMOS, Library:HDSOP-16-2, B.Cu at (81.5, 74.8)
- added Q4: NMOS, Library:HDSOP-16-2, B.Cu at (58.2, 99.2)
- added Q5: NMOS, Library:HDSOP-16-2, B.Cu at (69.8, 99.2)
- added Q6: NMOS, Library:HDSOP-16-2, B.Cu at (81.5, 99.2)
- added Q7: NMOS, Library:HDSOP-16-2, B.Cu at (117.0, 74.8)
- added Q8: NMOS, Library:HDSOP-16-2, B.Cu at (93.7, 74.8)
- added Q9: NMOS, Library:HDSOP-16-2, B.Cu at (105.3, 74.8)
- added R11: 0.3mr, Library:R5930, B.Cu at (58.8, 116.2)
- added R12: 0.3mr, Library:R5930, B.Cu at (70.4, 116.2)
- added R13: 0.3mr, Library:R5930, B.Cu at (82.1, 116.2)
- added R20: 0.3mr, Library:R5930, B.Cu at (94.3, 116.2)
- added R21: 0.3mr, Library:R5930, B.Cu at (105.9, 116.2)
- added R22: 0.3mr, Library:R5930, B.Cu at (117.6, 116.2)
- added R30: 0.3mr, Library:R5930, B.Cu at (129.9, 116.2)
- added R31: 0.3mr, Library:R5930, B.Cu at (141.5, 116.2)
- added R32: 0.3mr, Library:R5930, B.Cu at (153.1, 116.2)
- added U2: L6491, Package_SO:SO-14_3.9x8.65mm_P1.27mm, F.Cu at (69.8, 113.1)
- added U3: L6491, Package_SO:SO-14_3.9x8.65mm_P1.27mm, F.Cu at (105.3, 113.1)
- added U4: L6491, Package_SO:SO-14_3.9x8.65mm_P1.27mm, F.Cu at (140.9, 113.1)
Other:
- copper layers 2 -> 4
