File: tolt/tolt.kicad_pcb (KiCad board)
At the start: 4 copper layers, 30 parts, among them Q1 NMOS, Q10 NMOS, Q11 NMOS, Q12 NMOS, Q13 NMOS, Q14 NMOS, Q15 NMOS, Q16 NMOS, Q17 NMOS, Q18 NMOS, Q2 NMOS, Q3 NMOS, Q4 NMOS, Q5 NMOS, Q6 NMOS, Q7 NMOS, Q8 NMOS, Q9 NMOS, U2 L6491, U3 L6491, U4 L6491

Commit message: 6 layer
Other:
- copper layers 4 -> 6
Changed lines of the file:
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@@
 		(4 "In1.Cu" signal)
 		(6 "In2.Cu" signal)
+		(8 "In3.Cu" signal)
+		(10 "In4.Cu" signal)
 		(2 "B.Cu" signal)
 		(9 "F.Adhes" user "F.Adhesive")
@@
 			(layer "dielectric 2"
 				(type "core")
-				(thickness 1.24)
+				(thickness 0.535)
 				(material "FR4")
 				(epsilon_r 4.5)
@@
 				(type "prepreg")
 				(thickness 0.1)
+				(material "FR4")
+				(epsilon_r 4.5)
+				(loss_tangent 0.02)
+			)
+			(layer "In3.Cu"
+				(type "copper")
+				(thickness 0.035)
+			)
+			(layer "dielectric 4"
+				(type "core")
+				(thickness 0.535)
+				(material "FR4")
+				(epsilon_r 4.5)
+				(loss_tangent 0.02)
+			)
+			(layer "In4.Cu"
+				(type "copper")
+				(thickness 0.035)
+			)
+			(layer "dielectric 5"
+				(type "prepreg")
+				(thickness 0.1)

Commit message: footprints
Parts:
- added C1: 100n, Capacitor_SMD:C_0402_1005Metric, F.Cu at (83.5, 185.3)
- added C10: 2.2u, Capacitor_SMD:C_0603_1608Metric, F.Cu at (66.9, 183.7)
- added C11: 15p, Capacitor_SMD:C_0402_1005Metric, F.Cu at (83.5, 193.2)
- added C12: 15p, Capacitor_SMD:C_0402_1005Metric, F.Cu at (83.5, 195.2)
- added C13: 2.2u, Capacitor_SMD:C_0603_1608Metric, F.Cu at (66.9, 186.2)
- added C14: 2.2u, Capacitor_SMD:C_0603_1608Metric, F.Cu at (70.9, 171.2)
- added C15: 4.7u, Capacitor_SMD:C_0805_2012Metric, F.Cu at (78.9, 201.7)
- added C16: 220nF, Capacitor_SMD:C_0402_1005Metric, F.Cu at (78.2, 219.2)
- added C17: 4.7u, Capacitor_SMD:C_0805_2012Metric, F.Cu at (78.9, 204.7)
- added C18: 220nF, Capacitor_SMD:C_0402_1005Metric, F.Cu at (78.2, 221.2)
- added C19: 4.7u, Capacitor_SMD:C_0805_2012Metric, F.Cu at (78.9, 207.7)
- added C2: 100n, Capacitor_SMD:C_0402_1005Metric, F.Cu at (83.5, 187.3)
- added C20: 220nF, Capacitor_SMD:C_0402_1005Metric, F.Cu at (78.2, 223.1)
- added C21: 4.7u, Capacitor_SMD:C_0805_2012Metric, F.Cu at (78.9, 210.7)
- added C22: 4.7u, Capacitor_SMD:C_0805_2012Metric, F.Cu at (78.9, 213.7)
- added C23: 4.7u, Capacitor_SMD:C_0805_2012Metric, F.Cu at (78.9, 216.7)
- added C24: 100n, Capacitor_SMD:C_0402_1005Metric, F.Cu at (78.2, 225.1)
- added C25: 100n, Capacitor_SMD:C_0402_1005Metric, F.Cu at (78.2, 227.1)
- added C26: 100n, Capacitor_SMD:C_0402_1005Metric, F.Cu at (78.2, 229.0)
- added C27: 100n, Capacitor_SMD:C_0402_1005Metric, F.Cu at (83.5, 197.2)
- added C28: 100n, Capacitor_SMD:C_0402_1005Metric, F.Cu at (86.4, 185.3)
- added C29: 15n, Capacitor_SMD:C_0603_1608Metric, F.Cu at (70.9, 173.7)
- added C3: 100n, Capacitor_SMD:C_0402_1005Metric, F.Cu at (83.5, 189.3)
- added C30: 1n, Capacitor_SMD:C_0603_1608Metric, F.Cu at (70.9, 176.2)
- added C31: 100n, Capacitor_SMD:C_0402_1005Metric, F.Cu at (86.4, 187.3)
- added C32: 100n, Capacitor_SMD:C_0402_1005Metric, F.Cu at (86.4, 189.3)
- added C33: 100n, Capacitor_SMD:C_0402_1005Metric, F.Cu at (86.4, 191.2)
- added C34: 100n, Capacitor_SMD:C_0402_1005Metric, F.Cu at (86.4, 193.2)
- added C35: 1n, Capacitor_SMD:C_0603_1608Metric, F.Cu at (70.9, 178.7)
- added C36: 15n, Capacitor_SMD:C_0603_1608Metric, F.Cu at (70.9, 181.2)
- added C37: 100n, Capacitor_SMD:C_0402_1005Metric, F.Cu at (86.4, 195.2)
- added C38: 100n, Capacitor_SMD:C_0402_1005Metric, F.Cu at (86.4, 197.2)
- added C39: 100n, Capacitor_SMD:C_0402_1005Metric, F.Cu at (89.3, 185.3)
- added C4: 100n, Capacitor_SMD:C_0402_1005Metric, F.Cu at (83.5, 191.2)
- added C40: 1n, Capacitor_SMD:C_0603_1608Metric, F.Cu at (70.9, 183.7)
- added C41: 15n, Capacitor_SMD:C_0603_1608Metric, F.Cu at (70.9, 186.2)
- added C42: 10u, Capacitor_SMD:C_0603_1608Metric, F.Cu at (62.7, 201.4)
- added C43: 10u, Capacitor_SMD:C_0603_1608Metric, F.Cu at (62.7, 203.9)
- added C44: 10u, Capacitor_SMD:C_0603_1608Metric, F.Cu at (62.7, 206.4)
- added C45: 100n, Capacitor_SMD:C_0402_1005Metric, F.Cu at (89.3, 187.3)
- added C46: 100n, Capacitor_SMD:C_0402_1005Metric, F.Cu at (89.3, 189.3)
- added C47: 100n, Capacitor_SMD:C_0402_1005Metric, F.Cu at (89.3, 191.2)
- added C48: 100n, Capacitor_SMD:C_0402_1005Metric, F.Cu at (89.3, 193.2)
- added C49: 100n, Capacitor_SMD:C_0402_1005Metric, F.Cu at (89.3, 195.2)
- added C5: 2.2u, Capacitor_SMD:C_0603_1608Metric, F.Cu at (66.9, 171.2)
- added C50: 100n, Capacitor_SMD:C_0402_1005Metric, F.Cu at (89.3, 197.2)
- added C51: 4.7u, Capacitor_SMD:C_0603_1608Metric, F.Cu at (62.7, 208.9)
- added C52: 4.7u, Capacitor_SMD:C_0603_1608Metric, F.Cu at (62.7, 211.4)
- added C53: 4.7u, Capacitor_SMD:C_0603_1608Metric, F.Cu at (62.7, 213.9)
- added C54: 100n, Capacitor_SMD:C_0603_1608Metric, F.Cu at (62.7, 216.5)
- added C55: 100n, Capacitor_SMD:C_0603_1608Metric, F.Cu at (62.7, 219.0)
- added C56: 100n, Capacitor_SMD:C_0603_1608Metric, F.Cu at (62.7, 221.5)
- added C57: 100n, Capacitor_SMD:C_0603_1608Metric, F.Cu at (66.7, 201.4)
- added C58: 2.2uf, Capacitor_SMD:C_0603_1608Metric, F.Cu at (93.3, 227.3)
- added C59: 2.2uf, Capacitor_SMD:C_0603_1608Metric, F.Cu at (93.3, 229.8)
- added C6: 2.2u, Capacitor_SMD:C_0603_1608Metric, F.Cu at (66.9, 173.7)
- added C60: 2.2uf, Capacitor_SMD:C_0603_1608Metric, F.Cu at (93.3, 232.4)
- added C61: 33uF, Capacitor_THT:CP_Radial_D5.0mm_P2.00mm, F.Cu at (113.0, 187.1)
- added C62: 100nF, Capacitor_SMD:C_0603_1608Metric, F.Cu at (95.4, 171.2)
- added C63: 2.2uF, Capacitor_SMD:C_0603_1608Metric, F.Cu at (95.4, 173.7)
- added C64: 100nF, Capacitor_SMD:C_0603_1608Metric, F.Cu at (95.4, 176.2)
- added C65: 2.2uF, Capacitor_SMD:C_0603_1608Metric, F.Cu at (95.4, 178.7)
- added C66: 100uF, Capacitor_SMD:C_0603_1608Metric, F.Cu at (95.4, 181.2)
- added C67: 100nF, Capacitor_SMD:C_0603_1608Metric, F.Cu at (95.4, 183.7)
- added C68: 2.2uF, Capacitor_SMD:C_0603_1608Metric, F.Cu at (99.4, 171.2)
- added C69: 100nF, Capacitor_SMD:C_0603_1608Metric, F.Cu at (99.4, 173.7)
- added C7: 2.2u, Capacitor_SMD:C_0603_1608Metric, F.Cu at (66.9, 176.2)
- added C70: 2.2uF, Capacitor_SMD:C_0603_1608Metric, F.Cu at (99.4, 176.2)
- added C71: 10uF, Capacitor_SMD:C_0603_1608Metric, F.Cu at (99.4, 178.7)
- added C72: 22uF, Capacitor_SMD:C_0805_2012Metric, F.Cu at (102.2, 186.5)
- added C73: 10uF, Capacitor_SMD:C_0805_2012Metric, F.Cu at (102.2, 189.5)
- added C74: 100nF, Capacitor_SMD:C_0603_1608Metric, F.Cu at (99.4, 181.2)
- added C75: 2.2uF, Capacitor_SMD:C_0603_1608Metric, F.Cu at (99.4, 183.7)
- added C76: 100nF, Capacitor_SMD:C_0603_1608Metric, F.Cu at (103.4, 171.2)
- added C77: 2.2uF, Capacitor_SMD:C_0603_1608Metric, F.Cu at (103.4, 173.7)
- added C78: 2.2u, Capacitor_SMD:C_0603_1608Metric, F.Cu at (115.7, 227.3)
- added C79: 100n, Capacitor_SMD:C_0402_1005Metric, F.Cu at (115.1, 234.6)
- added C8: 2.2u, Capacitor_SMD:C_0603_1608Metric, F.Cu at (66.9, 178.7)
- added C80: 100n, Capacitor_SMD:C_0402_1005Metric, F.Cu at (92.7, 221.1)
- added C81: 4.7u, Capacitor_SMD:C_0805_2012Metric, F.Cu at (115.0, 217.9)
- added C82: 100n, Capacitor_SMD:C_0402_1005Metric, F.Cu at (92.7, 223.1)
- added C83: 4.7u, Capacitor_SMD:C_0805_2012Metric, F.Cu at (119.9, 227.6)
- added C84: 4.7u, Capacitor_SMD:C_0805_2012Metric, F.Cu at (119.9, 230.6)
- added C9: 2.2u, Capacitor_SMD:C_0603_1608Metric, F.Cu at (66.9, 181.2)
- added C91: 4.7u, Capacitor_SMD:C_0805_2012Metric, F.Cu at (115.0, 220.9)
- added D1: STTH2R06A, Diode_SMD:D_SMA, F.Cu at (85.2, 202.4)
- added D2: STTH2R06A, Diode_SMD:D_SMA, F.Cu at (85.2, 207.0)
- added D22: green, LED_SMD:LED_0603_1608Metric, F.Cu at (62.7, 233.3)
- added D23: LED, LED_SMD:LED_0603_1608Metric, F.Cu at (102.0, 192.3)
- added D26: red, LED_SMD:LED_0603_1608Metric, F.Cu at (62.7, 235.9)
- added D27: blue, LED_SMD:LED_0603_1608Metric, F.Cu at (62.7, 238.5)
- added D3: STTH2R06A, Diode_SMD:D_SMA, F.Cu at (85.2, 211.5)
- added J14: BOOT0, Jumper:SolderJumper-2_P1.3mm_Open_RoundedPad1.0x1.5mm, F.Cu at (67.1, 189.2)
- added J15: NRST, Jumper:SolderJumper-2_P1.3mm_Open_RoundedPad1.0x1.5mm, F.Cu at (67.1, 192.8)
- added J2: USB_C_Receptacle_USB2.0, Connector_USB:USB_C_Receptacle_G-Switch_GT-USB-7051x, F.Cu at (96.8, 216.4)
- added JP1: Jumper_3_Bridged12, Connector_PinHeader_2.54mm:PinHeader_1x03_P2.54mm_Vertical, F.Cu at (105.6, 202.4)
- added JP2: Jumper_2_Open, Jumper:SolderJumper-2_P1.3mm_Open_RoundedPad1.0x1.5mm, F.Cu at (110.6, 218.2)
- added JP3: Jumper_2_Open, Jumper:SolderJumper-2_P1.3mm_Open_RoundedPad1.0x1.5mm, F.Cu at (110.6, 221.8)
- added L3: 10uH, Inductor_SMD:L_Ferrocore_DLG-0403, F.Cu at (96.7, 188.0)
- added R1: 0, Resistor_SMD:R_0603_1608Metric, F.Cu at (66.7, 203.9)
- added R10: R, Resistor_SMD:R_0603_1608Metric, F.Cu at (97.3, 232.4)
- added R14: R, Resistor_SMD:R_0603_1608Metric, F.Cu at (97.3, 234.9)
- added R15: R, Resistor_SMD:R_0603_1608Metric, F.Cu at (97.3, 237.4)
- added R16: R, Resistor_SMD:R_0603_1608Metric, F.Cu at (97.3, 239.9)
- added R17: R, Resistor_SMD:R_0603_1608Metric, F.Cu at (101.3, 227.3)
- added R18: R, Resistor_SMD:R_0603_1608Metric, F.Cu at (101.3, 229.8)
- added R19: R, Resistor_SMD:R_0603_1608Metric, F.Cu at (101.3, 232.4)
- added R2: 0, Resistor_SMD:R_0603_1608Metric, F.Cu at (66.7, 206.4)
- added R23: R, Resistor_SMD:R_0603_1608Metric, F.Cu at (101.3, 234.9)
- added R24: R, Resistor_SMD:R_0603_1608Metric, F.Cu at (101.3, 237.4)
- added R25: R, Resistor_SMD:R_0603_1608Metric, F.Cu at (101.3, 239.9)
- added R26: 5k1, Resistor_SMD:R_0603_1608Metric, F.Cu at (93.3, 201.4)
- added R27: R, Resistor_SMD:R_0603_1608Metric, F.Cu at (105.3, 227.3)
- added R28: R, Resistor_SMD:R_0603_1608Metric, F.Cu at (105.3, 229.8)
- added R29: R, Resistor_SMD:R_0603_1608Metric, F.Cu at (105.3, 232.4)
- added R3: 0, Resistor_SMD:R_0603_1608Metric, F.Cu at (66.7, 208.9)
- added R33: 1k, Resistor_SMD:R_0603_1608Metric, F.Cu at (75.0, 171.2)
- added R34: 1k, Resistor_SMD:R_0603_1608Metric, F.Cu at (75.0, 173.7)
- added R35: 1k, Resistor_SMD:R_0603_1608Metric, F.Cu at (75.0, 176.2)
- added R36: 320k, Resistor_SMD:R_0603_1608Metric, F.Cu at (66.7, 211.4)
- added R37: 10k, Resistor_SMD:R_0603_1608Metric, F.Cu at (66.7, 213.9)
- added R38: 10k, Resistor_SMD:R_0603_1608Metric, F.Cu at (75.0, 178.7)
- added R39: 10k, Resistor_SMD:R_0603_1608Metric, F.Cu at (75.0, 181.2)
- added R4: 0, Resistor_SMD:R_0815_2038Metric, F.Cu at (107.7, 172.7)
- added R40: 10k, Resistor_SMD:R_0603_1608Metric, F.Cu at (66.7, 216.5)
- added R41: 10k, Resistor_SMD:R_0603_1608Metric, F.Cu at (66.7, 219.0)
- added R42: 10k, Resistor_SMD:R_0603_1608Metric, F.Cu at (66.7, 221.5)
- added R43: 240k, Resistor_SMD:R_0603_1608Metric, F.Cu at (70.7, 201.4)
- added R44: 5.1k, Resistor_SMD:R_0603_1608Metric, F.Cu at (70.7, 203.9)
- added R45: 240k, Resistor_SMD:R_0603_1608Metric, F.Cu at (70.7, 206.4)
- added R46: 5.1k, Resistor_SMD:R_0603_1608Metric, F.Cu at (70.7, 208.9)
- added R47: 240k, Resistor_SMD:R_0603_1608Metric, F.Cu at (70.7, 211.4)
- added R48: 5.1k, Resistor_SMD:R_0603_1608Metric, F.Cu at (70.7, 213.9)
- added R49: 480k, Resistor_SMD:R_2512_6332Metric, F.Cu at (83.9, 220.7)
- added R5: R, Resistor_SMD:R_0603_1608Metric, F.Cu at (93.3, 234.9)
- added R50: 10.2k, Resistor_SMD:R_0603_1608Metric, F.Cu at (70.7, 216.5)
- added R51: 320k, Resistor_SMD:R_0603_1608Metric, F.Cu at (70.7, 219.0)
- added R52: 10k, Resistor_SMD:R_0603_1608Metric, F.Cu at (70.7, 221.5)
- added R53: 320k, Resistor_SMD:R_0603_1608Metric, F.Cu at (74.7, 201.4)
- added R54: 10k, Resistor_SMD:R_0603_1608Metric, F.Cu at (74.7, 203.9)
- added R55: 10k, Resistor_SMD:R_0603_1608Metric, F.Cu at (74.7, 206.4)
- added R56: 10k, Resistor_SMD:R_0603_1608Metric, F.Cu at (74.7, 208.9)
- added R57: 10k, Resistor_SMD:R_0603_1608Metric, F.Cu at (74.7, 211.4)
- added R58: 10k_NTC, Resistor_SMD:R_0603_1608Metric_Pad0.98x0.95mm_HandSolder, F.Cu at (109.5, 227.3)
- added R59: 10k_NTC, Resistor_SMD:R_0603_1608Metric_Pad0.98x0.95mm_HandSolder, F.Cu at (109.5, 229.8)
- added R6: R, Resistor_SMD:R_0603_1608Metric, F.Cu at (93.3, 237.4)
- added R60: 10k_NTC, Resistor_SMD:R_0603_1608Metric_Pad0.98x0.95mm_HandSolder, F.Cu at (109.5, 232.4)
- added R61: 10k, Resistor_SMD:R_0603_1608Metric, F.Cu at (105.3, 234.9)
- added R62: 10k, Resistor_SMD:R_0603_1608Metric, F.Cu at (105.3, 237.4)
- added R63: 10k, Resistor_SMD:R_0603_1608Metric, F.Cu at (105.3, 239.9)
- added R64: 100k, Resistor_SMD:R_0603_1608Metric, F.Cu at (103.4, 176.2)
- added R65: 220r, Resistor_SMD:R_0603_1608Metric, F.Cu at (66.7, 233.3)
- added R66: 220r, Resistor_SMD:R_0603_1608Metric, F.Cu at (66.7, 235.8)
- added R67: 1k, Resistor_SMD:R_0603_1608Metric, F.Cu at (66.7, 238.3)
- added R68: 0, Resistor_SMD:R_0815_2038Metric, F.Cu at (112.1, 172.7)
- added R69: 0, Resistor_SMD:R_0815_2038Metric, F.Cu at (116.6, 172.7)
- added R7: R, Resistor_SMD:R_0603_1608Metric, F.Cu at (93.3, 239.9)
- added R70: 1k, Resistor_SMD:R_0603_1608Metric, F.Cu at (115.7, 229.8)
- added R71: 1k, Resistor_SMD:R_0603_1608Metric, F.Cu at (115.7, 232.4)
- added R72: 10k, Resistor_SMD:R_0603_1608Metric, F.Cu at (93.3, 203.9)
- added R73: 2k2, Resistor_SMD:R_0603_1608Metric, F.Cu at (93.3, 206.4)
- added R74: 2k2, Resistor_SMD:R_0603_1608Metric, F.Cu at (93.3, 208.9)
- added R75: 2k2, Resistor_SMD:R_0603_1608Metric, F.Cu at (93.3, 211.4)
- added R76: 4.3k, Resistor_SMD:R_0603_1608Metric, F.Cu at (97.3, 201.4)
- added R77: 4.3k, Resistor_SMD:R_0603_1608Metric, F.Cu at (97.3, 203.9)
- added R78: 4.3k, Resistor_SMD:R_0603_1608Metric, F.Cu at (97.3, 206.4)
- added R79: 2k2, Resistor_SMD:R_0603_1608Metric, F.Cu at (97.3, 208.9)
- added R8: R, Resistor_SMD:R_0603_1608Metric, F.Cu at (97.3, 227.3)
- added R80: 4.3k, Resistor_SMD:R_0603_1608Metric, F.Cu at (97.3, 211.4)
- added R81: 2k2, Resistor_SMD:R_0603_1608Metric, F.Cu at (101.3, 201.4)
- added R82: 4.3k, Resistor_SMD:R_0603_1608Metric, F.Cu at (101.3, 203.9)
- added R83: 120ohm, Resistor_SMD:R_0603_1608Metric, F.Cu at (101.3, 206.4)
- added R84: 5k1, Resistor_SMD:R_0603_1608Metric, F.Cu at (101.3, 208.9)
- added R9: R, Resistor_SMD:R_0603_1608Metric, F.Cu at (97.3, 229.8)
- added U1: STM32F405RGTx, Package_QFP:LQFP-64_10x10mm_P0.5mm, F.Cu at (84.2, 177.1)
- added U10: MC74VHC1GT66, Package_TO_SOT_SMD:SOT-353_SC-70-5, F.Cu at (62.8, 179.7)
- added U11: MC74VHC1GT66, Package_TO_SOT_SMD:SOT-353_SC-70-5, F.Cu at (62.8, 183.7)
- added U12: MC74VHC1GT66, Package_TO_SOT_SMD:SOT-353_SC-70-5, F.Cu at (62.8, 187.6)
- added U13: MC74VHC1GT66, Package_TO_SOT_SMD:SOT-353_SC-70-5, F.Cu at (62.8, 191.5)
- added U14: AMS1117-3.3, Package_TO_SOT_SMD:SOT-223-3_TabPin2, F.Cu at (110.4, 179.7)
- added U15: LP5907MFX-3.3, Package_TO_SOT_SMD:SOT-23-5, F.Cu at (108.0, 186.2)
- added U16: TPS62173DSG, Package_SON:WSON-8-1EP_2x2mm_P0.5mm_EP0.9x1.6mm, F.Cu at (112.8, 192.3)
- added U17: BMI160, Package_LGA:Bosch_LGA-14_3x2.5mm_P0.5mm, F.Cu at (120.2, 234.4)
- added U19: LP5907MFX-3.3, Package_TO_SOT_SMD:SOT-23-5, F.Cu at (108.0, 190.8)
- added U20: TJA1051T-3, Package_SO:SOIC-8_3.9x4.9mm_P1.27mm, F.Cu at (112.7, 213.2)
- added U21: SRV05-4, Package_TO_SOT_SMD:SOT-23-6, F.Cu at (105.9, 212.2)
- added U22: SRV05-4, Package_TO_SOT_SMD:SOT-23-6, F.Cu at (105.9, 216.9)
- added U23: SRV05-4, Package_TO_SOT_SMD:SOT-23-6, F.Cu at (105.9, 221.5)
- added U5: INA240/241, Package_TO_SOT_SMD:SOT-23-8, F.Cu at (79.5, 186.7)
- added U6: MC74VHC1GT66, Package_TO_SOT_SMD:SOT-353_SC-70-5, F.Cu at (62.8, 171.9)
- added U7: ~, Package_TO_SOT_SMD:SOT-23-8, F.Cu at (79.5, 191.3)
- added U8: MC74VHC1GT66, Package_TO_SOT_SMD:SOT-353_SC-70-5, F.Cu at (62.8, 175.8)
- added U9: ~, Package_TO_SOT_SMD:SOT-23-8, F.Cu at (79.5, 195.9)
- added Y1: 8m, Crystal:Crystal_SMD_3225-4Pin_3.2x2.5mm, F.Cu at (71.9, 189.7)
