File: tolt/tolt.kicad_pcb (KiCad board)
At the start: 4 copper layers, 30 parts, among them Q1 NMOS, Q10 NMOS, Q11 NMOS, Q12 NMOS, Q13 NMOS, Q14 NMOS, Q15 NMOS, Q16 NMOS, Q17 NMOS, Q18 NMOS, Q2 NMOS, Q3 NMOS, Q4 NMOS, Q5 NMOS, Q6 NMOS, Q7 NMOS, Q8 NMOS, Q9 NMOS, U2 L6491, U3 L6491, U4 L6491

Commit message: new file:   tolt/Library.pretty/PQDE6W.kicad_mod 	modified:   tolt/auxl.kicad_sch 	modified:   tolt/conn.kicad_sch 	modified:   tolt/converters.kicad_sch 	modified:   tolt/powerstage.kicad_sch 	modified:   tolt/tolt.kicad_pcb 	modified:   tolt/tolt.kicad_sch
Parts:
- added C1: 100n, Capacitor_SMD:C_0402_1005Metric, F.Cu at (-188.4, 89.7)
- added C10: 2.2u, Capacitor_SMD:C_0603_1608Metric, F.Cu at (-175.2, 90.0)
- added C100: 560u, Capacitor_THT:CP_Radial_D16.0mm_P7.50mm, F.Cu at (-155.9, -47.7)
- added C101: 1uf, Capacitor_SMD:C_2220_5750Metric_Pad1.97x5.40mm_HandSolder, F.Cu at (-128.0, -63.8)
- added C102: 1uf, Capacitor_SMD:C_2220_5750Metric_Pad1.97x5.40mm_HandSolder, F.Cu at (-128.0, -56.9)
- added C103: 1uf, Capacitor_SMD:C_2220_5750Metric_Pad1.97x5.40mm_HandSolder, F.Cu at (-128.0, -49.9)
- added C104: 1uf, Capacitor_SMD:C_2220_5750Metric_Pad1.97x5.40mm_HandSolder, F.Cu at (-128.0, -43.0)
- added C105: 1uf, Capacitor_SMD:C_2220_5750Metric_Pad1.97x5.40mm_HandSolder, F.Cu at (-119.2, -63.8)
- added C106: 1uf, Capacitor_SMD:C_2220_5750Metric_Pad1.97x5.40mm_HandSolder, F.Cu at (-119.2, -56.9)
- added C107: 1uf, Capacitor_SMD:C_2220_5750Metric_Pad1.97x5.40mm_HandSolder, F.Cu at (-119.2, -49.9)
- added C108: 1uf, Capacitor_SMD:C_2220_5750Metric_Pad1.97x5.40mm_HandSolder, F.Cu at (-119.2, -43.0)
- added C109: 1uf, Capacitor_SMD:C_2220_5750Metric_Pad1.97x5.40mm_HandSolder, F.Cu at (-110.4, -63.8)
- added C11: 15p, Capacitor_SMD:C_0402_1005Metric, F.Cu at (-188.4, 97.6)
- added C110: 1uf, Capacitor_SMD:C_2220_5750Metric_Pad1.97x5.40mm_HandSolder, F.Cu at (-110.4, -56.9)
- added C111: 1uf, Capacitor_SMD:C_2220_5750Metric_Pad1.97x5.40mm_HandSolder, F.Cu at (-110.4, -49.9)
- added C112: 1uf, Capacitor_SMD:C_2220_5750Metric_Pad1.97x5.40mm_HandSolder, F.Cu at (-110.4, -43.0)
- added C113: 1uf, Capacitor_SMD:C_2220_5750Metric_Pad1.97x5.40mm_HandSolder, F.Cu at (-101.6, -63.8)
- added C114: 1uf, Capacitor_SMD:C_2220_5750Metric_Pad1.97x5.40mm_HandSolder, F.Cu at (-101.6, -56.9)
- added C115: 1uf, Capacitor_SMD:C_2220_5750Metric_Pad1.97x5.40mm_HandSolder, F.Cu at (-101.6, -49.9)
- added C116: 1uf, Capacitor_SMD:C_2220_5750Metric_Pad1.97x5.40mm_HandSolder, F.Cu at (-101.6, -43.0)
- added C12: 15p, Capacitor_SMD:C_0402_1005Metric, F.Cu at (-188.4, 99.6)
- added C13: 2.2u, Capacitor_SMD:C_0603_1608Metric, F.Cu at (-175.2, 92.5)
- added C14: 2.2u, Capacitor_SMD:C_0603_1608Metric, F.Cu at (-175.2, 95.0)
- added C15: 4.7u, Capacitor_SMD:C_0805_2012Metric, F.Cu at (181.7, 105.3)
- added C16: 220nF, Capacitor_SMD:C_0402_1005Metric, F.Cu at (193.5, 104.8)
- added C17: 4.7u, Capacitor_SMD:C_0805_2012Metric, F.Cu at (181.7, 108.3)
- added C18: 220nF, Capacitor_SMD:C_0402_1005Metric, F.Cu at (193.5, 106.8)
- added C19: 4.7u, Capacitor_SMD:C_0805_2012Metric, F.Cu at (181.7, 111.3)
- added C2: 100n, Capacitor_SMD:C_0402_1005Metric, F.Cu at (-188.4, 91.7)
- added C20: 220nF, Capacitor_SMD:C_0402_1005Metric, F.Cu at (193.5, 108.7)
- added C21: 4.7u, Capacitor_SMD:C_0805_2012Metric, F.Cu at (181.7, 114.3)
- added C22: 4.7u, Capacitor_SMD:C_0805_2012Metric, F.Cu at (181.7, 117.4)
- added C23: 4.7u, Capacitor_SMD:C_0805_2012Metric, F.Cu at (181.7, 120.4)
- added C24: 100n, Capacitor_SMD:C_0402_1005Metric, F.Cu at (193.5, 110.7)
- added C25: 100n, Capacitor_SMD:C_0402_1005Metric, F.Cu at (193.5, 112.7)
- added C26: 100n, Capacitor_SMD:C_0402_1005Metric, F.Cu at (193.5, 114.6)
- added C27: 100n, Capacitor_SMD:C_0402_1005Metric, F.Cu at (-188.4, 101.6)
- added C28: 100n, Capacitor_SMD:C_0402_1005Metric, F.Cu at (-185.5, 89.7)
- added C29: 15n, Capacitor_SMD:C_0603_1608Metric, F.Cu at (-175.2, 97.5)
- added C3: 100n, Capacitor_SMD:C_0402_1005Metric, F.Cu at (-188.4, 93.7)
- added C30: 1n, Capacitor_SMD:C_0603_1608Metric, F.Cu at (-175.2, 100.0)
- added C31: 100n, Capacitor_SMD:C_0402_1005Metric, F.Cu at (-185.5, 91.7)
- added C32: 100n, Capacitor_SMD:C_0402_1005Metric, F.Cu at (-185.5, 93.7)
- added C33: 100n, Capacitor_SMD:C_0402_1005Metric, F.Cu at (-185.5, 95.6)
- added C34: 100n, Capacitor_SMD:C_0402_1005Metric, F.Cu at (-185.5, 97.6)
- added C35: 1n, Capacitor_SMD:C_0603_1608Metric, F.Cu at (-171.2, 90.0)
- added C36: 15n, Capacitor_SMD:C_0603_1608Metric, F.Cu at (-171.2, 92.5)
- added C37: 100n, Capacitor_SMD:C_0402_1005Metric, F.Cu at (-185.5, 99.6)
- added C38: 100n, Capacitor_SMD:C_0402_1005Metric, F.Cu at (-185.5, 101.6)
- added C39: 100n, Capacitor_SMD:C_0402_1005Metric, F.Cu at (-182.7, 89.7)
- added C4: 100n, Capacitor_SMD:C_0402_1005Metric, F.Cu at (-188.4, 95.6)
- added C40: 1n, Capacitor_SMD:C_0603_1608Metric, F.Cu at (-171.2, 95.0)
- added C41: 15n, Capacitor_SMD:C_0603_1608Metric, F.Cu at (-171.2, 97.5)
- added C42: 10u, Capacitor_SMD:C_1210_3225Metric_Pad1.33x2.70mm_HandSolder, F.Cu at (192.9, 119.6)
- added C43: 10u, Capacitor_SMD:C_1210_3225Metric_Pad1.33x2.70mm_HandSolder, F.Cu at (192.9, 123.8)
- added C44: 10u, Capacitor_SMD:C_1210_3225Metric_Pad1.33x2.70mm_HandSolder, F.Cu at (192.9, 128.1)
- added C45: 100n, Capacitor_SMD:C_0402_1005Metric, F.Cu at (-182.7, 91.7)
- added C46: 100n, Capacitor_SMD:C_0402_1005Metric, F.Cu at (-182.7, 93.7)
- added C47: 100n, Capacitor_SMD:C_0402_1005Metric, F.Cu at (-182.7, 95.6)
- added C48: 100n, Capacitor_SMD:C_0402_1005Metric, F.Cu at (-182.7, 97.6)
- added C49: 100n, Capacitor_SMD:C_0402_1005Metric, F.Cu at (-182.7, 99.6)
- added C5: 2.2u, Capacitor_SMD:C_0603_1608Metric, F.Cu at (-179.2, 90.0)
- added C50: 100n, Capacitor_SMD:C_0402_1005Metric, F.Cu at (-182.7, 101.6)
- added C51: 4.7u, Capacitor_SMD:C_0603_1608Metric_Pad1.08x0.95mm_HandSolder, F.Cu at (168.6, 105.1)
- added C52: 4.7u, Capacitor_SMD:C_0603_1608Metric_Pad1.08x0.95mm_HandSolder, F.Cu at (168.6, 107.6)
- added C53: 4.7u, Capacitor_SMD:C_0603_1608Metric_Pad1.08x0.95mm_HandSolder, F.Cu at (168.6, 110.1)
- added C54: 100n, Capacitor_SMD:C_0603_1608Metric_Pad1.08x0.95mm_HandSolder, F.Cu at (166.9, 68.7)
- added C55: 100n, Capacitor_SMD:C_0603_1608Metric_Pad1.08x0.95mm_HandSolder, F.Cu at (166.9, 71.2)
- added C56: 100n, Capacitor_SMD:C_0603_1608Metric_Pad1.08x0.95mm_HandSolder, F.Cu at (166.9, 73.7)
- added C57: 100n, Capacitor_SMD:C_0603_1608Metric_Pad1.08x0.95mm_HandSolder, F.Cu at (166.9, 76.2)
- added C58: 2.2uf, Capacitor_SMD:C_0603_1608Metric, F.Cu at (-113.5, 187.2)
- added C59: 2.2uf, Capacitor_SMD:C_0603_1608Metric, F.Cu at (-113.5, 189.7)
- added C6: 2.2u, Capacitor_SMD:C_0603_1608Metric, F.Cu at (-179.2, 92.5)
- added C60: 2.2uf, Capacitor_SMD:C_0603_1608Metric, F.Cu at (-113.5, 192.2)
- added C61: 33uF, Capacitor_SMD:CP_Elec_4x5.4, F.Cu at (-17.9, 170.0)
- added C62: 100nF, Capacitor_SMD:C_0402_1005Metric_Pad0.74x0.62mm_HandSolder, F.Cu at (-20.1, 158.2)
- added C63: 2.2uF, Capacitor_SMD:C_1210_3225Metric_Pad1.33x2.70mm_HandSolder, F.Cu at (-45.4, 186.0)
- added C64: 100nF, Capacitor_SMD:C_0402_1005Metric_Pad0.74x0.62mm_HandSolder, F.Cu at (-20.1, 160.2)
- added C65: 2.2uF, Capacitor_SMD:C_1210_3225Metric_Pad1.33x2.70mm_HandSolder, F.Cu at (-45.4, 190.3)
- added C66: 100uF, Capacitor_SMD:C_0402_1005Metric_Pad0.74x0.62mm_HandSolder, F.Cu at (-20.1, 162.1)
- added C67: 100nF, Capacitor_SMD:C_0402_1005Metric_Pad0.74x0.62mm_HandSolder, F.Cu at (-20.1, 164.1)
- added C68: 2.2uF, Capacitor_SMD:C_1210_3225Metric_Pad1.33x2.70mm_HandSolder, F.Cu at (-45.4, 194.5)
- added C69: 100nF, Capacitor_SMD:C_0402_1005Metric_Pad0.74x0.62mm_HandSolder, F.Cu at (-20.1, 166.1)
- added C7: 2.2u, Capacitor_SMD:C_0603_1608Metric, F.Cu at (-179.2, 95.0)
- added C70: 2.2uF, Capacitor_SMD:C_1210_3225Metric_Pad1.33x2.70mm_HandSolder, F.Cu at (-45.4, 198.8)
- added C71: 10uF, Capacitor_SMD:C_1210_3225Metric_Pad1.33x2.70mm_HandSolder, F.Cu at (-39.4, 186.0)
- added C72: 22uF, Capacitor_SMD:C_1210_3225Metric_Pad1.33x2.70mm_HandSolder, F.Cu at (-39.4, 190.3)
- added C73: 10uF, Capacitor_SMD:C_1210_3225Metric_Pad1.33x2.70mm_HandSolder, F.Cu at (-39.4, 194.5)
- added C74: 10uF, Capacitor_SMD:C_1210_3225Metric_Pad1.33x2.70mm_HandSolder, F.Cu at (-39.4, 198.8)
- added C75: 22uF, Capacitor_SMD:C_1210_3225Metric_Pad1.33x2.70mm_HandSolder, F.Cu at (-33.4, 186.0)
- added C76: 22uF, Capacitor_SMD:C_1210_3225Metric_Pad1.33x2.70mm_HandSolder, F.Cu at (-33.4, 190.3)
- added C77: 22uF, Capacitor_SMD:C_1210_3225Metric_Pad1.33x2.70mm_HandSolder, F.Cu at (-33.4, 194.5)
- added C78: 2.2u, Capacitor_SMD:C_0603_1608Metric, F.Cu at (-171.5, 105.8)
- added C79: 100n, Capacitor_SMD:C_0402_1005Metric, F.Cu at (-172.1, 123.5)
- added C8: 2.2u, Capacitor_SMD:C_0603_1608Metric, F.Cu at (-179.2, 97.5)
- added C80: 100n, Capacitor_SMD:C_0402_1005Metric, F.Cu at (-99.7, 115.2)
- added C81: 4.7u, Capacitor_SMD:C_0805_2012Metric, F.Cu at (-98.9, 109.7)
- added C82: 100n, Capacitor_SMD:C_0402_1005Metric, F.Cu at (-99.7, 117.2)
- added C83: 4.7u, Capacitor_SMD:C_0805_2012Metric, F.Cu at (-171.3, 113.6)
- added C84: 4.7u, Capacitor_SMD:C_0805_2012Metric, F.Cu at (-171.3, 116.6)
- added C85: 10uF, Capacitor_SMD:C_1210_3225Metric_Pad1.33x2.70mm_HandSolder, F.Cu at (-33.4, 198.8)
- added C86: 100nF, Capacitor_SMD:C_0805_2012Metric, F.Cu at (-11.8, 168.6)
- added C87: 100n, Capacitor_SMD:C_0402_1005Metric, F.Cu at (-99.7, 119.2)
- added C88: 10uF, Capacitor_SMD:C_1210_3225Metric_Pad1.33x2.70mm_HandSolder, F.Cu at (-98.2, 88.4)
- added C89: 560u, Capacitor_THT:CP_Radial_D16.0mm_P7.50mm, F.Cu at (-192.0, -82.8)
- added C9: 2.2u, Capacitor_SMD:C_0603_1608Metric, F.Cu at (-179.2, 100.0)
- added C90: 560u, Capacitor_THT:CP_Radial_D16.0mm_P7.50mm, F.Cu at (-192.0, -65.3)
- added C91: 4.7u, Capacitor_SMD:C_0805_2012Metric, F.Cu at (-98.9, 112.8)
- added C92: 560u, Capacitor_THT:CP_Radial_D16.0mm_P7.50mm, F.Cu at (-192.0, -47.7)
- added C93: 560u, Capacitor_THT:CP_Radial_D16.0mm_P7.50mm, F.Cu at (-192.0, -30.2)
- added C94: 560u, Capacitor_THT:CP_Radial_D16.0mm_P7.50mm, F.Cu at (-173.9, -82.8)
- added C95: 560u, Capacitor_THT:CP_Radial_D16.0mm_P7.50mm, F.Cu at (-173.9, -65.3)
- added C96: 560u, Capacitor_THT:CP_Radial_D16.0mm_P7.50mm, F.Cu at (-173.9, -47.7)
- added C97: 560u, Capacitor_THT:CP_Radial_D16.0mm_P7.50mm, F.Cu at (-173.9, -30.2)
- added C98: 560u, Capacitor_THT:CP_Radial_D16.0mm_P7.50mm, F.Cu at (-155.9, -82.8)
- added C99: 560u, Capacitor_THT:CP_Radial_D16.0mm_P7.50mm, F.Cu at (-155.9, -65.3)
- added D1: STTH2R06A, Diode_SMD:D_SMA, F.Cu at (188.0, 106.1)
- added D10: D, Diode_SMD:D_SOD-123, F.Cu at (31.5, 96.6)
- added D11: D, Diode_SMD:D_SOD-123, F.Cu at (31.5, 100.0)
- added D12: D, Diode_SMD:D_SOD-123, F.Cu at (37.3, 83.2)
- added D13: D, Diode_SMD:D_SOD-123, F.Cu at (37.3, 86.6)
- added D14: D, Diode_SMD:D_SOD-123, F.Cu at (37.3, 89.9)
- added D15: D, Diode_SMD:D_SOD-123, F.Cu at (37.3, 93.3)
- added D16: D, Diode_SMD:D_SOD-123, F.Cu at (37.3, 96.6)
- added D17: D, Diode_SMD:D_SOD-123, F.Cu at (37.3, 100.0)
- added D18: D, Diode_SMD:D_SOD-123, F.Cu at (43.1, 83.2)
- added D19: D, Diode_SMD:D_SOD-123, F.Cu at (43.1, 86.6)
- added D2: STTH2R06A, Diode_SMD:D_SMA, F.Cu at (188.0, 110.6)
- added D20: D, Diode_SMD:D_SOD-123, F.Cu at (43.1, 89.9)
- added D21: D, Diode_SMD:D_SOD-123, F.Cu at (43.1, 93.3)
- added D22: green, Diode_SMD:D_0603_1608Metric_Pad1.05x0.95mm_HandSolder, F.Cu at (-191.9, 133.4)
- added D23: CFSH05-20L, Diode_SMD:D_SOD-882, F.Cu at (-12.0, 164.6)
- added D24: BZT52C3V6-7-F, Diode_SMD:D_SOD-123, F.Cu at (-22.1, 191.2)
- added D25: BZT52C3V6-7-F, Diode_SMD:D_SOD-123, F.Cu at (-22.1, 194.6)
- added D26: red, Diode_SMD:D_0603_1608Metric_Pad1.05x0.95mm_HandSolder, F.Cu at (-191.9, 136.0)
- added D27: blue, Diode_SMD:D_0603_1608Metric_Pad1.05x0.95mm_HandSolder, F.Cu at (-191.9, 138.6)
- added D28: BAT46W, Diode_SMD:D_SOD-323F, F.Cu at (-115.9, 113.5)
- added D29: BZT52C5V6-7-F, Diode_SMD:D_SOD-123, F.Cu at (-22.1, 197.9)
- added D3: STTH2R06A, Diode_SMD:D_SMA, F.Cu at (188.0, 115.2)
- added D4: D, Diode_SMD:D_SOD-123F, F.Cu at (33.4, 103.9)
- added D5: D, Diode_SMD:D_SOD-123F, F.Cu at (33.4, 107.2)
- added D6: D, Diode_SMD:D_SOD-123, F.Cu at (31.5, 83.2)
- added D7: D, Diode_SMD:D_SOD-123, F.Cu at (31.5, 86.6)
- added D8: D, Diode_SMD:D_SOD-123, F.Cu at (31.5, 89.9)
- added D9: D, Diode_SMD:D_SOD-123, F.Cu at (31.5, 93.3)
- added J1: Conn_01x05, Connector_JST:JST_XH_B5B-XH-AM_1x05_P2.50mm_Vertical, F.Cu at (-126.6, 84.9)
- added J10: Conn_01x03, Connector_JST:JST_XH_B3B-XH-A_1x03_P2.50mm_Vertical, F.Cu at (-109.6, 108.3)
- added J14: BOOT0, Jumper:SolderJumper-2_P1.3mm_Open_RoundedPad1.0x1.5mm, F.Cu at (-168.1, 76.1)
- added J15: NRST, Jumper:SolderJumper-2_P1.3mm_Open_RoundedPad1.0x1.5mm, F.Cu at (-168.1, 79.6)
- added J2: USB_C_Receptacle_USB2.0, Connector_USB:USB_C_Receptacle_G-Switch_GT-USB-7051x, F.Cu at (-107.6, 116.4)
- added J3: Conn_01x06, Connector_JST:JST_XH_B6B-XH-A_1x06_P2.50mm_Vertical, F.Cu at (-126.6, 77.1)
- added J4: Conn_01x05, Connector_JST:JST_XH_B5B-XH-A_1x05_P2.50mm_Vertical, F.Cu at (-126.6, 92.7)
- added J5: Conn_01x03, Connector_JST:JST_XH_B3B-XH-A_1x03_P2.50mm_Vertical, F.Cu at (-109.6, 84.9)
- added J6: Conn_01x03, Connector_JST:JST_XH_B3B-XH-A_1x03_P2.50mm_Vertical, F.Cu at (-109.6, 92.7)
- added J7: Conn_01x05, Connector_JST:JST_XH_B5B-XH-A_1x05_P2.50mm_Vertical, F.Cu at (-126.6, 100.5)
- added J8: Conn_01x02, Connector_JST:JST_XH_B2B-XH-A_1x02_P2.50mm_Vertical, F.Cu at (-107.1, 77.1)
- added J9: Conn_01x03, Connector_JST:JST_XH_B3B-XH-A_1x03_P2.50mm_Vertical, F.Cu at (-109.6, 100.5)
- added JP1: Jumper_3_Bridged12, Jumper:SolderJumper-3_P1.3mm_Bridged2Bar12_RoundedPad1.0x1.5mm, F.Cu at (-98.3, 92.3)
- added JP2: Jumper_2_Open, Jumper:SolderJumper-2_P1.3mm_Open_RoundedPad1.0x1.5mm, F.Cu at (-115.9, 106.7)
- added JP3: Jumper_2_Open, Jumper:SolderJumper-2_P1.3mm_Open_RoundedPad1.0x1.5mm, F.Cu at (-115.9, 110.2)
- added JP4: Jumper_3_Bridged12, Jumper:SolderJumper-3_P1.3mm_Bridged2Bar12_RoundedPad1.0x1.5mm, F.Cu at (-18.9, 180.9)
- added L1: 10uh, Library:IND-SMD_L3.9-W3.9-1, F.Cu at (-27.7, 192.1)
- added L2: 10uh, Library:IND-SMD_L3.9-W3.9-1, F.Cu at (-27.7, 197.3)
- added L3: 10uH, Library:IND-SMD_L5.0-W5.0, F.Cu at (-18.2, 176.0)
- added L4: 10uh, Inductor_SMD:L_Abracon_ASPI-4030S, F.Cu at (-14.2, 186.7)
- added Q19: CJ3400, Package_TO_SOT_SMD:SOT-23_Handsoldering, F.Cu at (-97.9, 84.0)
- added R1: 0, Resistor_SMD:R_0603_1608Metric_Pad0.98x0.95mm_HandSolder, F.Cu at (168.6, 122.6)
- added R10: R, Resistor_SMD:R_0805_2012Metric_Pad1.20x1.40mm_HandSolder, F.Cu at (16.7, 97.8)
- added R14: R, Resistor_SMD:R_0805_2012Metric_Pad1.20x1.40mm_HandSolder, F.Cu at (16.7, 100.7)
- added R15: R, Resistor_SMD:R_0805_2012Metric_Pad1.20x1.40mm_HandSolder, F.Cu at (21.4, 83.0)
- added R16: R, Resistor_SMD:R_0805_2012Metric_Pad1.20x1.40mm_HandSolder, F.Cu at (21.4, 86.0)
- added R17: R, Resistor_SMD:R_0805_2012Metric_Pad1.20x1.40mm_HandSolder, F.Cu at (21.4, 88.9)
- added R18: R, Resistor_SMD:R_0805_2012Metric_Pad1.20x1.40mm_HandSolder, F.Cu at (21.4, 91.9)
- added R19: R, Resistor_SMD:R_0805_2012Metric_Pad1.20x1.40mm_HandSolder, F.Cu at (21.4, 94.8)
- added R2: 0, Resistor_SMD:R_0603_1608Metric_Pad0.98x0.95mm_HandSolder, F.Cu at (173.0, 105.1)
- added R23: R, Resistor_SMD:R_0805_2012Metric_Pad1.20x1.40mm_HandSolder, F.Cu at (21.4, 97.8)
- added R24: R, Resistor_SMD:R_0805_2012Metric_Pad1.20x1.40mm_HandSolder, F.Cu at (21.4, 100.7)
- added R25: R, Resistor_SMD:R_0805_2012Metric_Pad1.20x1.40mm_HandSolder, F.Cu at (26.2, 83.0)
- added R26: 5k1, Resistor_SMD:R_0603_1608Metric, F.Cu at (-128.1, 106.2)
- added R27: R, Resistor_SMD:R_0805_2012Metric_Pad1.20x1.40mm_HandSolder, F.Cu at (26.2, 86.0)
- added R28: R, Resistor_SMD:R_0805_2012Metric_Pad1.20x1.40mm_HandSolder, F.Cu at (26.2, 88.9)
- added R29: R, Resistor_SMD:R_0805_2012Metric_Pad1.20x1.40mm_HandSolder, F.Cu at (26.2, 91.9)
- added R3: 0, Resistor_SMD:R_0603_1608Metric_Pad0.98x0.95mm_HandSolder, F.Cu at (173.0, 107.6)
- added R33: 1k, Resistor_SMD:R_0603_1608Metric_Pad0.98x0.95mm_HandSolder, F.Cu at (-167.0, 90.0)
- added R34: 1k, Resistor_SMD:R_0603_1608Metric_Pad0.98x0.95mm_HandSolder, F.Cu at (-167.0, 92.5)
- added R35: 1k, Resistor_SMD:R_0603_1608Metric_Pad0.98x0.95mm_HandSolder, F.Cu at (-167.0, 95.0)
- added R36: 320k, Resistor_SMD:R_0603_1608Metric_Pad0.98x0.95mm_HandSolder, F.Cu at (173.0, 110.1)
- added R37: 10k, Resistor_SMD:R_0603_1608Metric_Pad0.98x0.95mm_HandSolder, F.Cu at (173.0, 112.6)
- added R38: 10k, Resistor_SMD:R_0603_1608Metric_Pad0.98x0.95mm_HandSolder, F.Cu at (-167.0, 97.5)
- added R39: 10k, Resistor_SMD:R_0603_1608Metric_Pad0.98x0.95mm_HandSolder, F.Cu at (-167.0, 100.0)
- added R4: 0, Resistor_SMD:R_0815_2038Metric, F.Cu at (-28.2, 186.7)
- added R40: 10k, Resistor_SMD:R_0603_1608Metric_Pad0.98x0.95mm_HandSolder, F.Cu at (173.0, 115.1)
- added R41: 10k, Resistor_SMD:R_0603_1608Metric_Pad0.98x0.95mm_HandSolder, F.Cu at (173.0, 117.6)
- added R42: 10k, Resistor_SMD:R_0603_1608Metric_Pad0.98x0.95mm_HandSolder, F.Cu at (173.0, 120.1)
- added R43: 240k, Resistor_SMD:R_1206_3216Metric_Pad1.30x1.75mm_HandSolder, F.Cu at (185.2, 75.2)
- added R44: 5.1k, Resistor_SMD:R_0603_1608Metric_Pad0.98x0.95mm_HandSolder, F.Cu at (171.2, 78.7)
- added R45: 240k, Resistor_SMD:R_1206_3216Metric_Pad1.30x1.75mm_HandSolder, F.Cu at (185.2, 78.5)
- added R46: 5.1k, Resistor_SMD:R_0603_1608Metric_Pad0.98x0.95mm_HandSolder, F.Cu at (175.6, 61.1)
- added R47: 240k, Resistor_SMD:R_1206_3216Metric_Pad1.30x1.75mm_HandSolder, F.Cu at (185.2, 81.8)
- added R48: 5.1k, Resistor_SMD:R_0603_1608Metric_Pad0.98x0.95mm_HandSolder, F.Cu at (175.6, 63.6)
- added R49: 480k, Resistor_SMD:R_1206_3216Metric_Pad1.30x1.75mm_HandSolder, F.Cu at (185.2, 85.1)
- added R5: R, Resistor_SMD:R_0805_2012Metric_Pad1.20x1.40mm_HandSolder, F.Cu at (16.7, 83.0)
- added R50: 10.2k, Resistor_SMD:R_0603_1608Metric_Pad0.98x0.95mm_HandSolder, F.Cu at (175.6, 66.2)
- added R51: 320k, Resistor_SMD:R_0603_1608Metric_Pad0.98x0.95mm_HandSolder, F.Cu at (177.3, 112.6)
- added R52: 10k, Resistor_SMD:R_0603_1608Metric_Pad0.98x0.95mm_HandSolder, F.Cu at (177.3, 115.1)
- added R53: 320k, Resistor_SMD:R_0603_1608Metric_Pad0.98x0.95mm_HandSolder, F.Cu at (177.3, 117.6)
- added R54: 10k, Resistor_SMD:R_0603_1608Metric_Pad0.98x0.95mm_HandSolder, F.Cu at (177.3, 120.1)
- added R55: 10k, Resistor_SMD:R_0603_1608Metric, F.Cu at (181.5, 123.1)
- added R56: 10k, Resistor_SMD:R_0603_1608Metric, F.Cu at (181.5, 125.6)
- added R57: 10k, Resistor_SMD:R_0603_1608Metric, F.Cu at (181.5, 128.1)
- added R58: 10k_NTC, Resistor_SMD:R_0603_1608Metric_Pad0.98x0.95mm_HandSolder, F.Cu at (-101.3, 187.2)
- added R59: 10k_NTC, Resistor_SMD:R_0603_1608Metric_Pad0.98x0.95mm_HandSolder, F.Cu at (-101.3, 189.7)
- added R6: R, Resistor_SMD:R_0805_2012Metric_Pad1.20x1.40mm_HandSolder, F.Cu at (16.7, 86.0)
- added R60: 10k_NTC, Resistor_SMD:R_0603_1608Metric_Pad0.98x0.95mm_HandSolder, F.Cu at (-101.3, 192.2)
- added R61: 10k, Resistor_SMD:R_0603_1608Metric, F.Cu at (-113.5, 194.8)
- added R62: 10k, Resistor_SMD:R_0603_1608Metric, F.Cu at (-113.5, 197.3)
- added R63: 10k, Resistor_SMD:R_0603_1608Metric, F.Cu at (-113.5, 199.8)
- added R64: 100k, Resistor_SMD:R_0603_1608Metric, F.Cu at (-11.4, 162.1)
- added R65: 220r, Resistor_SMD:R_0603_1608Metric, F.Cu at (-187.7, 133.3)
- added R66: 220r, Resistor_SMD:R_0603_1608Metric, F.Cu at (-187.7, 135.9)
- added R67: 1k, Resistor_SMD:R_0603_1608Metric, F.Cu at (-187.7, 138.4)
- added R68: 0, Resistor_SMD:R_0815_2038Metric, F.Cu at (-23.7, 186.7)
- added R69: 0, Resistor_SMD:R_0815_2038Metric, F.Cu at (-19.3, 186.7)
- added R7: R, Resistor_SMD:R_0805_2012Metric_Pad1.20x1.40mm_HandSolder, F.Cu at (16.7, 88.9)
- added R70: 1k, Resistor_SMD:R_0603_1608Metric, F.Cu at (-171.5, 108.3)
- added R71: 1k, Resistor_SMD:R_0603_1608Metric, F.Cu at (-171.5, 110.8)
- added R72: 10k, Resistor_SMD:R_0603_1608Metric, F.Cu at (-128.1, 108.7)
- added R73: 2k2, Resistor_SMD:R_0603_1608Metric, F.Cu at (-128.1, 111.2)
- added R74: 2k2, Resistor_SMD:R_0603_1608Metric, F.Cu at (-128.1, 113.7)
- added R75: 2k2, Resistor_SMD:R_0603_1608Metric, F.Cu at (-128.1, 116.2)
- added R76: 4.3k, Resistor_SMD:R_0603_1608Metric, F.Cu at (-128.1, 118.7)
- added R77: 4.3k, Resistor_SMD:R_0603_1608Metric, F.Cu at (-124.0, 106.2)
- added R78: 4.3k, Resistor_SMD:R_0603_1608Metric, F.Cu at (-124.0, 108.7)
- added R79: 2k2, Resistor_SMD:R_0603_1608Metric, F.Cu at (-124.0, 111.2)
- added R8: R, Resistor_SMD:R_0805_2012Metric_Pad1.20x1.40mm_HandSolder, F.Cu at (16.7, 91.9)
- added R80: 4.3k, Resistor_SMD:R_0603_1608Metric, F.Cu at (-124.0, 113.7)
- added R81: 2k2, Resistor_SMD:R_0603_1608Metric, F.Cu at (-124.0, 116.2)
- added R82: 4.3k, Resistor_SMD:R_0603_1608Metric, F.Cu at (-124.0, 118.7)
- added R83: 120ohm, Resistor_SMD:R_0603_1608Metric, F.Cu at (-120.0, 106.2)
- added R84: 5k1, Resistor_SMD:R_0603_1608Metric, F.Cu at (-120.0, 108.7)
- added R85: 10k, Resistor_SMD:R_0603_1608Metric, F.Cu at (20.3, 103.4)
- added R86: 10k, Resistor_SMD:R_0603_1608Metric, F.Cu at (20.3, 106.0)
- added R87: 10k, Resistor_SMD:R_0603_1608Metric, F.Cu at (20.3, 108.5)
- added R88: 10k, Resistor_SMD:R_0603_1608Metric, F.Cu at (20.3, 111.0)
- added R89: 10k, Resistor_SMD:R_0603_1608Metric, F.Cu at (20.3, 113.5)
- added R9: R, Resistor_SMD:R_0805_2012Metric_Pad1.20x1.40mm_HandSolder, F.Cu at (16.7, 94.8)
- added R90: 10k, Resistor_SMD:R_0603_1608Metric, F.Cu at (20.3, 116.0)
- added R91: 10k, Resistor_SMD:R_0603_1608Metric, F.Cu at (24.3, 103.4)
- added R92: 10k, Resistor_SMD:R_0603_1608Metric, F.Cu at (24.3, 106.0)
- added R93: 10k, Resistor_SMD:R_0603_1608Metric, F.Cu at (24.3, 108.5)
- added R94: 68k, Resistor_SMD:R_0603_1608Metric_Pad0.98x0.95mm_HandSolder, F.Cu at (-12.4, 180.1)
- added R95: 820k, Resistor_SMD:R_0603_1608Metric_Pad0.98x0.95mm_HandSolder, F.Cu at (-12.4, 182.6)
- added R96: 4R7, Resistor_SMD:R_0805_2012Metric, F.Cu at (-12.4, 174.4)
- added R97: 4R7, Resistor_SMD:R_0805_2012Metric, F.Cu at (-12.4, 177.3)
- added R98: 100r, Resistor_SMD:R_0603_1608Metric, F.Cu at (-120.0, 111.2)
- added R99: 10k, Resistor_SMD:R_0603_1608Metric, F.Cu at (-120.0, 113.7)
- added U1: STM32F405RGTx, Package_QFP:LQFP-64_10x10mm_P0.5mm, F.Cu at (-182.6, 81.5)
- added U10: MC74VHC1GT66, Package_TO_SOT_SMD:SOT-353_SC-70-5, F.Cu at (-192.0, 84.2)
- added U11: MC74VHC1GT66, Package_TO_SOT_SMD:SOT-353_SC-70-5, F.Cu at (-192.0, 88.1)
- added U12: MC74VHC1GT66, Package_TO_SOT_SMD:SOT-353_SC-70-5, F.Cu at (-192.0, 92.0)
- added U13: MC74VHC1GT66, Package_TO_SOT_SMD:SOT-353_SC-70-5, F.Cu at (-192.0, 95.9)
- added U14: AMS1117-3.3, Package_TO_SOT_SMD:SOT-223-3_TabPin2, F.Cu at (-14.3, 193.7)
- added U15: LP5907MFX-3.3, Package_TO_SOT_SMD:SOT-23-5, F.Cu at (-15.9, 159.6)
- added U16: TPS62173DSG, Package_SON:WSON-8-1EP_2x2mm_P0.5mm_EP0.9x1.6mm, F.Cu at (-11.2, 159.1)
- added U17: BMI160, Package_LGA:Bosch_LGA-14_3x2.5mm_P0.5mm, F.Cu at (-171.0, 120.4)
- added U18: ESP32-C3_SUPERMINI_SMD, Library:MODULE_ESP32-C3_SUPERMINI, F.Cu at (-183.8, 118.0)
- added U19: TLV61047DDC, Package_TO_SOT_SMD:SOT-23-5, F.Cu at (-15.9, 164.2)
- added U20: TJA1051T-3, Package_SO:SOIC-8_3.9x4.9mm_P1.27mm, F.Cu at (-96.9, 77.1)
- added U21: SRV05-4, Package_TO_SOT_SMD:SOT-23-6, F.Cu at (-98.6, 96.8)
- added U22: SRV05-4, Package_TO_SOT_SMD:SOT-23-6, F.Cu at (-98.6, 101.4)
- added U23: SRV05-4, Package_TO_SOT_SMD:SOT-23-6, F.Cu at (-98.6, 106.0)
- added U24: PQDE6W-Q110 / RD5-110S12W, Library:PQDE6W, F.Cu at (-47.7, 158.0)
- added U5: INA240/241, Package_TO_SOT_SMD:SOT-23-8, F.Cu at (-172.8, 76.7)
- added U6: MC74VHC1GT66, Package_TO_SOT_SMD:SOT-353_SC-70-5, F.Cu at (-192.0, 76.3)
- added U7: ~, Package_TO_SOT_SMD:SOT-23-8, F.Cu at (-172.8, 81.3)
- added U8: MC74VHC1GT66, Package_TO_SOT_SMD:SOT-353_SC-70-5, F.Cu at (-192.0, 80.2)
- added U9: ~, Package_TO_SOT_SMD:SOT-23-8, F.Cu at (-172.8, 85.9)
- added Y1: 8m, Crystal:Crystal_SMD_3225-4Pin_3.2x2.5mm, F.Cu at (-167.6, 83.7)
Connections:
- net +12V renamed +15V

Commit message: modified:   tolt/conn.kicad_sch 	modified:   tolt/converters.kicad_sch 	modified:   tolt/inter.kicad_sch 	modified:   tolt/powerstage.kicad_sch 	modified:   tolt/stm32.kicad_sch 	modified:   tolt/tolt.kicad_pcb 	modified:   tolt/tolt.kicad_pro
Parts:
- added C117: 2.2uF, Capacitor_SMD:C_1210_3225Metric, F.Cu at (-184.4, 213.2)
- added C118: 100nF, Capacitor_SMD:C_0402_1005Metric, F.Cu at (107.7, 155.4)
- added C119: 2.2uF, Capacitor_SMD:C_1210_3225Metric, F.Cu at (111.7, 152.6)
- added C120: 100nF, Capacitor_SMD:C_0402_1005Metric, F.Cu at (118.7, 155.3)
- added C121: 2.2uF, Capacitor_SMD:C_1210_3225Metric, F.Cu at (123.0, 152.6)
- added C122: 100nF, Capacitor_SMD:C_0402_1005Metric, F.Cu at (-124.5, 55.7)
- added C123: 100nF, Capacitor_SMD:C_0402_1005Metric, F.Cu at (129.5, 155.3)
- added C124: 2.2uF, Capacitor_SMD:C_1210_3225Metric, F.Cu at (130.6, 153.0)
- added C125: 100nF, Capacitor_SMD:C_0402_1005Metric, F.Cu at (91.6, 148.6)
- added C126: 2.2uF, Capacitor_SMD:C_1210_3225Metric, F.Cu at (92.6, 146.3)
- added C127: 100nF, Capacitor_SMD:C_0402_1005Metric, F.Cu at (96.7, 148.6)
- added R100: 2k2, Resistor_SMD:R_0603_1608Metric, F.Cu at (153.8, 153.2)
- added R101: 2k2, Resistor_SMD:R_0603_1608Metric, F.Cu at (153.8, 154.9)
- added R102: 2k2, Resistor_SMD:R_0603_1608Metric, F.Cu at (153.8, 151.4)
- C116: value 1uf -> 100nF; footprint Capacitor_SMD:C_2220_5750Metric_Pad1.97x5.40mm_HandSolder -> Capacitor_SMD:C_0402_1005Metric
- C51, C52, C53, C54, C55, C56, C57: footprint Capacitor_SMD:C_0603_1608Metric_Pad1.08x0.95mm_HandSolder -> Capacitor_SMD:C_0603_1608Metric
- C62, C64, C66, C67, C69: footprint Capacitor_SMD:C_0402_1005Metric_Pad0.74x0.62mm_HandSolder -> Capacitor_SMD:C_0402_1005Metric
- C63, C65, C68, C70, C71, C72, C73, C74, C75, C76, C77, C85, C88: footprint Capacitor_SMD:C_1210_3225Metric_Pad1.33x2.70mm_HandSolder -> Capacitor_SMD:C_1210_3225Metric
- D4, D5: footprint Diode_SMD:D_SOD-123F -> Diode_SMD:D_SOD-123
- R1, R2, R3, R33, R34, R35, R36, R37, R38, R39, R40, R41, R42, R44, R46, R48, R50, R51, R52, R53, R54, R94, R95: footprint Resistor_SMD:R_0603_1608Metric_Pad0.98x0.95mm_HandSolder -> Resistor_SMD:R_0603_1608Metric
- R10, R14, R15, R16, R17, R18, R19, R23, R24, R25, R27, R28, R29, R5, R6, R7, R8, R9: footprint Resistor_SMD:R_0805_2012Metric_Pad1.20x1.40mm_HandSolder -> Resistor_SMD:R_0805_2012Metric
- R43, R45, R47, R49: footprint Resistor_SMD:R_1206_3216Metric_Pad1.30x1.75mm_HandSolder -> Resistor_SMD:R_1206_3216Metric
- moved C95 347.0 mm to (149.4, 60.7), turned to 90 degrees
- moved C94 337.8 mm to (131.8, 60.7), turned to 90 degrees
- moved U8 332.1 mm to (123.4, 184.4)
- moved U1 327.9 mm to (139.4, 143.3)
- moved C12 320.7 mm to (129.5, 142.3)
- moved C11 320.4 mm to (129.5, 137.8), turned to 180 degrees
- moved C93 319.4 mm to (114.2, 60.7), turned to 90 degrees
- moved C39 317.9 mm to (119.8, 187.4)
- moved C105 317.8 mm to (154.1, 98.3), turned to -90 degrees
- moved C37 316.7 mm to (119.8, 183.4)
- moved C38 316.7 mm to (119.8, 185.4)
- moved U9 311.9 mm to (121.0, 190.7)
- moved C100 310.9 mm to (140.5, 46.1), turned to 90 degrees
- moved U6 310.3 mm to (99.0, 184.2)
- moved C92 308.3 mm to (96.7, 60.7), turned to 90 degrees
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Connections:
- C116 pad 1: +BATT -> VCC
- C116 pad 2: GNDPWR -> GND
- C21 pad 2: +12V -> +15V
- C22 pad 2: +12V -> +15V
- C23 pad 2: +12V -> +15V
- C24 pad 2: +12V -> +15V
- C25 pad 2: +12V -> +15V
- C26 pad 2: +12V -> +15V
- C42 pad 1: +12V -> +15V
- C43 pad 1: +12V -> +15V
- C44 pad 1: +12V -> +15V
- J3 pad 3: /IO/HALL_1 -> Net-(J3-Pin_3)
- J3 pad 4: /IO/HALL_2 -> Net-(J3-Pin_4)
- J3 pad 5: /IO/HALL_3 -> Net-(J3-Pin_5)
- R11 pad 1: GNDPWR -> /INTER/SENS_A+
- R11 pad 2: /INTER/SENS_A+ -> GNDPWR
- R20 pad 1: GNDPWR -> /INTER/SENS_B+
- R20 pad 2: /INTER/SENS_B+ -> GNDPWR
- R30 pad 1: GNDPWR -> /INTER/SENS_C+
- R30 pad 2: /INTER/SENS_C+ -> GNDPWR
- R73 pad 1: /IO/HALL_1 -> Net-(J3-Pin_3)
- R74 pad 1: /IO/HALL_2 -> Net-(J3-Pin_4)
- R75 pad 1: /IO/HALL_3 -> Net-(J3-Pin_5)
- R79 pad 1: adc1 -> /IO/SCK_ADC_EXT
- R79 pad 2: /IO/SCK_ADC_EXT -> adc1
- R80 pad 2: adc1 -> /IO/SCK_ADC_EXT
- R81 pad 1: adc2 -> /IO/MISO_ADC_EXT2
- R81 pad 2: /IO/MISO_ADC_EXT2 -> adc2
- R82 pad 2: adc2 -> /IO/MISO_ADC_EXT2
- U22 pad 1: adc1 -> adc2
- U22 pad 3: adc2 -> adc1
Routing:
- net Net-(J3-Pin_5): track 0.00 -> 1.41 mm
- net Net-(J3-Pin_4): track 0.00 -> 1.41 mm
- net Net-(J3-Pin_3): track 0.00 -> 1.41 mm
- net /IO/HALL_3: track 0.00 -> 1.39 mm
- net /IO/HALL_2: track 0.00 -> 1.39 mm
- net /IO/HALL_1: track 0.00 -> 1.39 mm
Other:
- board outline added: 111.1 x 130 mm

Commit message: some
Parts:
- moved C116 368.3 mm to (173.6, 134.9)
- moved C117 368.3 mm to (175.0, 132.7)
- moved C87 368.3 mm to (169.2, 134.5)
- moved J9 368.3 mm to (169.4, 138.4)
- moved R98 368.3 mm to (171.2, 134.6)
- moved U18 350.4 mm to (160.0, 185.7)
- moved C122 325.6 mm to (184.7, 157.6)
- moved J1 317.8 mm to (178.3, 162.4)
- moved R26 283.8 mm to (154.1, 137.3)
- moved R84 280.6 mm to (158.1, 145.6), turned to 180 degrees
- moved JP3 275.1 mm to (158.1, 136.2), turned to 90 degrees
- moved J2 264.9 mm to (156.1, 141.4)
- moved R83 221.6 mm to (97.5, 148.5), turned to 180 degrees
- moved U20 205.4 mm to (97.2, 144.0), turned to -90 degrees
- moved C45 101.6 mm to (-93.8, 140.8)
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Connections:
- J4 pad 2: Canh -> VCC
- J4 pad 3: VCC -> Canl
- J4 pad 4: Canl -> Canh
- J8 pad 1: Canh -> Canl
- J8 pad 2: Canl -> Canh

Commit message: aa
Parts:
- added REF**: CP_Radial_D18.0mm_P7.50mm, Capacitor_THT:CP_Radial_D18.0mm_P7.50mm, F.Cu at (110.3, 38.9)
- added REF**: CP_Radial_D18.0mm_P7.50mm, Capacitor_THT:CP_Radial_D18.0mm_P7.50mm, F.Cu at (100.2, 62.8)
- added REF**: CP_Radial_D18.0mm_P7.50mm, Capacitor_THT:CP_Radial_D18.0mm_P7.50mm, F.Cu at (130.8, 38.9)
- added REF**: CP_Radial_D18.0mm_P7.50mm, Capacitor_THT:CP_Radial_D18.0mm_P7.50mm, F.Cu at (90.0, 38.9)
- added REF**: CP_Radial_D18.0mm_P7.50mm, Capacitor_THT:CP_Radial_D18.0mm_P7.50mm, F.Cu at (59.7, 62.8)
- added REF**: CP_Radial_D18.0mm_P7.50mm, Capacitor_THT:CP_Radial_D18.0mm_P7.50mm, F.Cu at (79.8, 62.8)
- added REF**: CP_Radial_D18.0mm_P7.50mm, Capacitor_THT:CP_Radial_D18.0mm_P7.50mm, F.Cu at (120.6, 62.8)
- added REF**: CP_Radial_D18.0mm_P7.50mm, Capacitor_THT:CP_Radial_D18.0mm_P7.50mm, F.Cu at (140.9, 62.8)
- added REF**: CP_Radial_D18.0mm_P7.50mm, Capacitor_THT:CP_Radial_D18.0mm_P7.50mm, F.Cu at (69.7, 38.9)
- added REF**: CP_Radial_D18.0mm_P7.50mm, Capacitor_THT:CP_Radial_D18.0mm_P7.50mm, F.Cu at (151.0, 38.9)
- C11, C12, C27, C28, C29, C32, C33, C36, C37, C38, C41, U1, Y1: moved to B.Cu
- J1: footprint Connector_JST:JST_XH_B5B-XH-AM_1x05_P2.50mm_Vertical -> Connector_PinSocket_2.54mm:PinSocket_2x03_P2.54mm_Vertical; moved to B.Cu
- J10, J5, J6, J9: footprint Connector_JST:JST_XH_B3B-XH-A_1x03_P2.50mm_Vertical -> Connector_JST:JST_PH_B3B-PH-K_1x03_P2.00mm_Vertical
- J3: footprint Connector_JST:JST_XH_B6B-XH-A_1x06_P2.50mm_Vertical -> Connector_JST:JST_PH_B6B-PH-K_1x06_P2.00mm_Vertical
- J4, J7: footprint Connector_JST:JST_XH_B5B-XH-A_1x05_P2.50mm_Vertical -> Connector_JST:JST_PH_B5B-PH-K_1x05_P2.00mm_Vertical
- J8: footprint Connector_JST:JST_XH_B2B-XH-A_1x02_P2.50mm_Vertical -> Connector_JST:JST_PH_B2B-PH-K_1x02_P2.00mm_Vertical
- moved C79 62.1 mm to (-32.0, 137.4)
- moved C81 62.1 mm to (-47.7, 74.6)
- moved C91 62.1 mm to (-47.7, 77.6)
- moved U17 62.1 mm to (-30.9, 134.3)
- moved C1 62.1 mm to (-4.93, 74.5)
- moved C10 62.1 mm to (8.26, 74.7)
- moved C13 62.1 mm to (8.26, 77.3)
- moved C14 62.1 mm to (8.26, 79.8)
- moved C2 62.1 mm to (-4.93, 76.4)
- moved C3 62.1 mm to (-4.93, 78.4)
- moved C4 62.1 mm to (-4.93, 80.4)
- moved C45 62.1 mm to (-42.6, 105.7)
- moved C46 62.1 mm to (-42.6, 107.6)
- moved C47 62.1 mm to (-42.6, 109.6)
- moved C48 62.1 mm to (-42.6, 111.6)
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Connections:
- U8 pad 3: unconnected-(U8-GND-Pad3) -> GND

Commit message: b
Parts:
- moved L1 14.3 mm to (53.2, 254.4)
- moved U17 12.5 mm to (-25.5, 145.6)
- moved C78 12.5 mm to (-26.0, 131.0)
- moved C83 12.5 mm to (-25.7, 138.8)
- moved C84 12.5 mm to (-25.7, 141.8)
- moved R70 12.5 mm to (-26.0, 133.5)
- moved C79 12.5 mm to (-26.5, 148.7)
- moved R71 12.5 mm to (-26.0, 136.0)
- moved C89 10.6 mm to (62.1, 25.7)
- moved C96 10.6 mm to (70.8, 11.1)
- moved C100 10.6 mm to (141.1, 11.1)
- moved C90 10.6 mm to (79.7, 25.7)
- moved C92 10.6 mm to (97.2, 25.7)
- moved C93 10.6 mm to (114.8, 25.7)
- moved C94 10.6 mm to (132.4, 25.7)
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
Commit message: modified:   tolt/conn.kicad_sch 	modified:   tolt/powerstage.kicad_sch 	modified:   tolt/stm32.kicad_sch 	modified:   tolt/tolt.kicad_pcb 	modified:   tolt/tolt.kicad_pro 	modified:   tolt/tolt.kicad_sch
Parts:
- added C128: 1uf, Capacitor_SMD:C_2220_5750Metric_Pad1.97x5.40mm_HandSolder, F.Cu at (154.1, 72.3)
- added C129: 1uf, Capacitor_SMD:C_2220_5750Metric_Pad1.97x5.40mm_HandSolder, F.Cu at (147.1, 72.3)
- added C130: 1uf, Capacitor_SMD:C_2220_5750Metric_Pad1.97x5.40mm_HandSolder, F.Cu at (140.2, 72.3)
- added C131: 1uf, Capacitor_SMD:C_2220_5750Metric_Pad1.97x5.40mm_HandSolder, F.Cu at (133.2, 72.3)
- added C132: 1uf, Capacitor_SMD:C_2220_5750Metric_Pad1.97x5.40mm_HandSolder, F.Cu at (126.3, 72.3)
- added C133: 1uf, Capacitor_SMD:C_2220_5750Metric_Pad1.97x5.40mm_HandSolder, F.Cu at (119.3, 72.3)
- added C134: 1uf, Capacitor_SMD:C_2220_5750Metric_Pad1.97x5.40mm_HandSolder, F.Cu at (112.3, 72.3)
- added C135: 1uf, Capacitor_SMD:C_2220_5750Metric_Pad1.97x5.40mm_HandSolder, F.Cu at (105.4, 72.3)
- added C136: 1uf, Capacitor_SMD:C_2220_5750Metric_Pad1.97x5.40mm_HandSolder, F.Cu at (98.4, 72.3)
- added C137: 1uf, Capacitor_SMD:C_2220_5750Metric_Pad1.97x5.40mm_HandSolder, F.Cu at (91.5, 72.3)
- added C138: 1uf, Capacitor_SMD:C_2220_5750Metric_Pad1.97x5.40mm_HandSolder, F.Cu at (84.5, 72.3)
- added C139: 1uf, Capacitor_SMD:C_2220_5750Metric_Pad1.97x5.40mm_HandSolder, F.Cu at (77.6, 72.3)
- added C140: 1uf, Capacitor_SMD:C_2220_5750Metric_Pad1.97x5.40mm_HandSolder, F.Cu at (70.6, 72.3)
- added C141: 1uf, Capacitor_SMD:C_2220_5750Metric_Pad1.97x5.40mm_HandSolder, F.Cu at (63.7, 72.3)
- added C142: 1uf, Capacitor_SMD:C_2220_5750Metric_Pad1.97x5.40mm_HandSolder, F.Cu at (56.7, 72.3)
- added R103: 10k, Resistor_SMD:R_0603_1608Metric, F.Cu at (123.2, 81.5)
- added R104: 10k, Resistor_SMD:R_0603_1608Metric, F.Cu at (134.8, 81.5)
- added R105: 10k, Resistor_SMD:R_0603_1608Metric, F.Cu at (146.5, 81.5)
- added R106: 10k, Resistor_SMD:R_0603_1608Metric, F.Cu at (111.0, 81.5)
- added R107: 10k, Resistor_SMD:R_0603_1608Metric, F.Cu at (87.6, 81.5)
- added R108: 10k, Resistor_SMD:R_0603_1608Metric, F.Cu at (99.3, 81.5)
- added R109: 10k, Resistor_SMD:R_0603_1608Metric, F.Cu at (63.8, 81.5)
- added R110: 10k, Resistor_SMD:R_0603_1608Metric, F.Cu at (75.5, 81.5)
- added R111: 10k, Resistor_SMD:R_0603_1608Metric, F.Cu at (52.1, 81.5)
- C27, C28, C29, C32, C33, C36, C37, C38, C41: moved to F.Cu
- JP1, JP2, JP3, JP4, R58, R59, R60, R85, R86, R87, R88, R89, R90, R91, R92, R93: moved to B.Cu
- moved D27 219.6 mm to (166.1, 125.4), turned to 180 degrees
- moved D26 219.0 mm to (166.1, 128.0), turned to 180 degrees
- moved R67 218.8 mm to (169.6, 125.5), turned to 180 degrees
- moved D22 218.5 mm to (166.1, 130.6), turned to 180 degrees
- moved R66 218.3 mm to (169.6, 128.0), turned to 180 degrees
- moved R65 217.8 mm to (169.6, 130.6), turned to 180 degrees
- moved C84 202.7 mm to (174.0, 176.5), turned to 90 degrees
- moved U11 200.5 mm to (143.0, 149.2)
- moved C83 200.3 mm to (171.0, 176.5), turned to 90 degrees
- moved U23 199.8 mm to (134.2, 154.3)
- moved U12 195.5 mm to (138.7, 149.2)
- moved U13 190.5 mm to (134.5, 149.2)
- moved C48 189.1 mm to (142.4, 151.1)
- moved C45 188.2 mm to (140.9, 147.8), turned to 90 degrees
- moved C49 184.6 mm to (138.2, 151.1)
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Connections:
- U1 pad 2: unconnected-(U1-PC13-Pad2) -> /IO/HALL_3
- U1 pad 3: unconnected-(U1-PC14-Pad3) -> /IO/HALL_2
- U1 pad 33: /aux logic/scl_bmi -> unconnected-(U1-PB12-Pad33)
- U1 pad 37: /IO/HALL_1 -> unconnected-(U1-PC6-Pad37)
- U1 pad 38: /IO/HALL_2 -> unconnected-(U1-PC7-Pad38)
- U1 pad 39: /IO/HALL_3 -> unconnected-(U1-PC8-Pad39)
- U1 pad 4: unconnected-(U1-PC15-Pad4) -> /IO/HALL_1
- U1 pad 50: /logic/NRF_swdio -> unconnected-(U1-PA15-Pad50)
- U1 pad 55: /logic/NRF_swclk -> /aux logic/scl_bmi
Routing:
- net VCC: track 0.00 -> 26.2 mm, vias 0 -> 5
- net Net-(JP3-A): track 0.00 -> 9.16 mm, vias 0 -> 4
- net Net-(U24-VIN): track 0.00 -> 3.71 mm
Other:
- outline, holes or cut-outs redrawn
- copper layers 4 -> 6
- board text added: "JLCJLCJLCJLCJLC"
