File: tolt/tolt.kicad_pcb (KiCad board)
At the start: 6 copper layers, 111.1 x 130 mm, 356 parts, among them J1 Conn_01x05, J10 Conn_01x03, J14 BOOT0, J15 NRST, J2 USB_C_Receptacle_USB2.0, J3 Conn_01x06, J4 Conn_01x05, J5 Conn_01x03, J6 Conn_01x03, J7 Conn_01x05, J8 Conn_01x02, J9 Conn_01x03, Q1 NMOS, Q10 NMOS, Q11 NMOS, Q12 NMOS, Q13 NMOS, Q14 NMOS, Q15 NMOS, Q16 NMOS, Q17 NMOS, Q18 NMOS, Q19 CJ3400, Q2 NMOS, Q3 NMOS, Q4 NMOS, Q5 NMOS, Q6 NMOS, Q7 NMOS, Q8 NMOS, Q9 NMOS, U1 STM32F405RGTx, U10 MC74VHC1GT66, U11 MC74VHC1GT66, U12 MC74VHC1GT66, U13 MC74VHC1GT66, U14 AMS1117-3.3, U15 LP5907MFX-3.3, U16 TPS62173DSG, U17 BMI160, U18 ESP32-C3_SUPERMINI_SMD, U19 TLV61047DDC, U2 L6491, U20 TJA1051T-3, U21 SRV05-4, U22 SRV05-4, U23 SRV05-4, U24 PQDE6W-Q110 / RD5-110S12W, U3 L6491, U4 L6491, U5 INA240/241, U6 MC74VHC1GT66, U8 MC74VHC1GT66, Y1 8m

Commit message: Update PCB component placements and replace jumper
Moved several SMD components to new coordinates for layout optimization. Removed J14 (BOOT0 solder jumper) and added JP4 (3-pad solder jumper) for converter section. Updated silkscreen and fab UUIDs for multiple components.
Parts:
- J14, J15: moved to B.Cu
- JP4: moved to F.Cu
- moved J14 160.0 mm to (151.5, 145.0), turned to 180 degrees
- moved J15 150.0 mm to (136.3, 153.1), turned to 90 degrees
- moved R38 149.2 mm to (151.5, 145.7)
- moved R39 138.7 mm to (137.1, 153.3), turned to 90 degrees
- moved C58 39.5 mm to (26.7, 90.6)
- moved C60 39.5 mm to (26.9, 101.1)
- moved R61 39.5 mm to (26.7, 92.1)
- moved R63 39.5 mm to (26.9, 102.7)
- moved C14 34.4 mm to (32.0, 104.6)
- moved JP4 30.7 mm to (114.9, 135.5), turned to 180 degrees
- moved C76 26.1 mm to (114.0, 130.9)
- moved L4 26.1 mm to (108.7, 135.6)
- moved C74 26.1 mm to (104.7, 130.9)
- moved C75 26.1 mm to (117.4, 130.9)
- moved D23 26.1 mm to (111.5, 132.6)
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Routing:
- net Net-(J14-Pin_2): track 0.00 -> 6.88 mm, vias 0 -> 1
- net /IO/rst: track 0.00 -> 6.73 mm, vias 0 -> 1
