File: tolt/conn.kicad_sch (KiCad schematic)
At the start: 33 parts, among them J1 Conn_01x05, J2 USB_C_Receptacle_USB2.0, J3 Conn_01x06, J4 Conn_01x05, J5 Conn_01x03, J6 Conn_01x03, J7 Conn_01x05, J8 Conn_01x02, U20 TJA1051T-3, U21 SRV05-4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

Commit message: new file:   tolt/Library.pretty/IND-SMD_L3.9-W3.9-1.kicad_mod 	new file:   tolt/Library.pretty/IND-SMD_L5.0-W5.0.kicad_mod 	modified:   tolt/auxl.kicad_sch 	modified:   tolt/conn.kicad_sch 	modified:   tolt/converters.kicad_sch 	new file:   tolt/fp-lib-table 	modified:   tolt/inter.kicad_sch 	modified:   tolt/powerstage.kicad_sch 	modified:   tolt/stm32.kicad_sch 	modified:   tolt/tolt.kicad_sch
Parts:
- J1: footprint (none) -> Connector_JST:JST_XH_B5B-XH-AM_1x05_P2.50mm_Vertical
- J3: footprint (none) -> Connector_JST:JST_XH_B6B-XH-A_1x06_P2.50mm_Vertical
- J4, J7: footprint (none) -> Connector_JST:JST_XH_B5B-XH-A_1x05_P2.50mm_Vertical
- J5, J6: footprint (none) -> Connector_JST:JST_XH_B3B-XH-A_1x03_P2.50mm_Vertical
- J8: footprint (none) -> Connector_JST:JST_XH_B2B-XH-A_1x02_P2.50mm_Vertical
- JP1: footprint (none) -> Jumper:SolderJumper-3_P1.3mm_Bridged2Bar12_RoundedPad1.0x1.5mm
Changed lines of the file:
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@@
 			)
 		)
-		(property "Footprint" ""
+		(property "Footprint" "Connector_JST:JST_XH_B3B-XH-A_1x03_P2.50mm_Vertical"
 			(at 248.666 140.462 0)
 			(effects
@@
 			)
 		)
-		(property "Footprint" ""
+		(property "Footprint" "Connector_JST:JST_XH_B5B-XH-A_1x05_P2.50mm_Vertical"
 			(at 203.454 81.026 0)
 			(effects
@@
 			)
 		)
-		(property "Footprint" ""
+		(property "Footprint" "Connector_JST:JST_XH_B5B-XH-A_1x05_P2.50mm_Vertical"
 			(at 242.062 44.958 0)
 			(effects
@@
 			)
 		)
-		(property "Footprint" ""
+		(property "Footprint" "Connector_JST:JST_XH_B6B-XH-A_1x06_P2.50mm_Vertical"
 			(at 137.922 43.942 0)
 			(effects
@@
 			)
 		)
-		(property "Footprint" ""
+		(property "Footprint" "Connector_JST:JST_XH_B2B-XH-A_1x02_P2.50mm_Vertical"
 			(at 220.218 28.448 0)
 			(effects
@@
 			)
 		)
-		(property "Footprint" ""
+		(property "Footprint" "Connector_JST:JST_XH_B5B-XH-AM_1x05_P2.50mm_Vertical"
 			(at 248.92 79.756 0)
 			(effects
@@
 			)
 		)
-		(property "Footprint" ""
+		(property "Footprint" "Jumper:SolderJumper-3_P1.3mm_Bridged2Bar12_RoundedPad1.0x1.5mm"
 			(at 107.442 27.686 0)
 			(effects
@@
 			)
 		)
-		(property "Footprint" ""
+		(property "Footprint" "Connector_JST:JST_XH_B3B-XH-A_1x03_P2.50mm_Vertical"
 			(at 248.666 110.998 0)
 			(effects

Commit message: new file:   tolt/Library.pretty/PQDE6W.kicad_mod 	modified:   tolt/auxl.kicad_sch 	modified:   tolt/conn.kicad_sch 	modified:   tolt/converters.kicad_sch 	modified:   tolt/powerstage.kicad_sch 	modified:   tolt/tolt.kicad_pcb 	modified:   tolt/tolt.kicad_sch
Parts:
- added C87: 100n, Capacitor_SMD:C_0402_1005Metric, symbol Device:C
- added C88: 10uF, Capacitor_SMD:C_1210_3225Metric_Pad1.33x2.70mm_HandSolder, symbol Device:C
- added D28: BAT46W, Diode_SMD:D_SOD-323F, symbol Device:D_Zener
- added J10, J9: Conn_01x03, Connector_JST:JST_XH_B3B-XH-A_1x03_P2.50mm_Vertical, symbol Connector_Generic:Conn_01x03
- added Q19: CJ3400, Package_TO_SOT_SMD:SOT-23_Handsoldering, symbol Simulation_SPICE:NMOS
- added R98: 100r, Resistor_SMD:R_0603_1608Metric, symbol Device:R
- added R99: 10k, Resistor_SMD:R_0603_1608Metric, symbol Device:R
Connections:
- net GND: now also C87.1, C88.1, J10.1 (Pin_1), J9.1 (Pin_1), Q19.1 (D), R99.1
- net VCC: now also J9.3 (Pin_3)
- net ppm: now reaches U23.4 (IO3)
- net ppm: now also J9.2 (Pin_2), R98.2
- new net: D28.2 (A), J10.2 (Pin_2), Q19.3 (S)
- new net +12V: C88.2, D28.1 (K), J10.3 (Pin_3)
- new net SERVO: C87.2, R98.1
- new net aux: Q19.2 (G), R99.2

Commit message: modified:   tolt/conn.kicad_sch 	modified:   tolt/converters.kicad_sch 	modified:   tolt/inter.kicad_sch 	modified:   tolt/powerstage.kicad_sch 	modified:   tolt/stm32.kicad_sch 	modified:   tolt/tolt.kicad_pcb 	modified:   tolt/tolt.kicad_pro
Parts:
- added C116, C118, C120, C122, C123, C125, C127: 100nF, Capacitor_SMD:C_0402_1005Metric, symbol Device:C
- added C117, C119, C121, C124, C126: 2.2uF, Capacitor_SMD:C_1210_3225Metric, symbol Device:C
- added R100, R101, R102: 2k2, Resistor_SMD:R_0603_1608Metric, symbol Device:R
- C88: footprint Capacitor_SMD:C_1210_3225Metric_Pad1.33x2.70mm_HandSolder -> Capacitor_SMD:C_1210_3225Metric
Connections:
- net +5V: now also C118.1, C119.1, C120.1, C121.1, C122.2, C125.1, C126.1
- net GND: now also C116.2, C117.2, C118.2, C119.2, C120.2, C121.2, C122.1, C123.2, C124.2, C125.2, C126.2, C127.2
- net HALL_1: now also R102.1; no longer J3.3 (Pin_3), R73.1
- net HALL_2: now also R101.1; no longer J3.4 (Pin_4), R74.1
- net HALL_3: now also R100.1; no longer J3.5 (Pin_5), R75.1
- net MISO_ADC_EXT2: now also R81.1, R82.2; no longer R81.2
- net SCK_ADC_EXT: now also R79.1, R80.2; no longer R79.2
- net VCC: now also C116.1, C117.1, C123.1, C124.1, C127.1
- net adc1: now also R79.2, U22.3 (IO2); no longer R79.1, R80.2, U22.1 (IO1)
- net adc2: now also R81.2, U22.1 (IO1); no longer R81.1, R82.2, U22.3 (IO2)
- new net: J3.5 (Pin_5), R100.2, R75.1
- new net: J3.3 (Pin_3), R102.2, R73.1
- new net: J3.4 (Pin_4), R101.2, R74.1
Other:
- moved on the sheet: R76, R77, R78, R79, R80, R81, R82

Commit message: some
Connections:
- net Canh: now also J4.4 (Pin_4), J8.2 (Pin_2); no longer J4.2 (Pin_2), J8.1 (Pin_1)
- net Canl: now also J4.3 (Pin_3), J8.1 (Pin_1); no longer J4.4 (Pin_4), J8.2 (Pin_2)
- net VCC: now also J4.2 (Pin_2); no longer J4.3 (Pin_3)
Changed lines of the file:
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@@
+	)
+	(junction
+		(at 222.758 42.418)
+		(diameter 0)
+		(color 0 0 0 0)
 	)
 	(junction
@@
 	)
 	(junction
-		(at 220.218 41.148)
+		(at 220.218 48.768)
 		(diameter 0)
 		(color 0 0 0 0)
@@
 	(junction
 		(at 107.442 70.358)
-		(diameter 0)
-		(color 0 0 0 0)
-	)
-	(junction
-		(at 222.758 47.498)
 		(diameter 0)
 		(color 0 0 0 0)
@@
 	(wire
 		(pts
-			(xy 220.218 42.418) (xy 236.982 42.418)
-		)
-		(stroke
-			(width 0)
-			(type default)
-		)
-	)
-	(wire
-		(pts
 			(xy 267.208 75.438) (xy 243.586 75.438)
 		)
@@
 	(wire
 		(pts
+			(xy 221.234 42.418) (xy 222.758 42.418)
+		)
+		(stroke
+			(width 0)
+			(type default)
+		)
+	)
+	(wire
+		(pts
 			(xy 59.944 145.034) (xy 59.944 147.574)
 		)
@@
 	(wire
 		(pts
-			(xy 222.758 33.528) (xy 222.758 47.498)
-		)
-		(stroke
-			(width 0)
-			(type default)
-		)
-	)
-	(wire
-		(pts
 			(xy 151.638 126.746) (xy 151.638 129.286)
 		)
@@
 	(wire
 		(pts
+			(xy 222.758 42.418) (xy 232.918 42.418)
+		)
+		(stroke
+			(width 0)
+			(type default)
+		)
+	)
+	(wire
+		(pts
 			(xy 107.442 31.496) (xy 115.316 31.496)
 		)
@@
 	(wire
 		(pts
-			(xy 220.218 33.528) (xy 220.218 41.148)
+			(xy 229.616 44.958) (xy 236.982 44.958)
 		)
 		(stroke
@@
 	(wire
 		(pts
-			(xy 208.534 41.148) (xy 220.218 41.148)
+			(xy 208.534 41.148) (xy 221.234 41.148)
 		)
 		(stroke
@@
 	(wire
 		(pts
+			(xy 220.218 33.528) (xy 220.218 48.768)
+		)
+		(stroke
+			(width 0)
+			(type default)
+		)
+	)
+	(wire
+		(pts
 			(xy 103.886 166.624) (xy 91.186 166.624)
 		)
@@
 	(wire
 		(pts
-			(xy 222.758 47.498) (xy 236.982 47.498)
-		)
-		(stroke
-			(width 0)
-			(type default)
-		)
-	)
-	(wire
-		(pts
 			(xy 244.094 84.836) (xy 243.84 84.836)
 		)
@@
 	(wire
 		(pts
-			(xy 220.218 41.148) (xy 220.218 42.418)
+			(xy 222.758 33.528) (xy 222.758 42.418)
+		)
+		(stroke
+			(width 0)
+			(type default)
+		)
+	)
+	(wire
+		(pts
+			(xy 221.234 41.148) (xy 221.234 42.418)
 		)
 		(stroke
@@
 	(wire
 		(pts
-			(xy 208.534 48.768) (xy 222.758 48.768)
+			(xy 208.534 48.768) (xy 220.218 48.768)
 		)
 		(stroke
@@
 	(wire
 		(pts
+			(xy 222.758 47.498) (xy 229.616 47.498)
+		)
+		(stroke
+			(width 0)
+			(type default)
+		)
+	)
+	(wire
+		(pts
 			(xy 124.46 30.734) (xy 124.46 41.402)
 		)
@@
 	(wire
 		(pts
+			(xy 232.918 47.498) (xy 236.982 47.498)
+		)
+		(stroke
+			(width 0)
+			(type default)
+		)
+	)
+	(wire
+		(pts
 			(xy 99.314 39.116) (xy 99.314 49.022)
 		)
@@
 	(wire
 		(pts
+			(xy 220.218 48.768) (xy 222.758 48.768)
+		)
+		(stroke
+			(width 0)
+			(type default)
+		)
+	)
+	(wire
+		(pts
 			(xy 244.856 58.42) (xy 232.156 58.42)
 		)
@@
 	(wire
 		(pts
+			(xy 232.918 42.418) (xy 232.918 47.498)
+		)
+		(stroke
+			(width 0)
+			(type default)
+		)
+	)
+	(wire
+		(pts
 			(xy 243.332 74.676) (xy 243.586 74.676)
 		)
@@
 		(pts
 			(xy 122.682 38.862) (xy 122.682 31.496)
+		)
+		(stroke
+			(width 0)
+			(type default)
+		)
+	)
+	(wire
+		(pts
+			(xy 229.616 44.958) (xy 229.616 47.498)
 		)
 		(stroke
@@
 	(symbol
 		(lib_id "power:VCC")
-		(at 236.982 44.958 90)
+		(at 236.982 42.418 90)
 		(unit 1)
 		(exclude_from_sim no)
@@
 		(fields_autoplaced yes)
 		(property "Reference" "#PWR0213"
-			(at 240.792 44.958 0)
+			(at 240.792 42.418 0)
 			(effects
 				(font
@@
 		)
 		(property "Value" "VCC"
-			(at 233.426 44.9579 90)
+			(at 233.426 42.4179 90)
 			(effects
 				(font
@@
 		)
 		(property "Footprint" ""
-			(at 236.982 44.958 0)
+			(at 236.982 42.418 0)
 			(effects
 				(font
@@
 		)
 		(property "Datasheet" ""
-			(at 236.982 44.958 0)
+			(at 236.982 42.418 0)
 			(effects
 				(font
@@
 		)
 		(property "Description" "Power symbol creates a global label with name \"VCC\""
-			(at 236.982 44.958 0)
-			(effects
-				(font
+			(at 236.982 42.418 0)
+			(effects
+				(font

Commit message: aa
Parts:
- J1: footprint Connector_JST:JST_XH_B5B-XH-AM_1x05_P2.50mm_Vertical -> Connector_PinSocket_2.54mm:PinSocket_2x03_P2.54mm_Vertical; symbol Connector_Generic:Conn_01x05 -> Connector_Generic:Conn_01x06
- J10, J5, J6, J9: footprint Connector_JST:JST_XH_B3B-XH-A_1x03_P2.50mm_Vertical -> Connector_JST:JST_PH_B3B-PH-K_1x03_P2.00mm_Vertical
- J3: footprint Connector_JST:JST_XH_B6B-XH-A_1x06_P2.50mm_Vertical -> Connector_JST:JST_PH_B6B-PH-K_1x06_P2.00mm_Vertical
- J4, J7: footprint Connector_JST:JST_XH_B5B-XH-A_1x05_P2.50mm_Vertical -> Connector_JST:JST_PH_B5B-PH-K_1x05_P2.00mm_Vertical; symbol Connector_Generic:Conn_01x05 -> Connector_Generic:Conn_01x06
- J8: footprint Connector_JST:JST_XH_B2B-XH-A_1x02_P2.50mm_Vertical -> Connector_JST:JST_PH_B2B-PH-K_1x02_P2.00mm_Vertical
Connections:
- no-connect marks 2 -> 3
Changed lines of the file:
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@@
 	)
 	(no_connect
+		(at 243.84 87.376)
+	)
+	(no_connect
 		(at 59.944 155.194)
 	)
@@
 			)
 		)
-		(property "Footprint" "Connector_JST:JST_XH_B3B-XH-A_1x03_P2.50mm_Vertical"
+		(property "Footprint" "Connector_JST:JST_PH_B3B-PH-K_1x03_P2.00mm_Vertical"
 			(at 91.948 145.542 0)
 			(effects
@@
 			)
 		)
-		(property "Footprint" "Connector_JST:JST_XH_B3B-XH-A_1x03_P2.50mm_Vertical"
+		(property "Footprint" "Connector_JST:JST_PH_B3B-PH-K_1x03_P2.00mm_Vertical"
 			(at 248.666 140.462 0)
 			(effects
@@
 			)
 		)
-		(property "Footprint" "Connector_JST:JST_XH_B3B-XH-A_1x03_P2.50mm_Vertical"
+		(property "Footprint" "Connector_JST:JST_PH_B3B-PH-K_1x03_P2.00mm_Vertical"
 			(at 135.128 109.474 0)
 			(effects
@@
 	)
 	(symbol
-		(lib_id "Connector_Generic:Conn_01x05")
+		(lib_id "Connector_Generic:Conn_01x06")
 		(at 203.454 81.026 0)
 		(unit 1)
@@
 		(fields_autoplaced yes)
 		(property "Reference" "J7"
-			(at 205.74 79.7559 0)
+			(at 205.74 81.0259 0)
 			(effects
 				(font
@@
 		)
 		(property "Value" "Conn_01x05"
-			(at 205.74 82.2959 0)
+			(at 205.74 83.5659 0)
 			(effects
 				(font
@@
 			)
 		)
-		(property "Footprint" "Connector_JST:JST_XH_B5B-XH-A_1x05_P2.50mm_Vertical"
+		(property "Footprint" "Connector_JST:JST_PH_B5B-PH-K_1x05_P2.00mm_Vertical"
 			(at 203.454 81.026 0)
 			(effects
@@
 			)
 		)
-		(property "Description" "Generic connector, single row, 01x05, script generated (kicad-library-utils/schlib/autogen/connector/)"
+		(property "Description" "Generic connector, single row, 01x06, script generated (kicad-library-utils/schlib/autogen/connector/)"
 			(at 203.454 81.026 0)
 			(effects
@@
 		(pin "5"
 		)
+		(pin "6"
+		)
 		(instances
 			(project ""
@@
 	)
 	(symbol
-		(lib_id "Connector_Generic:Conn_01x05")
+		(lib_id "Connector_Generic:Conn_01x06")
 		(at 242.062 44.958 0)
 		(unit 1)
@@
 		(fields_autoplaced yes)
 		(property "Reference" "J4"
-			(at 244.348 43.6879 0)
+			(at 245.11 44.9579 0)
 			(effects
 				(font
@@
 		)
 		(property "Value" "Conn_01x05"
-			(at 244.348 46.2279 0)
+			(at 245.11 47.4979 0)
 			(effects
 				(font
@@
 			)
 		)
-		(property "Footprint" "Connector_JST:JST_XH_B5B-XH-A_1x05_P2.50mm_Vertical"
+		(property "Footprint" "Connector_JST:JST_PH_B5B-PH-K_1x05_P2.00mm_Vertical"
 			(at 242.062 44.958 0)
 			(effects
@@
 			)
 		)
-		(property "Description" "Generic connector, single row, 01x05, script generated (kicad-library-utils/schlib/autogen/connector/)"
+		(property "Description" "Generic connector, single row, 01x06, script generated (kicad-library-utils/schlib/autogen/connector/)"
 			(at 242.062 44.958 0)
 			(effects
@@
 		(pin "3"
 		)
+		(pin "6"
+		)
 		(instances
 			(project "tolt"
@@
 			)
 		)
-		(property "Footprint" "Connector_JST:JST_XH_B6B-XH-A_1x06_P2.50mm_Vertical"
+		(property "Footprint" "Connector_JST:JST_PH_B6B-PH-K_1x06_P2.00mm_Vertical"
 			(at 137.922 43.942 0)
 			(effects
@@
 		(pin "4"
 		)
-		(pin "6"
-		)
 		(pin "2"
 		)
 		(pin "5"
 		)
+		(pin "6"
+		)
 		(instances
 			(project ""
@@
 			)
 		)
-		(property "Footprint" "Connector_JST:JST_XH_B2B-XH-A_1x02_P2.50mm_Vertical"
+		(property "Footprint" "Connector_JST:JST_PH_B2B-PH-K_1x02_P2.00mm_Vertical"
 			(at 220.218 28.448 0)
 			(effects
@@
 	)
 	(symbol
-		(lib_id "Connector_Generic:Conn_01x05")
+		(lib_id "Connector_Generic:Conn_01x06")
 		(at 248.92 79.756 0)
 		(unit 1)
@@
 		(fields_autoplaced yes)
 		(property "Reference" "J1"
-			(at 251.206 78.4859 0)
+			(at 251.46 79.7559 0)
 			(effects
 				(font
@@
 		)
 		(property "Value" "Conn_01x05"
-			(at 251.206 81.0259 0)
+			(at 251.46 82.2959 0)
 			(effects
 				(font
@@
 			)
 		)
-		(property "Footprint" "Connector_JST:JST_XH_B5B-XH-AM_1x05_P2.50mm_Vertical"
+		(property "Footprint" "Connector_PinSocket_2.54mm:PinSocket_2x03_P2.54mm_Vertical"
 			(at 248.92 79.756 0)
 			(effects
@@
 			)
 		)
-		(property "Description" "Generic connector, single row, 01x05, script generated (kicad-library-utils/schlib/autogen/connector/)"
+		(property "Description" "Generic connector, single row, 01x06, script generated (kicad-library-utils/schlib/autogen/connector/)"
 			(at 248.92 79.756 0)
 			(effects
@@
 		(pin "3"
 		)
+		(pin "6"
+		)
 		(instances
 			(project ""
@@
 			)
 		)
-		(property "Footprint" "Connector_JST:JST_XH_B3B-XH-A_1x03_P2.50mm_Vertical"
+		(property "Footprint" "Connector_JST:JST_PH_B3B-PH-K_1x03_P2.00mm_Vertical"
 			(at 248.666 110.998 0)
 			(effects

Commit message: b
Connections:
- no-connect marks 3 -> 4
Changed lines of the file:
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@@
+	)
+	(no_connect
+		(at 198.374 88.646)
 	)
 	(no_connect

Commit message: modified:   tolt/conn.kicad_sch 	modified:   tolt/powerstage.kicad_sch 	modified:   tolt/stm32.kicad_sch 	modified:   tolt/tolt.kicad_pcb 	modified:   tolt/tolt.kicad_pro 	modified:   tolt/tolt.kicad_sch
Parts:
- removed J4, J7: Conn_01x05, Connector_JST:JST_PH_B5B-PH-K_1x05_P2.00mm_Vertical, symbol Connector_Generic:Conn_01x06
- added J4, J7: Conn_01x05, Connector_JST:JST_PH_B5B-PH-K_1x05_P2.00mm_Vertical, symbol Connector_Generic:Conn_01x05
Connections:
- net +5V: now also J4.1 (Pin_1)
- net ADC_15: now also J7.2 (Pin_2)
- net Canh: now also J4.4 (Pin_4)
- net Canl: now also J4.3 (Pin_3)
- net GND: now also J4.5 (Pin_5), J7.5 (Pin_5)
- net RX_SDA_NSS: now also J7.4 (Pin_4)
- net TX_SCL_MOSI: now also J7.3 (Pin_3)
- net VCC: now also J4.2 (Pin_2), J7.1 (Pin_1)
Changed lines of the file:
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@@
 	(wire
 		(pts
+			(xy 236.982 47.244) (xy 236.982 46.228)
+		)
+		(stroke
+			(width 0)
+			(type default)
+		)
+	)
+	(wire
+		(pts
 			(xy 208.534 41.148) (xy 221.234 41.148)
 		)
@@
 	(wire
 		(pts
+			(xy 195.326 86.106) (xy 198.374 86.106)
+		)
+		(stroke
+			(width 0)
+			(type default)
+		)
+	)
+	(wire
+		(pts
 			(xy 103.886 166.624) (xy 91.186 166.624)
 		)
@@
 	(wire
 		(pts
+			(xy 236.982 41.148) (xy 236.982 42.418)
+		)
+		(stroke
+			(width 0)
+			(type default)
+		)
+	)
+	(wire
+		(pts
 			(xy 244.094 84.836) (xy 243.84 84.836)
 		)
@@
 	(wire
 		(pts
-			(xy 232.918 47.498) (xy 236.982 47.498)
+			(xy 232.918 47.244) (xy 236.982 47.244)
 		)
 		(stroke
@@
 	(wire
 		(pts
+			(xy 236.982 44.958) (xy 236.982 43.688)
+		)
+		(stroke
+			(width 0)
+			(type default)
+		)
+	)
+	(wire
+		(pts
+			(xy 236.982 48.768) (xy 236.982 50.038)
+		)
+		(stroke
+			(width 0)
+			(type default)
+		)
+	)
+	(wire
+		(pts
 			(xy 107.442 62.738) (xy 107.442 59.436)
 		)
@@
 	(wire
 		(pts
+			(xy 236.982 38.608) (xy 236.982 39.878)
+		)
+		(stroke
+			(width 0)
+			(type default)
+		)
+	)
+	(wire
+		(pts
 			(xy 164.084 121.666) (xy 161.544 121.666)
 		)
@@
 	(wire
 		(pts
-			(xy 232.918 42.418) (xy 232.918 47.498)
+			(xy 232.918 42.418) (xy 232.918 47.244)
 		)
 		(stroke
@@
 	(symbol
 		(lib_id "power:GND")
-		(at 198.374 86.106 0)
+		(at 195.326 86.106 0)
 		(unit 1)
 		(exclude_from_sim no)
@@
 		(fields_autoplaced yes)
 		(property "Reference" "#PWR0208"
-			(at 198.374 92.456 0)
+			(at 195.326 92.456 0)
 			(effects
 				(font
@@
 		)
 		(property "Value" "GND"
-			(at 198.374 91.186 0)
+			(at 195.326 91.186 0)
 			(effects
 				(font
@@
 		)
 		(property "Footprint" ""
-			(at 198.374 86.106 0)
+			(at 195.326 86.106 0)
 			(effects
 				(font
@@
 		)
 		(property "Datasheet" ""
-			(at 198.374 86.106 0)
+			(at 195.326 86.106 0)
 			(effects
 				(font
@@
 		)
 		(property "Description" ""
-			(at 198.374 86.106 0)
+			(at 195.326 86.106 0)
 			(effects
 				(font
@@
 	)
 	(symbol
-		(lib_id "Connector_Generic:Conn_01x06")
-		(at 203.454 81.026 0)
-		(unit 1)
-		(exclude_from_sim no)
-		(in_bom yes)
-		(on_board yes)
-		(dnp no)
-		(fields_autoplaced yes)
-		(property "Reference" "J7"
-			(at 205.74 81.0259 0)
-			(effects
-				(font
-					(size 1.27 1.27)
-				)
-				(justify left)
-			)
-		)
-		(property "Value" "Conn_01x05"
-			(at 205.74 83.5659 0)
-			(effects
-				(font
-					(size 1.27 1.27)
-				)
-				(justify left)
-			)
-		)
-		(property "Footprint" "Connector_JST:JST_PH_B5B-PH-K_1x05_P2.00mm_Vertical"
-			(at 203.454 81.026 0)
-			(effects
-				(font
-					(size 1.27 1.27)
-				)
-				(hide yes)
-			)
-		)
-		(property "Datasheet" "~"
-			(at 203.454 81.026 0)
-			(effects
-				(font
-					(size 1.27 1.27)
-				)
-				(hide yes)
-			)
-		)
-		(property "Description" "Generic connector, single row, 01x06, script generated (kicad-library-utils/schlib/autogen/connector/)"
-			(at 203.454 81.026 0)
-			(effects
-				(font
-					(size 1.27 1.27)
-				)
-				(hide yes)
-			)
-		)
-		(pin "1"
-		)
-		(pin "4"
-		)
-		(pin "3"
-		)
-		(pin "2"
-		)
-		(pin "5"
-		)
-		(pin "6"
-		)
-		(instances
-			(project ""
-				(path "/38c63d96-01d7-4159-b7c0-aa8cee77c3e9/4189330a-b7ac-4caa-ad9c-153fd2ec5fe4"
-					(reference "J7")
-					(unit 1)
-				)
-			)
-		)
-	)
-	(symbol
-		(lib_id "Connector_Generic:Conn_01x06")
-		(at 242.062 44.958 0)
-		(unit 1)
-		(exclude_from_sim no)
-		(in_bom yes)
-		(on_board yes)
-		(dnp no)
-		(fields_autoplaced yes)
-		(property "Reference" "J4"
-			(at 245.11 44.9579 0)
-			(effects
-				(font
-					(size 1.27 1.27)
-				)
-				(justify left)
-			)
-		)
-		(property "Value" "Conn_01x05"
-			(at 245.11 47.4979 0)
-			(effects
-				(font
-					(size 1.27 1.27)
-				)
-				(justify left)
-			)
-		)
-		(property "Footprint" "Connector_JST:JST_PH_B5B-PH-K_1x05_P2.00mm_Vertical"
-			(at 242.062 44.958 0)
-			(effects
-				(font
-					(size 1.27 1.27)
-				)
-				(hide yes)
-			)
-		)
-		(property "Datasheet" "~"
-			(at 242.062 44.958 0)
-			(effects
-				(font
-					(size 1.27 1.27)
-				)
-				(hide yes)
-			)
-		)
-		(property "Description" "Generic connector, single row, 01x06, script generated (kicad-library-utils/schlib/autogen/connector/)"
-			(at 242.062 44.958 0)
-			(effects
-				(font
-					(size 1.27 1.27)
-				)
-				(hide yes)
-			)
-		)
-		(pin "2"
-		)
-		(pin "4"
-		)
-		(pin "5"
-		)
-		(pin "1"
-		)
-		(pin "3"
-		)
-		(pin "6"
-		)
-		(instances
-			(project "tolt"
-				(path "/38c63d96-01d7-4159-b7c0-aa8cee77c3e9/4189330a-b7ac-4caa-ad9c-153fd2ec5fe4"
-					(reference "J4")
-					(unit 1)
-				)
-			)
-		)
-	)
-	(symbol
 		(lib_id "power:GND")
 		(at 132.842 51.562 0)
@@
 	)
 	(symbol
+		(lib_id "Connector_Generic:Conn_01x05")
+		(at 203.454 81.026 0)
+		(unit 1)
+		(exclude_from_sim no)
+		(in_bom yes)
+		(on_board yes)
+		(dnp no)
+		(fields_autoplaced yes)
+		(property "Reference" "J7"
+			(at 206.502 79.7559 0)
+			(effects
+				(font
+					(size 1.27 1.27)
+				)
+				(justify left)
+			)
+		)
+		(property "Value" "Conn_01x05"
+			(at 206.502 82.2959 0)
+			(effects
+				(font
+					(size 1.27 1.27)
+				)
+				(justify left)
+			)
+		)
+		(property "Footprint" "Connector_JST:JST_PH_B5B-PH-K_1x05_P2.00mm_Vertical"
+			(at 203.454 81.026 0)
+			(effects
+				(font
+					(size 1.27 1.27)
+				)
+				(hide yes)
+			)
+		)
+		(property "Datasheet" "~"
+			(at 203.454 81.026 0)
+			(effects
+				(font
+					(size 1.27 1.27)
+				)
+				(hide yes)
+			)
+		)
+		(property "Description" "Generic connector, single row, 01x05, script generated (kicad-library-utils/schlib/autogen/connector/)"
+			(at 203.454 81.026 0)
+			(effects
+				(font
+					(size 1.27 1.27)
+				)
+				(hide yes)
+			)
+		)
+		(pin "1"
+		)
+		(pin "3"
+		)
+		(pin "2"
+		)
+		(pin "5"
+		)
+		(pin "4"
+		)
+		(instances
+			(project "tolt"
+				(path "/38c63d96-01d7-4159-b7c0-aa8cee77c3e9/4189330a-b7ac-4caa-ad9c-153fd2ec5fe4"
+					(reference "J7")
+					(unit 1)
+				)
+			)
+		)
+	)
+	(symbol
 		(lib_id "power:GND")
 		(at 44.704 165.354 0)
@@
 					(unit 1)
 				)
+			)
+		)
+	)
+	(symbol
+		(lib_id "Connector_Generic:Conn_01x05")
+		(at 242.062 43.688 0)
+		(unit 1)
+		(exclude_from_sim no)
+		(in_bom yes)
+		(on_board yes)
+		(dnp no)
+		(fields_autoplaced yes)
+		(property "Reference" "J4"
+			(at 245.11 42.4179 0)
+			(effects
+				(font
+					(size 1.27 1.27)
+				)
+				(justify left)
+			)
+		)
+		(property "Value" "Conn_01x05"
+			(at 245.11 44.9579 0)
+			(effects
+				(font
+					(size 1.27 1.27)
+				)
+				(justify left)
+			)
+		)
+		(property "Footprint" "Connector_JST:JST_PH_B5B-PH-K_1x05_P2.00mm_Vertical"
+			(at 242.062 43.688 0)
+			(effects
+				(font
+					(size 1.27 1.27)
+				)
+				(hide yes)
+			)
+		)
+		(property "Datasheet" "~"
+			(at 242.062 43.688 0)
+			(effects
+				(font
+					(size 1.27 1.27)
+				)
+				(hide yes)
+			)
+		)
+		(property "Description" "Generic connector, single row, 01x05, script generated (kicad-library-utils/schlib/autogen/connector/)"
+			(at 242.062 43.688 0)
+			(effects
+				(font
+					(size 1.27 1.27)
+				)
+				(hide yes)
+			)
+		)
+		(pin "1"
+		)
+		(pin "3"
+		)
+		(pin "2"
+		)
+		(pin "5"
+		)
+		(pin "4"
+		)
+		(instances
+			(project ""
+				(path "/38c63d96-01d7-4159-b7c0-aa8cee77c3e9/4189330a-b7ac-4caa-ad9c-153fd2ec5fe4"
+					(reference "J4")
+					(unit 1)
+				)
