File: tolt/conn.kicad_sch (KiCad schematic)
At the start: 56 parts, among them J1 Conn_01x05, J10 Conn_01x03, J2 USB_C_Receptacle_USB2.0, J3 Conn_01x06, J4 Conn_01x05, J5 Conn_01x03, J6 Conn_01x03, J7 Conn_01x05, J8 Conn_01x02, J9 Conn_01x03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

Commit message: modified:   tolt/conn.kicad_sch 	modified:   tolt/tolt.kicad_pcb 	modified:   tolt/tolt.kicad_pro
Parts:
- removed J1: Conn_01x05, Connector_PinSocket_2.54mm:PinSocket_2x03_P2.54mm_Vertical, symbol Connector_Generic:Conn_01x06
- added J1: Conn_01x05, Connector_JST:JST_PH_B5B-PH-K_1x05_P2.00mm_Vertical, symbol Connector_Generic:Conn_01x05
Connections:
- net +5V: now also J1.5 (Pin_5)
- net GND: now also J1.1 (Pin_1)
- net SWCLK: now also J1.2 (Pin_2)
- net SWDIO: now also J1.3 (Pin_3)
- net rst: now also J1.4 (Pin_4)
- no-connect marks 4 -> 3
Changed lines of the file:
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@@
 	)
 	(junction
+		(at 243.586 74.676)
+		(diameter 0)
+		(color 0 0 0 0)
+	)
+	(junction
 		(at 208.534 41.148)
 		(diameter 0)
@@
 	)
 	(junction
-		(at 177.546 106.934)
+		(at 243.84 84.836)
 		(diameter 0)
 		(color 0 0 0 0)
 	)
 	(junction
-		(at 162.052 84.836)
+		(at 177.546 106.934)
 		(diameter 0)
 		(color 0 0 0 0)
 	)
 	(junction
-		(at 91.186 159.004)
+		(at 162.052 84.836)
 		(diameter 0)
 		(color 0 0 0 0)
 	)
 	(junction
-		(at 243.586 74.676)
+		(at 91.186 159.004)
 		(diameter 0)
 		(color 0 0 0 0)
@@
 	)
 	(junction
-		(at 243.84 84.836)
-		(diameter 0)
-		(color 0 0 0 0)
-	)
-	(junction
 		(at 107.442 46.482)
 		(diameter 0)
@@
 	)
 	(no_connect
-		(at 243.84 87.376)
-	)
-	(no_connect
 		(at 198.374 88.646)
 	)
@@
 	(wire
 		(pts
-			(xy 243.586 79.756) (xy 243.84 79.756)
-		)
-		(stroke
-			(width 0)
-			(type default)
-		)
-	)
-	(wire
-		(pts
 			(xy 122.682 38.862) (xy 132.842 38.862)
 		)
@@
 	(wire
 		(pts
-			(xy 244.094 84.836) (xy 243.84 84.836)
-		)
-		(stroke
-			(width 0)
-			(type default)
-		)
-	)
-	(wire
-		(pts
 			(xy 265.176 159.258) (xy 252.476 159.258)
 		)
@@
 	(wire
 		(pts
-			(xy 243.586 77.216) (xy 243.84 77.216)
+			(xy 267.208 83.058) (xy 244.094 83.058)
 		)
 		(stroke
@@
 	(wire
 		(pts
-			(xy 267.208 83.058) (xy 244.094 83.058)
+			(xy 222.758 48.768) (xy 222.758 47.498)
 		)
 		(stroke
@@
 	(wire
 		(pts
-			(xy 222.758 48.768) (xy 222.758 47.498)
+			(xy 243.586 74.676) (xy 243.84 74.676)
 		)
 		(stroke
@@
 	(wire
 		(pts
-			(xy 243.586 74.676) (xy 243.84 74.676)
-		)
-		(stroke
-			(width 0)
-			(type default)
-		)
-	)
-	(wire
-		(pts
 			(xy 232.156 140.462) (xy 233.934 140.462)
 		)
@@
 	(wire
 		(pts
-			(xy 243.586 82.296) (xy 243.84 82.296)
-		)
-		(stroke
-			(width 0)
-			(type default)
-		)
-	)
-	(wire
-		(pts
 			(xy 111.252 145.542) (xy 114.3 145.542)
 		)
@@
 	(wire
 		(pts
+			(xy 243.84 84.836) (xy 244.094 84.836)
+		)
+		(stroke
+			(width 0)
+			(type default)
+		)
+	)
+	(wire
+		(pts
 			(xy 151.638 109.474) (xy 140.208 109.474)
 		)
@@
 	(hierarchical_label "SWCLK"
 		(shape output)
-		(at 243.586 77.216 180)
+		(at 243.84 77.216 180)
 		(effects
 			(font
@@
 	(hierarchical_label "SWDIO"
 		(shape bidirectional)
-		(at 243.586 79.756 180)
+		(at 243.84 79.756 180)
 		(effects
 			(font
@@
 	(hierarchical_label "rst"
 		(shape output)
-		(at 243.586 82.296 180)
+		(at 243.84 82.296 180)
 		(effects
 			(font
@@
 	)
 	(symbol
+		(lib_id "Connector_Generic:Conn_01x05")
+		(at 248.92 79.756 0)
+		(unit 1)
+		(exclude_from_sim no)
+		(in_bom yes)
+		(on_board yes)
+		(dnp no)
+		(fields_autoplaced yes)
+		(property "Reference" "J1"
+			(at 251.968 78.4859 0)
+			(effects
+				(font
+					(size 1.27 1.27)
+				)
+				(justify left)
+			)
+		)
+		(property "Value" "Conn_01x05"
+			(at 251.968 81.0259 0)
+			(effects
+				(font
+					(size 1.27 1.27)
+				)
+				(justify left)
+			)
+		)
+		(property "Footprint" "Connector_JST:JST_PH_B5B-PH-K_1x05_P2.00mm_Vertical"
+			(at 248.92 79.756 0)
+			(effects
+				(font
+					(size 1.27 1.27)
+				)
+				(hide yes)
+			)
+		)
+		(property "Datasheet" "~"
+			(at 248.92 79.756 0)
+			(effects
+				(font
+					(size 1.27 1.27)
+				)
+				(hide yes)
+			)
+		)
+		(property "Description" "Generic connector, single row, 01x05, script generated (kicad-library-utils/schlib/autogen/connector/)"
+			(at 248.92 79.756 0)
+			(effects
+				(font
+					(size 1.27 1.27)
+				)
+				(hide yes)
+			)
+		)
+		(pin "1"
+		)
+		(pin "3"
+		)
+		(pin "2"
+		)
+		(pin "5"
+		)
+		(pin "4"
+		)
+		(instances
+			(project "tolt"
+				(path "/38c63d96-01d7-4159-b7c0-aa8cee77c3e9/4189330a-b7ac-4caa-ad9c-153fd2ec5fe4"
+					(reference "J1")
+					(unit 1)
+				)
+			)
+		)
+	)
+	(symbol
 		(lib_id "Simulation_SPICE:NMOS")
 		(at 154.178 121.666 180)
@@
 					(unit 1)
 				)
-			)
-		)
-	)
-	(symbol
-		(lib_id "Connector_Generic:Conn_01x06")
-		(at 248.92 79.756 0)
-		(unit 1)
-		(exclude_from_sim no)
-		(in_bom yes)
-		(on_board yes)
-		(dnp no)
-		(fields_autoplaced yes)
-		(property "Reference" "J1"
-			(at 251.46 79.7559 0)
-			(effects
-				(font
-					(size 1.27 1.27)
-				)
-				(justify left)
-			)
-		)
-		(property "Value" "Conn_01x05"
-			(at 251.46 82.2959 0)
-			(effects
-				(font
-					(size 1.27 1.27)
-				)
-				(justify left)
-			)
-		)
-		(property "Footprint" "Connector_PinSocket_2.54mm:PinSocket_2x03_P2.54mm_Vertical"
-			(at 248.92 79.756 0)
-			(effects
-				(font
-					(size 1.27 1.27)
-				)
-				(hide yes)
-			)
-		)
-		(property "Datasheet" "~"
-			(at 248.92 79.756 0)
-			(effects
-				(font
-					(size 1.27 1.27)
-				)
-				(hide yes)
-			)
-		)
-		(property "Description" "Generic connector, single row, 01x06, script generated (kicad-library-utils/schlib/autogen/connector/)"
-			(at 248.92 79.756 0)
-			(effects
-				(font
-					(size 1.27 1.27)
-				)
-				(hide yes)
-			)
-		)
-		(pin "2"
-		)
-		(pin "4"
-		)
-		(pin "5"
-		)
-		(pin "1"
-		)
-		(pin "3"
-		)
-		(pin "6"
-		)
-		(instances
-			(project ""
-				(path "/38c63d96-01d7-4159-b7c0-aa8cee77c3e9/4189330a-b7ac-4caa-ad9c-153fd2ec5fe4"
-					(reference "J1")
-					(unit 1)
-				)
