File: tolt/conn.kicad_sch (KiCad schematic)
At the start: 56 parts, among them J1 Conn_01x05, J10 Conn_01x03, J2 USB_C_Receptacle_USB2.0, J3 Conn_01x06, J4 Conn_01x05, J5 Conn_01x03, J6 Conn_01x03, J7 Conn_01x05, J8 Conn_01x02, J9 Conn_01x03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

Commit message: modified:   tolt/conn.kicad_sch 	modified:   tolt/powerstage.kicad_sch 	modified:   tolt/stm32.kicad_sch 	modified:   tolt/tolt.kicad_pcb 	modified:   tolt/tolt.kicad_pro 	modified:   tolt/tolt.kicad_sch
Connections:
- net +12V: now also J10.2 (Pin_2); no longer J10.3 (Pin_3)
- net at D28.2 (A), Q19.3 (S): now also J10.3 (Pin_3); no longer J10.2 (Pin_2)
Changed lines of the file:
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@@
+	)
+	(junction
+		(at 161.544 121.666)
+		(diameter 0)
+		(color 0 0 0 0)
+	)
+	(junction
+		(at 162.052 77.216)
+		(diameter 0)
+		(color 0 0 0 0)
 	)
 	(junction
 		(at 158.75 106.934)
-		(diameter 0)
-		(color 0 0 0 0)
-	)
-	(junction
-		(at 161.544 121.666)
-		(diameter 0)
-		(color 0 0 0 0)
-	)
-	(junction
-		(at 162.052 77.216)
 		(diameter 0)
 		(color 0 0 0 0)
@@
 	(wire
 		(pts
-			(xy 151.638 115.316) (xy 151.638 109.474)
+			(xy 151.638 115.316) (xy 151.638 106.934)
 		)
 		(stroke
@@
 	(wire
 		(pts
+			(xy 158.75 109.474) (xy 158.75 106.934)
+		)
+		(stroke
+			(width 0)
+			(type default)
+		)
+	)
+	(wire
+		(pts
 			(xy 115.316 62.738) (xy 115.316 59.436)
 		)
@@
 	(wire
 		(pts
-			(xy 140.208 106.934) (xy 158.75 106.934)
-		)
-		(stroke
-			(width 0)
-			(type default)
-		)
-	)
-	(wire
-		(pts
 			(xy 99.314 62.738) (xy 99.314 59.436)
 		)
@@
 	(wire
 		(pts
-			(xy 151.638 109.474) (xy 140.208 109.474)
+			(xy 140.208 106.934) (xy 151.638 106.934)
 		)
 		(stroke
@@
 		)
 		(stroke
+			(width 0)
+			(type default)
+		)
+	)
+	(wire
+		(pts
+			(xy 140.208 109.474) (xy 158.75 109.474)
+		)
+		(stroke

Commit message: move comp
Parts:
- added J11: Conn_01x02, Connector_JST:JST_XH_B2B-XH-A_1x02_P2.50mm_Vertical, symbol Connector_Generic:Conn_01x02
- J1: footprint Connector_JST:JST_PH_B5B-PH-K_1x05_P2.00mm_Vertical -> Connector_PinSocket_2.00mm:PinSocket_1x05_P2.00mm_Vertical
- Q19: footprint Package_TO_SOT_SMD:SOT-23_Handsoldering -> Package_TO_SOT_SMD:SOT-23
Connections:
- net +12V: now also J11.2 (Pin_2)
- net GND: now also J11.1 (Pin_1)
Changed lines of the file:
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@@
 	)
 	(symbol
+		(lib_id "power:+12V")
+		(at 155.956 152.908 270)
+		(unit 1)
+		(exclude_from_sim no)
+		(in_bom yes)
+		(on_board yes)
+		(dnp no)
+		(fields_autoplaced yes)
+		(property "Reference" "#PWR055"
+			(at 152.146 152.908 0)
+			(effects
+				(font
+					(size 1.27 1.27)
+				)
+				(hide yes)
+			)
+		)
+		(property "Value" "+12V"
+			(at 160.02 152.9079 90)
+			(effects
+				(font
+					(size 1.27 1.27)
+				)
+				(justify left)
+			)
+		)
+		(property "Footprint" ""
+			(at 155.956 152.908 0)
+			(effects
+				(font
+					(size 1.27 1.27)
+				)
+				(hide yes)
+			)
+		)
+		(property "Datasheet" ""
+			(at 155.956 152.908 0)
+			(effects
+				(font
+					(size 1.27 1.27)
+				)
+				(hide yes)
+			)
+		)
+		(property "Description" "Power symbol creates a global label with name \"+12V\""
+			(at 155.956 152.908 0)
+			(effects
+				(font
+					(size 1.27 1.27)
+				)
+				(hide yes)
+			)
+		)
+		(pin "1"
+		)
+		(instances
+			(project ""
+				(path "/38c63d96-01d7-4159-b7c0-aa8cee77c3e9/4189330a-b7ac-4caa-ad9c-153fd2ec5fe4"
+					(reference "#PWR055")
+					(unit 1)
+				)
+			)
+		)
+	)
+	(symbol
 		(lib_id "power:+5V")
 		(at 252.476 151.638 0)
@@
 	)
 	(symbol
+		(lib_id "Connector_Generic:Conn_01x02")
+		(at 150.876 155.448 180)
+		(unit 1)
+		(exclude_from_sim no)
+		(in_bom yes)
+		(on_board yes)
+		(dnp no)
+		(fields_autoplaced yes)
+		(property "Reference" "J11"
+			(at 150.876 146.05 0)
+			(effects
+				(font
+					(size 1.27 1.27)
+				)
+			)
+		)
+		(property "Value" "Conn_01x02"
+			(at 150.876 148.59 0)
+			(effects
+				(font
+					(size 1.27 1.27)
+				)
+			)
+		)
+		(property "Footprint" "Connector_JST:JST_XH_B2B-XH-A_1x02_P2.50mm_Vertical"
+			(at 150.876 155.448 0)
+			(effects
+				(font
+					(size 1.27 1.27)
+				)
+				(hide yes)
+			)
+		)
+		(property "Datasheet" "~"
+			(at 150.876 155.448 0)
+			(effects
+				(font
+					(size 1.27 1.27)
+				)
+				(hide yes)
+			)
+		)
+		(property "Description" "Generic connector, single row, 01x02, script generated (kicad-library-utils/schlib/autogen/connector/)"
+			(at 150.876 155.448 0)
+			(effects
+				(font
+					(size 1.27 1.27)
+				)
+				(hide yes)
+			)
+		)
+		(pin "2"
+		)
+		(pin "1"
+		)
+		(instances
+			(project ""
+				(path "/38c63d96-01d7-4159-b7c0-aa8cee77c3e9/4189330a-b7ac-4caa-ad9c-153fd2ec5fe4"
+					(reference "J11")
+					(unit 1)
+				)
+			)
+		)
+	)
+	(symbol
 		(lib_id "power:GND")
 		(at 233.68 126.238 0)
@@
 			)
 		)
-		(property "Footprint" "Connector_JST:JST_PH_B5B-PH-K_1x05_P2.00mm_Vertical"
+		(property "Footprint" "Connector_PinSocket_2.00mm:PinSocket_1x05_P2.00mm_Vertical"
 			(at 248.92 79.756 0)
 			(effects
@@
 			)
 		)
-		(property "Footprint" "Package_TO_SOT_SMD:SOT-23_Handsoldering"
+		(property "Footprint" "Package_TO_SOT_SMD:SOT-23"
 			(at 149.098 124.206 0)
 			(effects
@@
 					(unit 1)
 				)
+			)
+		)
+	)
+	(symbol
+		(lib_name "GND_1")
+		(lib_id "power:GND")
+		(at 155.956 155.448 90)
+		(unit 1)
+		(exclude_from_sim no)
+		(in_bom yes)
+		(on_board yes)
+		(dnp no)
+		(fields_autoplaced yes)
+		(property "Reference" "#PWR056"
+			(at 162.306 155.448 0)
+			(effects
+				(font
+					(size 1.27 1.27)
+				)
+				(hide yes)
+			)
+		)
+		(property "Value" "GND"
+			(at 160.02 155.4479 90)
+			(effects
+				(font
+					(size 1.27 1.27)
+				)
+				(justify right)
+			)
+		)
+		(property "Footprint" ""
+			(at 155.956 155.448 0)
+			(effects
+				(font
+					(size 1.27 1.27)
+				)
+				(hide yes)
+			)
+		)
+		(property "Datasheet" ""
+			(at 155.956 155.448 0)
+			(effects
+				(font
+					(size 1.27 1.27)
+				)
+				(hide yes)
+			)
+		)
+		(property "Description" "Power symbol creates a global label with name \"GND\" , ground"
+			(at 155.956 155.448 0)
+			(effects
+				(font
+					(size 1.27 1.27)
+				)
+				(hide yes)
+			)
+		)
+		(pin "1"
+		)
+		(instances
+			(project ""
+				(path "/38c63d96-01d7-4159-b7c0-aa8cee77c3e9/4189330a-b7ac-4caa-ad9c-153fd2ec5fe4"
+					(reference "#PWR056")
+					(unit 1)
+				)

Commit message: .
Parts:
- added J12: USB_C_Receptacle_USB2.0, Connector_USB:USB_C_Receptacle_G-Switch_GT-USB-7051x, symbol Connector:USB_C_Receptacle_USB2.0
- added JP5: Jumper_2_Open, Jumper:SolderJumper-2_P1.3mm_Open_RoundedPad1.0x1.5mm, symbol Jumper:Jumper_2_Open
- added R96, R97: 5k1, Resistor_SMD:R_0603_1608Metric, symbol Device:R
- J1: value Conn_01x05 -> Conn_01x06; footprint Connector_PinSocket_2.00mm:PinSocket_1x05_P2.00mm_Vertical -> Connector_PinSocket_2.00mm:PinSocket_2x03_P2.00mm_Vertical; symbol Connector_Generic:Conn_01x05 -> Connector_Generic:Conn_02x03_Odd_Even
Connections:
- net +5V: now also J1.4 (Pin_4), JP5.2 (B); no longer J1.5 (Pin_5)
- net Canh: now also U22.6 (IO4); no longer U22.4 (IO3)
- net Canl: now also U22.4 (IO3); no longer U22.6 (IO4)
- net GND: now also J1.2 (Pin_2), J12.A1 (GND), J12.A12 (GND), J12.B1 (GND), J12.B12 (GND), J12.S1 (SHIELD), R96.1, R97.1; no longer J1.1 (Pin_1)
- net SWCLK: now also J1.1 (Pin_1); no longer J1.2 (Pin_2)
- net rst: now also J1.5 (Pin_5); no longer J1.4 (Pin_4)
- new net: J12.A4 (VBUS), J12.A9 (VBUS), J12.B4 (VBUS), J12.B9 (VBUS), JP5.1 (A)
- new net: J12.B5 (CC2), R97.2
- new net: J12.A5 (CC1), R96.2
- new net ESP_D+: J12.A6 (D+), J12.B6 (D+)
- new net ESP_D-: J12.A7 (D-), J12.B7 (D-)
- no-connect marks 3 -> 6
Other:
- moved on the sheet: C116, C117, C87, J11, J9, R98

Commit message: FINAL
Parts:
- removed J11: Conn_01x02, Connector_JST:JST_XH_B2B-XH-A_1x02_P2.50mm_Vertical, symbol Connector_Generic:Conn_01x02
- C116, C118, C120, C122, C123, C125, C127, C80, C82, C87: LCSC (none) -> C60474
- C117, C119, C121, C124, C126: LCSC (none) -> C55151
- C81, C91: LCSC (none) -> C98192
- C88: LCSC (none) -> C138687
- D28: LCSC (none) -> C114696
- J1: value Conn_01x06 -> Conn_01x05
- J12, J2: LCSC (none) -> C2843970
- Q19: LCSC (none) -> C19019
- R100, R101, R102, R73, R74, R75, R79, R81: LCSC (none) -> C114662
- R26, R84, R96, R97: LCSC (none) -> C2907114
- R72, R99: LCSC (none) -> C25804
- R76, R77, R78, R80, R82: LCSC (none) -> C2930099
- R83: LCSC (none) -> C114640
- R98: LCSC (none) -> C105588
- U20: LCSC (none) -> C38695
- U21, U22, U23: LCSC (none) -> C151305

Commit message: fixes
to be reviewed furthermore
Parts:
- J12, J2: footprint Connector_USB:USB_C_Receptacle_G-Switch_GT-USB-7051x -> Connector_USB:USB_C_Receptacle_G-Switch_GT-USB-7010ASV
Changed lines of the file:
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@@
 			)
 		)
-		(property "Footprint" "Connector_USB:USB_C_Receptacle_G-Switch_GT-USB-7051x"
+		(property "Footprint" "Connector_USB:USB_C_Receptacle_G-Switch_GT-USB-7010ASV"
 			(at 144.78 163.83 0)
 			(effects
@@
 			)
 		)
-		(property "Footprint" "Connector_USB:USB_C_Receptacle_G-Switch_GT-USB-7051x"
+		(property "Footprint" "Connector_USB:USB_C_Receptacle_G-Switch_GT-USB-7010ASV"
 			(at 48.514 142.494 0)
 			(effects
