File: tolt/conn.kicad_sch (KiCad schematic)
At the start: 56 parts, among them J1 Conn_01x05, J10 Conn_01x03, J2 USB_C_Receptacle_USB2.0, J3 Conn_01x06, J4 Conn_01x05, J5 Conn_01x03, J6 Conn_01x03, J7 Conn_01x05, J8 Conn_01x02, J9 Conn_01x03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

Commit message: usb conn
changed usb conn to flat
Parts:
- J2: footprint Connector_USB:USB_C_Receptacle_G-Switch_GT-USB-7051x -> Connector_USB:USB_C_Receptacle_G-Switch_GT-USB-7010ASV
Changed lines of the file:
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@@
 			)
 		)
-		(property "Footprint" "Connector_USB:USB_C_Receptacle_G-Switch_GT-USB-7051x"
+		(property "Footprint" "Connector_USB:USB_C_Receptacle_G-Switch_GT-USB-7010ASV"
 			(at 48.514 142.494 0)
 			(effects

Commit message: begenning of lcsc part assign
Parts:
- C88: LCSC (none) -> C138687
- Q19: footprint Package_TO_SOT_SMD:SOT-23_Handsoldering -> Package_TO_SOT_SMD:SOT-23
- R72, R99: LCSC (none) -> C25804
Changed lines of the file:
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@@
 			)
 		)
+		(property "LCSC" "C25804"
+			(at 124.46 26.924 0)
+			(effects
+				(font
+					(size 1.27 1.27)
+				)
+				(hide yes)
+			)
+		)
 		(pin "1"
 		)
@@
 			)
 		)
+		(property "LCSC" "C25804"
+			(at 161.544 125.476 0)
+			(effects
+				(font
+					(size 1.27 1.27)
+				)
+				(hide yes)
+			)
+		)
 		(pin "1"
 		)
@@
 			)
 		)
-		(property "Footprint" "Package_TO_SOT_SMD:SOT-23_Handsoldering"
+		(property "Footprint" "Package_TO_SOT_SMD:SOT-23"
 			(at 149.098 124.206 0)
 			(effects
@@
 			(at 177.546 110.744 0)
 			(effects
+				(font
+					(size 1.27 1.27)
+				)
+				(hide yes)
+			)
+		)
+		(property "LCSC" "C138687"
+			(at 177.546 110.744 0)
+			(effects

Commit message: more assign+12-5v change
changed with TPS82130
Since using esp32 will increase consumption by a lot
Parts:
- R100, R101, R102, R73, R74, R75, R79, R81: LCSC (none) -> C114662
- R26, R84: LCSC (none) -> C2907114
- R76, R77, R78, R80, R82: LCSC (none) -> C2930099
Changed lines of the file:
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@@
 			)
 		)
+		(property "LCSC" "C114662"
+			(at 99.314 35.306 0)
+			(effects
+				(font
+					(size 1.27 1.27)
+				)
+				(hide yes)
+			)
+		)
 		(pin "1"
 		)
@@
 			)
 		)
+		(property "LCSC" "C2930099"
+			(at 233.934 151.892 0)
+			(effects
+				(font
+					(size 1.27 1.27)
+				)
+				(hide yes)
+			)
+		)
 		(pin "1"
 		)
@@
 			)
 		)
+		(property "LCSC" "C2907114"
+			(at 63.754 132.334 90)
+			(effects
+				(font
+					(size 1.27 1.27)
+				)
+				(hide yes)
+			)
+		)
 		(pin "1"
 		)
@@
 			)
 		)
+		(property "LCSC" "C114662"
+			(at 233.68 114.808 0)
+			(effects
+				(font
+					(size 1.27 1.27)
+				)
+				(hide yes)
+			)
+		)
 		(pin "1"
 		)
@@
 			)
 		)
+		(property "LCSC" "C114662"
+			(at 115.316 35.306 0)
+			(effects
+				(font
+					(size 1.27 1.27)
+				)
+				(hide yes)
+			)
+		)
 		(pin "1"
 		)
@@
 			)
 		)
+		(property "LCSC" "C2907114"
+			(at 63.754 134.874 90)
+			(effects
+				(font
+					(size 1.27 1.27)
+				)
+				(hide yes)
+			)
+		)
 		(pin "1"
 		)
@@
 			)
 		)
+		(property "LCSC" "C114662"
+			(at 107.442 35.306 0)
+			(effects
+				(font
+					(size 1.27 1.27)
+				)
+				(hide yes)
+			)
+		)
 		(pin "1"
 		)
@@
 			)
 		)
+		(property "LCSC" "C2930099"
+			(at 233.68 122.428 0)
+			(effects
+				(font
+					(size 1.27 1.27)
+				)
+				(hide yes)
+			)
+		)
 		(pin "1"
 		)
@@
 			)
 		)
+		(property "LCSC" "C2930099"
+			(at 107.442 66.548 0)
+			(effects
+				(font
+					(size 1.27 1.27)
+				)
+				(hide yes)
+			)
+		)
 		(pin "1"
 		)
@@
 			)
 		)
+		(property "LCSC" "C114662"
+			(at 107.442 55.626 0)
+			(effects
+				(font
+					(size 1.27 1.27)
+				)
+				(hide yes)
+			)
+		)
 		(pin "1"
 		)
@@
 			)
 		)
+		(property "LCSC" "C2930099"
+			(at 115.316 66.548 0)
+			(effects
+				(font
+					(size 1.27 1.27)
+				)
+				(hide yes)
+			)
+		)
 		(pin "1"
 		)
@@
 			)
 		)
+		(property "LCSC" "C2930099"
+			(at 99.314 66.548 0)
+			(effects
+				(font
+					(size 1.27 1.27)
+				)
+				(hide yes)
+			)
+		)
 		(pin "1"
 		)
@@
 			)
 		)
+		(property "LCSC" "C114662"
+			(at 233.934 144.272 0)
+			(effects
+				(font
+					(size 1.27 1.27)
+				)
+				(hide yes)
+			)
+		)
 		(pin "1"
 		)
@@
 			)
 		)
+		(property "LCSC" "C114662"
+			(at 99.314 55.626 0)
+			(effects
+				(font
+					(size 1.27 1.27)
+				)
+				(hide yes)
+			)
+		)
 		(pin "1"
 		)
@@
 			(at 115.316 55.626 0)
 			(effects
+				(font
+					(size 1.27 1.27)
+				)
+				(hide yes)
+			)
+		)
+		(property "LCSC" "C114662"
+			(at 115.316 55.626 0)
+			(effects

Commit message: hm
weird huh it didnt fucking save
Parts:
- C116, C118, C120, C122, C123, C125, C127: LCSC (none) -> C24497
- C117, C119, C121, C124, C126: LCSC (none) -> C913904
- C80, C82, C87: LCSC (none) -> C60474
- C81, C91: LCSC (none) -> C98192
- D28: LCSC (none) -> C114696
- J1, J4, J7: LCSC (none) -> C265085
- J10, J5, J6, J9: LCSC (none) -> C160353
- J2: LCSC (none) -> C2843970
- J3: LCSC (none) -> C471518
- J8: LCSC (none) -> C265372
- Q19: LCSC (none) -> C19019

Commit message: Done
hopefully finished ?
needs sanity check and more checks
Parts:
- R83: LCSC (none) -> C114640
- R98: LCSC (none) -> C105588
- U20: LCSC (none) -> C38695
- U21, U22, U23: LCSC (none) -> C151305
Changed lines of the file:
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@@
 			)
 		)
+		(property "LCSC" "C114640"
+			(at 208.534 44.958 0)
+			(effects
+				(font
+					(size 1.27 1.27)
+				)
+				(hide yes)
+			)
+		)
 		(pin "1"
 		)
@@
 			)
 		)
+		(property "LCSC" "C151305"
+			(at 45.212 91.44 0)
+			(effects
+				(font
+					(size 1.27 1.27)
+				)
+				(hide yes)
+			)
+		)
 		(pin "6"
 		)
@@
 			)
 		)
+		(property "LCSC" "C151305"
+			(at 94.488 91.44 0)
+			(effects
+				(font
+					(size 1.27 1.27)
+				)
+				(hide yes)
+			)
+		)
 		(pin "6"
 		)
@@
 			)
 		)
+		(property "LCSC" "C105588"
+			(at 107.442 145.542 90)
+			(effects
+				(font
+					(size 1.27 1.27)
+				)
+				(hide yes)
+			)
+		)
 		(pin "1"
 		)
@@
 			)
 		)
+		(property "LCSC" "C151305"
+			(at 45.466 49.53 0)
+			(effects
+				(font
+					(size 1.27 1.27)
+				)
+				(hide yes)
+			)
+		)
 		(pin "6"
 		)
@@
 			(at 188.976 44.958 0)
 			(effects
+				(font
+					(size 1.27 1.27)
+				)
+				(hide yes)
+			)
+		)
+		(property "LCSC" "C38695"
+			(at 188.976 44.958 0)
+			(effects

Commit message: fab
finally.
Parts:
- C117, C119, C121, C124, C126: LCSC C913904 -> C326565
Changed lines of the file:
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@@
 			)
 		)
-		(property "LCSC" "C913904"
+		(property "LCSC" "C326565"
 			(at 103.886 162.814 0)
 			(effects
@@
 			)
 		)
-		(property "LCSC" "C913904"
+		(property "LCSC" "C326565"
 			(at 244.856 62.23 0)
 			(effects
@@
 			)
 		)
-		(property "LCSC" "C913904"
+		(property "LCSC" "C326565"
 			(at 265.176 123.698 0)
 			(effects
@@
 			)
 		)
-		(property "LCSC" "C913904"
+		(property "LCSC" "C326565"
 			(at 265.176 155.448 0)
 			(effects
@@
 			)
 		)
-		(property "LCSC" "C913904"
+		(property "LCSC" "C326565"
 			(at 174.752 81.026 0)
 			(effects
