File: tolt/stm32.kicad_sch (KiCad schematic)
At the start: 53 parts, among them J14 BOOT0, J15 NRST, U1 STM32F405RGTx, U10 MC74VHC1GT66, U11 MC74VHC1GT66, U12 MC74VHC1GT66, U13 MC74VHC1GT66, U5 INA240/241, U6 MC74VHC1GT66, U8 MC74VHC1GT66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

Commit message: modified:   tolt/conn.kicad_sch 	modified:   tolt/converters.kicad_sch 	modified:   tolt/inter.kicad_sch 	modified:   tolt/powerstage.kicad_sch 	modified:   tolt/stm32.kicad_sch 	modified:   tolt/tolt.kicad_pcb 	modified:   tolt/tolt.kicad_pro
Parts:
- R33, R34, R35, R38, R39: footprint Resistor_SMD:R_0603_1608Metric_Pad0.98x0.95mm_HandSolder -> Resistor_SMD:R_0603_1608Metric
Changed lines of the file:
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@@
 			)
 		)
-		(property "Footprint" "Resistor_SMD:R_0603_1608Metric_Pad0.98x0.95mm_HandSolder"
+		(property "Footprint" "Resistor_SMD:R_0603_1608Metric"
 			(at 248.92 38.608 90)
 			(effects
@@
 			)
 		)
-		(property "Footprint" "Resistor_SMD:R_0603_1608Metric_Pad0.98x0.95mm_HandSolder"
+		(property "Footprint" "Resistor_SMD:R_0603_1608Metric"
 			(at 251.46 88.9 90)
 			(effects
@@
 			)
 		)
-		(property "Footprint" "Resistor_SMD:R_0603_1608Metric_Pad0.98x0.95mm_HandSolder"
+		(property "Footprint" "Resistor_SMD:R_0603_1608Metric"
 			(at 69.85 57.15 0)
 			(effects
@@
 			)
 		)
-		(property "Footprint" "Resistor_SMD:R_0603_1608Metric_Pad0.98x0.95mm_HandSolder"
+		(property "Footprint" "Resistor_SMD:R_0603_1608Metric"
 			(at 47.752 62.23 0)
 			(effects
@@
 			)
 		)
-		(property "Footprint" "Resistor_SMD:R_0603_1608Metric_Pad0.98x0.95mm_HandSolder"
+		(property "Footprint" "Resistor_SMD:R_0603_1608Metric"
 			(at 250.698 140.208 90)
 			(effects

Commit message: aa
Connections:
- net GND: now also U8.3 (GND)
Changed lines of the file:
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@@
+	(symbol
+		(lib_id "power:GND")
+		(at 226.314 147.828 0)
+		(unit 1)
+		(exclude_from_sim no)
+		(in_bom yes)
+		(on_board yes)
+		(dnp no)
+		(fields_autoplaced yes)
+		(property "Reference" "#PWR0299"
+			(at 226.314 154.178 0)
+			(effects
+				(font
+					(size 1.27 1.27)
+				)
+				(hide yes)
+			)
+		)
+		(property "Value" "GND"
+			(at 226.314 152.908 0)
+			(effects
+				(font
+					(size 1.27 1.27)
+				)
+			)
+		)
+		(property "Footprint" ""
+			(at 226.314 147.828 0)
+			(effects
+				(font
+					(size 1.27 1.27)
+				)
+				(hide yes)
+			)
+		)
+		(property "Datasheet" ""
+			(at 226.314 147.828 0)
+			(effects
+				(font
+					(size 1.27 1.27)
+				)
+				(hide yes)
+			)
+		)
+		(property "Description" ""
+			(at 226.314 147.828 0)
+			(effects
+				(font
+					(size 1.27 1.27)
+				)
+				(hide yes)
+			)
+		)
+		(pin "1"
+		)
+		(instances
+			(project "tolt"
+				(path "/38c63d96-01d7-4159-b7c0-aa8cee77c3e9/410a2c08-a3a0-4066-ae14-a5c75baf28bb"
+					(reference "#PWR0299")
+					(unit 1)
+				)
+			)
+		)
+	)
 	(symbol
 		(lib_id "power:GND")

Commit message: modified:   tolt/conn.kicad_sch 	modified:   tolt/powerstage.kicad_sch 	modified:   tolt/stm32.kicad_sch 	modified:   tolt/tolt.kicad_pcb 	modified:   tolt/tolt.kicad_pro 	modified:   tolt/tolt.kicad_sch
Connections:
- net NRF_swclk is gone; now on net scl_bmi: U1.55 (PB3)
- net HALL_1: now also U1.4 (PC15); no longer U1.37 (PC6)
- net HALL_2: now also U1.3 (PC14); no longer U1.38 (PC7)
- net HALL_3: now also U1.2 (PC13); no longer U1.39 (PC8)
- net scl_bmi: no longer U1.33 (PB12)
- net NRF_swdio: no longer names the net of U1.50 (PA15)
- no-connect marks 7 -> 8
Other:
- note added: "Halls from gpio c 6-7-8 to 13-14-15"
Changed lines of the file:
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@@
+		)
+	)
+	(text "Halls from gpio c 6-7-8 to 13-14-15"
+		(exclude_from_sim no)
+		(at 50.546 105.156 0)
+		(effects
+			(font
+				(size 1.27 1.27)
+			)
 		)
 	)
@@
 	)
 	(no_connect
+		(at 109.474 138.684)
+	)
+	(no_connect
+		(at 73.914 108.204)
+	)
+	(no_connect
+		(at 73.914 103.124)
+	)
+	(no_connect
 		(at 269.24 45.72)
 	)
@@
 	)
 	(no_connect
-		(at 73.914 125.984)
+		(at 109.474 113.284)
 	)
 	(no_connect
-		(at 109.474 113.284)
-	)
-	(no_connect
-		(at 73.914 120.904)
-	)
-	(no_connect
-		(at 73.914 123.444)
+		(at 73.914 105.664)
 	)
 	(wire
@@
 	(hierarchical_label "HALL_2"
 		(shape input)
-		(at 73.914 105.664 180)
+		(at 73.914 123.444 180)
 		(effects
 			(font
@@
 	(hierarchical_label "scl_bmi"
 		(shape bidirectional)
-		(at 109.474 138.684 0)
+		(at 109.474 115.824 0)
 		(effects
 			(font
@@
 		(shape output)
 		(at 109.474 90.424 0)
-		(effects
-			(font
-				(size 1.27 1.27)
-			)
-			(justify left)
-		)
-	)
-	(hierarchical_label "NRF_swclk"
-		(shape output)
-		(at 109.474 115.824 0)
 		(effects
 			(font
@@
 	(hierarchical_label "HALL_3"
 		(shape input)
-		(at 73.914 108.204 180)
+		(at 73.914 120.904 180)
 		(effects
 			(font
@@
 		(shape output)
 		(at 109.474 125.984 0)
-		(effects
-			(font
-				(size 1.27 1.27)
-			)
-			(justify left)
-		)
-	)
-	(hierarchical_label "NRF_swdio"
-		(shape bidirectional)
-		(at 109.474 103.124 0)
 		(effects
 			(font
@@
 	(hierarchical_label "HALL_1"
 		(shape input)
-		(at 73.914 103.124 180)
-		(effects
-			(font
+		(at 73.914 125.984 180)
+		(effects
+			(font

Commit message: modified:   tolt/conn.kicad_sch 	modified:   tolt/powerstage.kicad_sch 	modified:   tolt/stm32.kicad_sch 	modified:   tolt/tolt.kicad_pcb 	modified:   tolt/tolt.kicad_pro 	modified:   tolt/tolt.kicad_sch
Connections:
- net CURRENT_1: now also C40.1, R35.2, U8.1; no longer C30.1, R33.2, U10.1
- net CURRENT_3: now also C30.1, R33.2, U10.1; no longer C40.1, R35.2, U8.1
- net SENS_A+ renamed SENS_C_P
- net SENS_A- renamed SENS_C_N
- net SENS_B+ renamed SENS_B_P
- net SENS_B- renamed SENS_B_N
- net SENS_C+ renamed SENS_A_P
- net SENS_C- renamed SENS_A_N
Other:
- moved on the sheet: C29, C30, C40, C41, R33, R35, U10, U5, U8, U9
