File: tolt/stm32.kicad_sch (KiCad schematic)
At the start: 53 parts, among them J14 BOOT0, J15 NRST, U1 STM32F405RGTx, U10 MC74VHC1GT66, U11 MC74VHC1GT66, U12 MC74VHC1GT66, U13 MC74VHC1GT66, U5 INA240/241, U6 MC74VHC1GT66, U8 MC74VHC1GT66, Y1 8m

Commit message: modified:   tolt/stm32.kicad_sch 	modified:   tolt/tolt.kicad_pcb 	modified:   tolt/tolt.kicad_pro 	modified:   tolt/tolt.kicad_sch
Connections:
- net BRK: now reaches U1.50 (PA15)
Other:
- note added: "#define HW_USE_BRK #define BRK_GPIO GPIOB #define BRK_PIN 12"
Changed lines of the file:
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@@
+		)
+	)
+	(text "#define HW_USE_BRK\n\n#define BRK_GPIO				GPIOB\n#define BRK_PIN					12\n"
+		(exclude_from_sim no)
+		(at 121.92 104.394 0)
+		(effects
+			(font
+				(size 1.27 1.27)
+			)
+			(justify left)
 		)
 	)
@@
 		)
 	)
+	(hierarchical_label "BRK"
+		(shape bidirectional)
+		(at 109.474 103.124 0)
+		(effects
+			(font
+				(size 1.27 1.27)
+			)
+			(justify left)
+		)
+	)

Commit message: more files :3
Connections:
- net VCC: no longer C10.2, C27.2, C28.2, C31.2, C32.2, C33.2, C34.2, C37.2, C38.2, C39.2, C48.2, C49.2, C50.2, C9.2, U1.13 (VDDA), U10.5 (V+), U11.5 (V+), U12.5 (V+), U13.5 (V+), U5.6 (Vs), U5.7 (REF1), U6.5 (V+), U7.6 (Vs), U7.7 (REF1), U8.5 (V+), U9.6 (Vs), U9.7 (REF1)
- new net VDDA: C10.2, C27.2, C28.2, C31.2, C32.2, C33.2, C34.2, C37.2, C38.2, C39.2, C48.2, C49.2, C50.2, C9.2, U1.13 (VDDA), U10.5 (V+), U11.5 (V+), U12.5 (V+), U13.5 (V+), U5.6 (Vs), U5.7 (REF1), U6.5 (V+), U7.6 (Vs), U7.7 (REF1), U8.5 (V+), U9.6 (Vs), U9.7 (REF1)
Other:
- moved on the sheet: C10, C27, C28, C29, C31, C32, C33, C34, C36, C37, C39, C41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

Commit message: more assign+12-5v change
changed with TPS82130
Since using esp32 will increase consumption by a lot
Parts:
- R33, R34, R35: LCSC (none) -> C2907114
- U1: LCSC (none) -> C5290473
Changed lines of the file:
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@@
 			)
 		)
+		(property "LCSC" "C2907114"
+			(at 250.698 141.986 90)
+			(effects
+				(font
+					(size 1.27 1.27)
+				)
+				(hide yes)
+			)
+		)
 		(pin "1"
 		)
@@
 			)
 		)
+		(property "LCSC" "C5290473"
+			(at 91.694 108.204 0)
+			(effects
+				(font
+					(size 1.27 1.27)
+				)
+				(hide yes)
+			)
+		)
 		(pin "13"
 		)
@@
 			)
 		)
+		(property "LCSC" "C2907114"
+			(at 251.46 90.678 90)
+			(effects
+				(font
+					(size 1.27 1.27)
+				)
+				(hide yes)
+			)
+		)
 		(pin "1"
 		)
@@
 			(effects
 				(font
+					(size 1.27 1.27)
+				)
+				(hide yes)
+			)
+		)
+		(property "LCSC" "C2907114"
+			(at 248.92 40.386 90)
+			(effects
+				(font

Commit message: hm
weird huh it didnt fucking save
Parts:
- C1, C2, C27, C28, C3, C31, C32, C33, C34, C37, C38, C39, C4, C45, C46, C47, C48, C49, C50: LCSC (none) -> C60474
- C10, C13, C14, C5, C6, C7, C8, C9: LCSC (none) -> C913904
- C11, C12: LCSC (none) -> C1591
- C29, C36, C41: LCSC (none) -> C296713
- C30, C35, C40: LCSC (none) -> C1588

Commit message: Done
hopefully finished ?
needs sanity check and more checks
Parts:
- U10, U11, U12, U13, U6, U8: LCSC (none) -> C484737
- U7, U9: value ~ -> INA240/241
- Y1: LCSC (none) -> C7275084
Connections:
- net +3V3 is gone; now on net VCC: J14.1 (Pin_1)
Changed lines of the file:
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@@
 	(wire
 		(pts
-			(xy 41.656 59.69) (xy 35.306 59.69)
+			(xy 41.656 59.69) (xy 35.56 59.69)
 		)
 		(stroke
@@
 	)
 	(symbol
-		(lib_id "power:+3V3")
-		(at 35.306 59.69 0)
-		(unit 1)
-		(exclude_from_sim no)
-		(in_bom yes)
-		(on_board yes)
-		(dnp no)
-		(fields_autoplaced yes)
-		(property "Reference" "#PWR0101"
-			(at 35.306 63.5 0)
-			(effects
-				(font
-					(size 1.27 1.27)
-				)
-				(hide yes)
-			)
-		)
-		(property "Value" "+3V3"
-			(at 35.306 54.61 0)
-			(effects
-				(font
-					(size 1.27 1.27)
-				)
-			)
-		)
-		(property "Footprint" ""
-			(at 35.306 59.69 0)
-			(effects
-				(font
-					(size 1.27 1.27)
-				)
-				(hide yes)
-			)
-		)
-		(property "Datasheet" ""
-			(at 35.306 59.69 0)
-			(effects
-				(font
-					(size 1.27 1.27)
-				)
-				(hide yes)
-			)
-		)
-		(property "Description" "Power symbol creates a global label with name \"+3V3\""
-			(at 35.306 59.69 0)
-			(effects
-				(font
-					(size 1.27 1.27)
-				)
-				(hide yes)
-			)
-		)
-		(pin "1"
-		)
-		(instances
-			(project "tolt"
-				(path "/38c63d96-01d7-4159-b7c0-aa8cee77c3e9/410a2c08-a3a0-4066-ae14-a5c75baf28bb"
-					(reference "#PWR0101")
-					(unit 1)
-				)
-			)
-		)
-	)
-	(symbol
 		(lib_id "power:VDDA")
 		(at 240.03 95.25 0)
@@
 			)
 		)
+		(property "LCSC" "C7275084"
+			(at 32.766 76.454 90)
+			(effects
+				(font
+					(size 1.27 1.27)
+				)
+				(hide yes)
+			)
+		)
 		(pin "1"
 		)
@@
 			)
 		)
+		(property "LCSC" "C484737"
+			(at 232.41 93.98 90)
+			(effects
+				(font
+					(size 1.27 1.27)
+				)
+				(hide yes)
+			)
+		)
 		(pin "3"
 		)
@@
 			)
 		)
+		(property "LCSC" "C484737"
+			(at 232.41 146.05 90)
+			(effects
+				(font
+					(size 1.27 1.27)
+				)
+				(hide yes)
+			)
+		)
 		(pin "3"
 		)
@@
 			)
 		)
+		(property "LCSC" "C484737"
+			(at 182.88 45.72 90)
+			(effects
+				(font
+					(size 1.27 1.27)
+				)
+				(hide yes)
+			)
+		)
 		(pin "3"
 		)
@@
 			)
 		)
+		(property "LCSC" "C484737"
+			(at 181.61 142.24 90)
+			(effects
+				(font
+					(size 1.27 1.27)
+				)
+				(hide yes)
+			)
+		)
 		(pin "3"
 		)
@@
 	)
 	(symbol
+		(lib_id "power:VCC")
+		(at 35.56 59.69 0)
+		(unit 1)
+		(exclude_from_sim no)
+		(in_bom yes)
+		(on_board yes)
+		(dnp no)
+		(fields_autoplaced yes)
+		(property "Reference" "#PWR059"
+			(at 35.56 63.5 0)
+			(effects
+				(font
+					(size 1.27 1.27)
+				)
+				(hide yes)
+			)
+		)
+		(property "Value" "VCC"
+			(at 35.56 54.356 0)
+			(effects
+				(font
+					(size 1.27 1.27)
+				)
+			)
+		)
+		(property "Footprint" ""
+			(at 35.56 59.69 0)
+			(effects
+				(font
+					(size 1.27 1.27)
+				)
+				(hide yes)
+			)
+		)
+		(property "Datasheet" ""
+			(at 35.56 59.69 0)
+			(effects
+				(font
+					(size 1.27 1.27)
+				)
+				(hide yes)
+			)
+		)
+		(property "Description" "Power symbol creates a global label with name \"VCC\""
+			(at 35.56 59.69 0)
+			(effects
+				(font
+					(size 1.27 1.27)
+				)
+				(hide yes)
+			)
+		)
+		(pin "1"
+		)
+		(instances
+			(project "tolt"
+				(path "/38c63d96-01d7-4159-b7c0-aa8cee77c3e9/410a2c08-a3a0-4066-ae14-a5c75baf28bb"
+					(reference "#PWR059")
+					(unit 1)
+				)
+			)
+		)
+	)
+	(symbol
 		(lib_id "Device:C")
 		(at 181.61 129.286 180)
@@
 		(on_board yes)
 		(dnp no)
-		(fields_autoplaced yes)
 		(property "Reference" "U9"
 			(at 261.62 41.91 0)
@@
 			)
 		)
-		(property "Value" "~"
-			(at 261.62 49.53 0)
+		(property "Value" "INA240/241"
+			(at 261.62 43.434 0)
 			(effects
 				(font
@@
 			)
 		)
+		(property "LCSC" "C484737"
+			(at 229.87 43.18 90)
+			(effects
+				(font
+					(size 1.27 1.27)
+				)
+				(hide yes)
+			)
+		)
 		(pin "3"
 		)
@@
 		(on_board yes)
 		(dnp no)
-		(fields_autoplaced yes)
 		(property "Reference" "U7"
 			(at 264.16 92.202 0)
@@
 			)
 		)
-		(property "Value" "~"
-			(at 264.16 99.822 0)
+		(property "Value" "INA240/241"
+			(at 264.16 93.726 0)
 			(effects
 				(font
@@
 			(effects
 				(font
+					(size 1.27 1.27)
+				)
+				(hide yes)
+			)
+		)
+		(property "LCSC" "C484737"
+			(at 182.88 92.71 90)
+			(effects
+				(font

Commit message: fab
finally.
Parts:
- C10, C13, C14, C5, C6, C7, C8, C9: value 2.2u -> 2.2uf
- R33, R34, R35: LCSC C2907114 -> C22548
- U1: LCSC C5290473 -> C15742
Changed lines of the file:
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@@
 			)
 		)
-		(property "Value" "2.2u"
+		(property "Value" "2.2uf"
 			(at 48.26 138.684 0)
 			(effects
@@
 			)
 		)
-		(property "LCSC" "C2907114"
+		(property "LCSC" "C22548"
 			(at 250.698 141.986 90)
 			(effects
@@
 			)
 		)
-		(property "LCSC" "C5290473"
+		(property "LCSC" "C15742"
 			(at 91.694 108.204 0)
 			(effects
@@
 			)
 		)
-		(property "LCSC" "C2907114"
+		(property "LCSC" "C22548"
 			(at 251.46 90.678 90)
 			(effects
@@
 			)
 		)
-		(property "Value" "2.2u"
+		(property "Value" "2.2uf"
 			(at 54.61 167.64 0)
 			(effects
@@
 			)
 		)
-		(property "Value" "2.2u"
+		(property "Value" "2.2uf"
 			(at 63.5 138.684 0)
 			(effects
@@
 			)
 		)
-		(property "Value" "2.2u"
+		(property "Value" "2.2uf"
 			(at 109.982 35.052 0)
 			(effects
@@
 			)
 		)
-		(property "Value" "2.2u"
+		(property "Value" "2.2uf"
 			(at 121.158 35.052 0)
 			(effects
@@
 			)
 		)
-		(property "Value" "2.2u"
+		(property "Value" "2.2uf"
 			(at 39.624 167.64 0)
 			(effects
@@
 			)
 		)
-		(property "Value" "2.2u"
+		(property "Value" "2.2uf"
 			(at 98.552 35.052 0)
 			(effects
@@
 			)
 		)
-		(property "Value" "2.2u"
+		(property "Value" "2.2uf"
 			(at 132.588 35.052 0)
 			(effects
@@
 			)
 		)
-		(property "LCSC" "C2907114"
+		(property "LCSC" "C22548"
 			(at 248.92 40.386 90)
 			(effects
