File: tolt/converters.kicad_sch (KiCad schematic)
At the start: 17 parts, among them U14 AMS1117, U15 LP5907MFX-3.3

Commit message: .
Connections:
- net GND: now reaches C67.2, C68.2, C69.2, C70.2, D25.2 (A), U15.2 (GND)
- net GND: now also C61.2, C62.2, C63.2, C64.2, C65.2, C66.2, D23.1 (K), D24.2 (A), U14.1 (ADJ)
Other:
- moved on the sheet: C61, C62, C63, C64, C65, C66, D23, D24, L1, U14

Commit message: revert the mess
i am stupid
Parts:
- removed U14: AMS1117, Package_TO_SOT_SMD:SOT-223-3_TabPin2, symbol Regulator_Linear:AMS1117
- added C71: 10uF, Capacitor_SMD:C_0603_1608Metric, symbol Device:C
- added C72: 22uF, Capacitor_SMD:C_0805_2012Metric, symbol Device:C
- added C73: 10uF, Capacitor_SMD:C_0805_2012Metric, symbol Device:C
- added C74, C76: 100nF, symbol Device:C
- added C75, C77: 2.2uF, symbol Device:C
- added D28: 1N5227B, symbol Device:D_Zener
- added D29: 1N4733A, symbol Device:D_Zener
- added L3: 10uH, Inductor_SMD:L_Ferrocore_DLG-0403, symbol Device:L
- added L4: L, symbol Device:L
- added R4, R68, R69: 0, Resistor_SMD:R_0815_2038Metric, symbol Device:R
- added R64: 100k, Resistor_SMD:R_0603_1608Metric, symbol Device:R
- added U14: AMS1117-3.3, Package_TO_SOT_SMD:SOT-223-3_TabPin2, symbol Regulator_Linear:AMS1117-3.3
- added U16: TPS62173DSG, Package_SON:WSON-8-1EP_2x2mm_P0.5mm_EP0.9x1.6mm, symbol Regulator_Switching:TPS62173DSG
- added U19: LP5907MFX-3.3, Package_TO_SOT_SMD:SOT-23-5, symbol Regulator_Linear:LP5907MFX-3.3
- D24, D25: value D_Zener -> 1N5227B
Connections:
- net +12V: now also C71.2, U16.2 (VIN), U16.3 (EN)
- net +5V: now also C72.2, C73.2, D29.1 (K), L3.2, L4.1, R64.2, U16.6 (VOS)
- net GND: now also C71.1, C72.1, C73.1, D29.2 (A), R4.2, R68.1, R69.1, U14.1 (GND), U16.1 (PGND), U16.4 (AGND), U16.5 (FB), U16.9 (PAD); no longer C67.2, C68.2, C69.2, C70.2, D25.2 (A), U15.2 (GND)
- net VCC: now also U14.2 (VO)
- net at C61.1, C62.1, C63.1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: now also U14.3 (VI)
- new net: C74.1, C75.1, L4.2, U19.1 (IN), U19.3 (EN)
- new net: L3.1, U16.7 (SW)
- new net: R64.1, U16.8 (PG)
- new net GNDPWR: R4.1, R68.2, R69.2
- new net GNDRF: C74.2, C75.2, C76.2, C77.2, D28.2 (A), U19.2 (GND)
- new net VDDRF: C76.1, C77.1, D28.1 (K), U19.5 (OUT)
- new net VSSA: C67.2, C68.2, C69.2, C70.2, D25.2 (A), U15.2 (GND)
Other:
- note added: "12-5v"
- moved on the sheet: C61, C62, C63, C64, C65, C66, C67, C68, C69, C70, D23, D24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

Commit message: new file:   tolt/Library.pretty/IND-SMD_L3.9-W3.9-1.kicad_mod 	new file:   tolt/Library.pretty/IND-SMD_L5.0-W5.0.kicad_mod 	modified:   tolt/auxl.kicad_sch 	modified:   tolt/conn.kicad_sch 	modified:   tolt/converters.kicad_sch 	new file:   tolt/fp-lib-table 	modified:   tolt/inter.kicad_sch 	modified:   tolt/powerstage.kicad_sch 	modified:   tolt/stm32.kicad_sch 	modified:   tolt/tolt.kicad_sch
Parts:
- removed C74, C76: 100nF, symbol Device:C
- removed C75, C77: 2.2uF, symbol Device:C
- removed D23: LED, symbol Device:LED
- removed D28: 1N5227B, symbol Device:D_Zener
- removed L4: L, symbol Device:L
- removed U19: LP5907MFX-3.3, Package_TO_SOT_SMD:SOT-23-5, symbol Regulator_Linear:LP5907MFX-3.3
- C61: footprint (none) -> Capacitor_SMD:CP_Elec_4x5.4
- C62, C64, C66, C67, C69: footprint (none) -> Capacitor_SMD:C_0402_1005Metric_Pad0.74x0.62mm_HandSolder
- C63, C65, C68, C70: footprint (none) -> Capacitor_SMD:C_1210_3225Metric_Pad1.33x2.70mm_HandSolder
- C71: footprint Capacitor_SMD:C_0603_1608Metric -> Capacitor_SMD:C_1210_3225Metric_Pad1.33x2.70mm_HandSolder
- C72, C73: footprint Capacitor_SMD:C_0805_2012Metric -> Capacitor_SMD:C_1210_3225Metric_Pad1.33x2.70mm_HandSolder
- D24, D25: value 1N5227B -> BZT52C3V6-7-F; footprint (none) -> Diode_SMD:D_SOD-123
- D29: value 1N4733A -> BZT52C5V6-7-F; footprint (none) -> Diode_SMD:D_SOD-123
- L1, L2: value L -> 10uh; footprint (none) -> Library:IND-SMD_L3.9-W3.9-1
- L3: footprint Inductor_SMD:L_Ferrocore_DLG-0403 -> Library:IND-SMD_L5.0-W5.0
Other:
- moved on the sheet: C61, C62, C63, C64, C65, C66, C67, C68, C69, C70, D24, D25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

Commit message: modified:   tolt/converters.kicad_sch 	modified:   tolt/inter.kicad_sch 	modified:   tolt/tolt.kicad_sch
Parts:
- added C74: 10uF, Capacitor_SMD:C_1210_3225Metric_Pad1.33x2.70mm_HandSolder, symbol Device:C
- added C75, C76: 22uF, Capacitor_SMD:C_1210_3225Metric_Pad1.33x2.70mm_HandSolder, symbol Device:C
- added D23: D_Schottky, symbol Device:D_Schottky
- added JP4: Jumper_3_Bridged12, Jumper:SolderJumper-3_P1.3mm_Bridged2Bar12_RoundedPad1.0x1.5mm, symbol Jumper:Jumper_3_Bridged12
- added L4: L, symbol Device:L
- added R94: 68k, Resistor_SMD:R_0603_1608Metric_Pad0.98x0.95mm_HandSolder, symbol Device:R
- added R95: 820k, Resistor_SMD:R_0603_1608Metric_Pad0.98x0.95mm_HandSolder, symbol Device:R
- added U19: TLV61047DDC, Package_TO_SOT_SMD:SOT-23-5, symbol Regulator_Switching:TLV61047DDC
Connections:
- net +12V: now also JP4.2 (C)
- net GND: now also C74.1, C75.1, C76.1, R94.2, U19.2 (GND)
- new net: D23.2 (A), L4.2, U19.1 (SW)
- new net: R94.1, R95.2, U19.3 (FB)
- new net: C74.2, JP4.3 (B), L4.1, U19.4 (EN), U19.5 (VIN)
- new net +15V: C75.2, C76.2, D23.1 (K), JP4.1 (A), R95.1
Other:
- note added: "12-15v"
- note added: "use higheest accuracy resistors for FB operation !!!"
- moved on the sheet: R4, R68, R69

Commit message: new file:   tolt/Library.pretty/PQDE6W.kicad_mod 	modified:   tolt/auxl.kicad_sch 	modified:   tolt/conn.kicad_sch 	modified:   tolt/converters.kicad_sch 	modified:   tolt/powerstage.kicad_sch 	modified:   tolt/tolt.kicad_pcb 	modified:   tolt/tolt.kicad_sch
Parts:
- added C77: 22uF, Capacitor_SMD:C_1210_3225Metric_Pad1.33x2.70mm_HandSolder, symbol Device:C
- added C85: 10uF, Capacitor_SMD:C_1210_3225Metric_Pad1.33x2.70mm_HandSolder, symbol Device:C
- added C86: 100nF, Capacitor_SMD:C_0805_2012Metric, symbol Device:C
- added R96, R97: 4R7, Resistor_SMD:R_0805_2012Metric, symbol Device:R
- added U24: PQDE6W-Q110 / RD5-110S12W, Library:PQDE6W, symbol CCC_ESC_Custom_Symbols:PQDE6W-Q110
- D23: value D_Schottky -> CFSH05-20L; footprint (none) -> Diode_SMD:D_SOD-882
- L4: value L -> 10uh; footprint (none) -> Inductor_SMD:L_Abracon_ASPI-4030S
Connections:
- net +12V: now also C77.2, C85.2, U24.4 (VOUT)
- net GND: now also C77.1, C85.1, C86.2, U24.2 (GND_IN), U24.3 (GND_OUT)
- new net: C86.1, R96.1, R97.1, U24.1 (VIN)
- new net +BATT: R96.2, R97.2
Other:
- note added: "Footprint for CUI isolated module for up to 160V operation. Only allows 500mA. HiLink HLK-10D11012 CUI PQDE6W-Q110 Or anything that exceeds your battery voltage and gives 12V out"
- note added: "borrowed from MP2-ESC."
- moved on the sheet: C61, C62, C63, C64, C65, C66, C67, C68, C69, C70, C71, C72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

Commit message: modified:   tolt/conn.kicad_sch 	modified:   tolt/converters.kicad_sch 	modified:   tolt/inter.kicad_sch 	modified:   tolt/powerstage.kicad_sch 	modified:   tolt/stm32.kicad_sch 	modified:   tolt/tolt.kicad_pcb 	modified:   tolt/tolt.kicad_pro
Parts:
- C62, C64, C66, C67, C69: footprint Capacitor_SMD:C_0402_1005Metric_Pad0.74x0.62mm_HandSolder -> Capacitor_SMD:C_0402_1005Metric
- C63, C65, C68, C70, C71, C72, C73, C74, C75, C76, C77, C85: footprint Capacitor_SMD:C_1210_3225Metric_Pad1.33x2.70mm_HandSolder -> Capacitor_SMD:C_1210_3225Metric
- R94, R95: footprint Resistor_SMD:R_0603_1608Metric_Pad0.98x0.95mm_HandSolder -> Resistor_SMD:R_0603_1608Metric
Changed lines of the file:
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@@
 			)
 		)
-		(property "Footprint" "Capacitor_SMD:C_1210_3225Metric_Pad1.33x2.70mm_HandSolder"
+		(property "Footprint" "Capacitor_SMD:C_1210_3225Metric"
 			(at 63.7032 94.234 0)
 			(effects
@@
 			)
 		)
-		(property "Footprint" "Capacitor_SMD:C_0402_1005Metric_Pad0.74x0.62mm_HandSolder"
+		(property "Footprint" "Capacitor_SMD:C_0402_1005Metric"
 			(at 51.2572 94.234 0)
 			(effects
@@
 			)
 		)
-		(property "Footprint" "Capacitor_SMD:C_0402_1005Metric_Pad0.74x0.62mm_HandSolder"
+		(property "Footprint" "Capacitor_SMD:C_0402_1005Metric"
 			(at 90.8812 94.234 0)
 			(effects
@@
 			)
 		)
-		(property "Footprint" "Capacitor_SMD:C_0402_1005Metric_Pad0.74x0.62mm_HandSolder"
+		(property "Footprint" "Capacitor_SMD:C_0402_1005Metric"
 			(at 52.5272 135.382 0)
 			(effects
@@
 			)
 		)
-		(property "Footprint" "Resistor_SMD:R_0603_1608Metric_Pad0.98x0.95mm_HandSolder"
+		(property "Footprint" "Resistor_SMD:R_0603_1608Metric"
 			(at 221.996 46.482 90)
 			(effects
@@
 			)
 		)
-		(property "Footprint" "Capacitor_SMD:C_1210_3225Metric_Pad1.33x2.70mm_HandSolder"
+		(property "Footprint" "Capacitor_SMD:C_1210_3225Metric"
 			(at 103.6828 35.306 0)
 			(effects
@@
 			)
 		)
-		(property "Footprint" "Capacitor_SMD:C_0402_1005Metric_Pad0.74x0.62mm_HandSolder"
+		(property "Footprint" "Capacitor_SMD:C_0402_1005Metric"
 			(at 92.4052 135.382 0)
 			(effects
@@
 			)
 		)
-		(property "Footprint" "Capacitor_SMD:C_1210_3225Metric_Pad1.33x2.70mm_HandSolder"
+		(property "Footprint" "Capacitor_SMD:C_1210_3225Metric"
 			(at 247.1928 123.952 0)
 			(effects
@@
 			)
 		)
-		(property "Footprint" "Capacitor_SMD:C_1210_3225Metric_Pad1.33x2.70mm_HandSolder"
+		(property "Footprint" "Capacitor_SMD:C_1210_3225Metric"
 			(at 236.5248 123.952 0)
 			(effects
@@
 			)
 		)
-		(property "Footprint" "Capacitor_SMD:C_1210_3225Metric_Pad1.33x2.70mm_HandSolder"
+		(property "Footprint" "Capacitor_SMD:C_1210_3225Metric"
 			(at 183.4388 44.704 0)
 			(effects
@@
 			)
 		)
-		(property "Footprint" "Capacitor_SMD:C_1210_3225Metric_Pad1.33x2.70mm_HandSolder"
+		(property "Footprint" "Capacitor_SMD:C_1210_3225Metric"
 			(at 104.8512 135.382 0)
 			(effects
@@
 			)
 		)
-		(property "Footprint" "Capacitor_SMD:C_1210_3225Metric_Pad1.33x2.70mm_HandSolder"
+		(property "Footprint" "Capacitor_SMD:C_1210_3225Metric"
 			(at 39.1668 34.29 0)
 			(effects
@@
 			)
 		)
-		(property "Footprint" "Capacitor_SMD:C_1210_3225Metric_Pad1.33x2.70mm_HandSolder"
+		(property "Footprint" "Capacitor_SMD:C_1210_3225Metric"
 			(at 245.9228 40.132 0)
 			(effects
@@
 			)
 		)
-		(property "Footprint" "Capacitor_SMD:C_1210_3225Metric_Pad1.33x2.70mm_HandSolder"
+		(property "Footprint" "Capacitor_SMD:C_1210_3225Metric"
 			(at 256.8448 40.132 0)
 			(effects
@@
 			)
 		)
-		(property "Footprint" "Capacitor_SMD:C_1210_3225Metric_Pad1.33x2.70mm_HandSolder"
+		(property "Footprint" "Capacitor_SMD:C_1210_3225Metric"
 			(at 64.9732 135.382 0)
 			(effects
@@
 			)
 		)
-		(property "Footprint" "Resistor_SMD:R_0603_1608Metric_Pad0.98x0.95mm_HandSolder"
+		(property "Footprint" "Resistor_SMD:R_0603_1608Metric"
 			(at 221.996 54.102 90)
 			(effects
@@
 			)
 		)
-		(property "Footprint" "Capacitor_SMD:C_1210_3225Metric_Pad1.33x2.70mm_HandSolder"
+		(property "Footprint" "Capacitor_SMD:C_1210_3225Metric"
 			(at 103.3272 94.234 0)
 			(effects
@@
 			)
 		)
-		(property "Footprint" "Capacitor_SMD:C_0402_1005Metric_Pad0.74x0.62mm_HandSolder"
+		(property "Footprint" "Capacitor_SMD:C_0402_1005Metric"
 			(at 117.8052 135.382 0)
 			(effects
@@
 			)
 		)
-		(property "Footprint" "Capacitor_SMD:C_1210_3225Metric_Pad1.33x2.70mm_HandSolder"
+		(property "Footprint" "Capacitor_SMD:C_1210_3225Metric"
 			(at 93.0148 35.306 0)
 			(effects

Commit message: ltc
Parts:
- removed C86: 100nF, Capacitor_SMD:C_0805_2012Metric, symbol Device:C
- removed U24: PQDE6W-Q110 / RD5-110S12W, Library:PQDE6W, symbol CCC_ESC_Custom_Symbols:PQDE6W-Q110
- added C143: 1uF, symbol Device:C
- added C86: 33uF, symbol Device:C_Polarized
- added D30: D_Schottky, symbol Device:D_Schottky
- added L5: 150uH, symbol Device:L
- added R112: 267k, symbol Device:R
- added R113: 196k, symbol Device:R
- added U24: LTC7138xMSE, Package_SO:Analog_MSOP-12-16-1EP_3x4.039mm_P0.5mm_EP1.651x2.845mm, symbol Regulator_Switching:LTC7138xMSE
Connections:
- net +12V: now also L5.2, R112.1
- net GND: now also R113.2, U24.17 (GND), U24.6 (VPRG2), U24.8 (GND)
- net at R96.1, R97.1: now also C86.1
- new net: D30.1 (K), L5.1, U24.1 (SW)
- new net: U24.10 (SS), U24.7 (VPRG1)
- new net: D30.2 (A), U24.16 (ANODE)
- new net: R112.2, R113.1, U24.9 (VFB)
- no-connect marks 0 -> 2
Other:
- note removed: "Footprint for CUI isolated module for up to 160V operation. Only allows 500mA. HiLink HLK-10D11012 CUI PQDE6W-Q110 Or anything that exceeds your battery voltage and gives 12V out"
- note removed: "borrowed from MP2-ESC."
- moved on the sheet: C77, C85, R96, R97

Commit message: a
Parts:
- added D31: D_Schottky, symbol Device:D_Schottky
- added R114, R115, R116: R, symbol Device:R
- C143: footprint (none) -> Capacitor_SMD:C_2220_5750Metric
- C86: footprint (none) -> Capacitor_Tantalum_SMD:CP_EIA-3528-15_AVX-H
Connections:
- net GND: now also C143.2, C86.2, R116.2
- net at U24.12 (OVLO): now also R115.2, R116.1
- net at U24.14 (RUN): now also R114.2, R115.1
- net at U24.3 (VIN): now also C143.1, C86.1, D31.1 (K), R114.1
- net at R96.1, R97.1: now also D31.2 (A); no longer C86.1
Other:
- moved on the sheet: C143, C61, C62, C63, C64, C65, C66, C67, C68, C69, C70, C71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
