File: tolt/converters.kicad_sch (KiCad schematic)
At the start: 61 parts, among them J11 Conn_01x05, U14 AMS1117-3.3, U15 LP5907MFX-3.3, U16 TPS82130, U24 LTC7138xMSE, U25 LNK306D

Commit message: hm
weird huh it didnt fucking save
Parts:
- C102, C105: LCSC (none) -> C153032
- C147: LCSC (none) -> C60474
- C148, C77: LCSC (none) -> C52306
- C150: LCSC C24497 -> C60474
- C62, C64, C67, C69: LCSC (none) -> C24497
- C63, C65, C68, C70: LCSC (none) -> C913904
- D24, D25: LCSC (none) -> C726991
Changed lines of the file:
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@@
 			)
 		)
+		(property "LCSC" "C913904"
+			(at 63.754 100.076 0)
+			(effects
+				(font
+					(size 1.27 1.27)
+				)
+				(hide yes)
+			)
+		)
 		(pin "1"
 		)
@@
 			)
 		)
+		(property "LCSC" "C24497"
+			(at 51.308 100.076 0)
+			(effects
+				(font
+					(size 1.27 1.27)
+				)
+				(hide yes)
+			)
+		)
 		(pin "1"
 		)
@@
 			)
 		)
+		(property "LCSC" "C24497"
+			(at 90.932 100.076 0)
+			(effects
+				(font
+					(size 1.27 1.27)
+				)
+				(hide yes)
+			)
+		)
 		(pin "1"
 		)
@@
 			)
 		)
+		(property "LCSC" "C24497"
+			(at 157.48 100.33 0)
+			(effects
+				(font
+					(size 1.27 1.27)
+				)
+				(hide yes)
+			)
+		)
 		(pin "1"
 		)
@@
 			)
 		)
+		(property "LCSC" "C52306"
+			(at 160.274 164.846 0)
+			(effects
+				(font
+					(size 1.27 1.27)
+				)
+				(hide yes)
+			)
+		)
 		(pin "1"
 		)
@@
 			)
 		)
+		(property "LCSC" "C24497"
+			(at 197.358 100.33 0)
+			(effects
+				(font
+					(size 1.27 1.27)
+				)
+				(hide yes)
+			)
+		)
 		(pin "1"
 		)
@@
 			)
 		)
+		(property "LCSC" "C52306"
+			(at 138.176 164.846 0)
+			(effects
+				(font
+					(size 1.27 1.27)
+				)
+				(hide yes)
+			)
+		)
 		(pin "1"
 		)
@@
 			)
 		)
+		(property "LCSC" "C913904"
+			(at 209.804 100.33 0)
+			(effects
+				(font
+					(size 1.27 1.27)
+				)
+				(hide yes)
+			)
+		)
 		(pin "1"
 		)
@@
 			)
 		)
+		(property "LCSC" "C726991"
+			(at 234.442 100.33 90)
+			(effects
+				(font
+					(size 1.27 1.27)
+				)
+				(hide yes)
+			)
+		)
 		(pin "2"
 		)
@@
 			)
 		)
+		(property "LCSC" "C153032"
+			(at 19.05 173.99 0)
+			(effects
+				(font
+					(size 1.27 1.27)
+				)
+				(hide yes)
+			)
+		)
 		(pin "1"
 		)
@@
 			)
 		)
+		(property "LCSC" "C153032"
+			(at 30.48 173.99 0)
+			(effects
+				(font
+					(size 1.27 1.27)
+				)
+				(hide yes)
+			)
+		)
 		(pin "1"
 		)
@@
 			)
 		)
+		(property "LCSC" "C913904"
+			(at 169.926 100.33 0)
+			(effects
+				(font
+					(size 1.27 1.27)
+				)
+				(hide yes)
+			)
+		)
 		(pin "1"
 		)
@@
 			)
 		)
-		(property "LCSC" "C24497"
+		(property "LCSC" "C60474"
 			(at 264.922 50.546 0)
 			(effects
@@
 			)
 		)
+		(property "LCSC" "C60474"
+			(at 215.392 58.166 0)
+			(effects
+				(font
+					(size 1.27 1.27)
+				)
+				(hide yes)
+			)
+		)
 		(pin "1"
 		)
@@
 			)
 		)
+		(property "LCSC" "C726991"
+			(at 115.57 100.076 90)
+			(effects
+				(font
+					(size 1.27 1.27)
+				)
+				(hide yes)
+			)
+		)
 		(pin "2"
 		)
@@
 			(at 103.378 100.076 0)
 			(effects
+				(font
+					(size 1.27 1.27)
+				)
+				(hide yes)
+			)
+		)
+		(property "LCSC" "C913904"
+			(at 103.378 100.076 0)
+			(effects

Commit message: Done
hopefully finished ?
needs sanity check and more checks
Parts:
- added C76: 100n, Capacitor_SMD:C_0402_1005Metric, symbol Device:C
- added D23: MMSZ5242B, Diode_SMD:D_SOD-123, symbol Device:D_Zener
- added Q20: BSS131, Package_TO_SOT_SMD:SOT-23, symbol Transistor_FET:BSS138
- added R96: 470k, Resistor_SMD:R_1206_3216Metric, symbol Device:R
- added R97: 470r, Resistor_SMD:R_0603_1608Metric, symbol Device:R
- C143: LCSC (none) -> C153032
- C61: LCSC (none) -> C41416645
- D30, D31, D32: footprint Diode_SMD:D_2512_6332Metric -> Diode_SMD:D_SMA; LCSC (none) -> C64988
- L1, L2: LCSC (none) -> C6127589
- L5: value 150uH -> 220uH; footprint Library:IND-SMD_L5.0-W5.0 -> Library:IND-SMD_L8.0-W8.0_FNR80XXS; LCSC (none) -> C168148
- R112: value 267k -> 2.8M; LCSC (none) -> C705779
- R113: value 196k -> 200k; LCSC (none) -> C728585
- R114: value R -> 4.7M; footprint Resistor_SMD:R_0603_1608Metric -> Resistor_SMD:R_1206_3216Metric; LCSC (none) -> C137260
- R115: value R -> 1k; LCSC (none) -> C2907114
- R116: value R -> 100k; LCSC (none) -> C14675
- U14: LCSC (none) -> C6186
- U15: LCSC (none) -> C5370990
Connections:
- net GND: now also R116.1, U24.12 (OVLO), U24.7 (VPRG1), C76.1, D23.2 (A), Q20.2 (S); no longer R116.2
- net at U24.10 (SS): now also C76.2; no longer U24.7 (VPRG1)
- net at R114.2, R115.1: now also Q20.3 (D); no longer U24.14 (RUN)
- net at C143.1, C86.1, D31.1 (K)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: now also R96.2
- net Vreg_en: now reaches J11.4 (Pin_4)
- net Vreg_en: now also R97.1
- new net: R115.2, U24.14 (RUN)
- new net: D23.1 (K), Q20.1 (G), R116.2, R96.1, R97.2
- no-connect marks 3 -> 2
Other:
- note added: "Vout=0.8*(1+R1/R2) R2=200k Vout=12v solve for R1 12=0.8+0.8*R1/200k 11.2=0.8*R1/200K R1=11.2*200k/0.8 =2 800 000 ohm or 2.8Mohm"
- note added: "pull low vreg en"
- moved on the sheet: C143, C148, C149, C77, C85, C86, D30, D31, D32, L5, R112, R113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
