File: tolt/inter.kicad_sch (KiCad schematic)
At the start: 51 parts, among them U2 L6491, U3 L6491, U4 L6491

Commit message: move comp
Parts:
- R36, R51, R53: value 320k -> 650k
- R43, R45, R47: value 240k -> 305k
- R49: value 480k -> 610k
Other:
- note added: "500a ocp limit for 40s 650k 10k divider = 50mV from 3v3"
Changed lines of the file:
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@@
 		)
 	)
+	(text "500a ocp limit for 40s\n650k 10k divider = 50mV from 3v3\n"
+		(exclude_from_sim no)
+		(at 117.094 80.772 0)
+		(effects
+			(font
+				(size 1.27 1.27)
+			)
+		)
+	)
 	(text_box "Need to add lowpass filter and check how sd/od really works (seems to be pulled high normally)\nCheck the driver datasheet\n"
 		(exclude_from_sim no)
@@
 			)
 		)
-		(property "Value" "320k"
+		(property "Value" "650k"
 			(at 85.09 169.9259 0)
 			(effects
@@
 			)
 		)
-		(property "Value" "320k"
+		(property "Value" "650k"
 			(at 85.09 114.5539 0)
 			(effects
@@
 		(fields_autoplaced yes)
 		(property "Reference" "R47"
-			(at 251.968 30.9879 0)
+			(at 252.73 30.9879 0)
 			(effects
 				(font
@@
 			)
 		)
-		(property "Value" "240k"
-			(at 251.968 33.5279 0)
+		(property "Value" "305k"
+			(at 252.73 33.5279 0)
 			(effects
 				(font
@@
 			)
 		)
-		(property "Value" "320k"
+		(property "Value" "650k"
 			(at 83.82 62.9919 0)
 			(effects
@@
 		(fields_autoplaced yes)
 		(property "Reference" "R43"
-			(at 216.408 30.2259 0)
+			(at 217.17 30.2259 0)
 			(effects
 				(font
@@
 			)
 		)
-		(property "Value" "240k"
-			(at 216.408 32.7659 0)
+		(property "Value" "305k"
+			(at 217.17 32.7659 0)
 			(effects
 				(font
@@
 		(fields_autoplaced yes)
 		(property "Reference" "R49"
-			(at 269.494 31.7499 0)
+			(at 269.24 31.7499 0)
 			(effects
 				(font
@@
 			)
 		)
-		(property "Value" "480k"
-			(at 269.494 34.2899 0)
+		(property "Value" "610k"
+			(at 269.24 34.2899 0)
 			(effects
 				(font
@@
 		(fields_autoplaced yes)
 		(property "Reference" "R45"
-			(at 234.188 30.2259 0)
+			(at 234.95 30.2259 0)
 			(effects
 				(font
@@
 			)
 		)
-		(property "Value" "240k"
-			(at 234.188 32.7659 0)
+		(property "Value" "305k"
+			(at 234.95 32.7659 0)
 			(effects
 				(font

Commit message: FINAL
Parts:
- C15, C17, C19, C21, C22, C23: LCSC (none) -> C98192
- C16, C18, C20: LCSC (none) -> C64705
- C24, C25, C26: LCSC (none) -> C60474
- C42, C43, C44: footprint Capacitor_SMD:C_1210_3225Metric_Pad1.33x2.70mm_HandSolder -> Capacitor_SMD:C_1210_3225Metric; LCSC (none) -> C138687
- C51, C52, C53: LCSC (none) -> C1705
- C54, C55, C56, C57: LCSC (none) -> C14663
- D1, D2, D3: LCSC (none) -> C50432
- R36, R51, R53: value 650k -> 649k; LCSC (none) -> C2849080
- R37, R52, R54: LCSC (none) -> C25804
- R43, R45, R47: value 305k -> 309k; LCSC (none) -> C870641
- R44, R46, R48: LCSC (none) -> C105580
- R49: value 610k -> 619k; LCSC (none) -> C870826
- R50: LCSC (none) -> C22772
- U2, U3, U4: LCSC (none) -> C2970144

Commit message: aa
Connections:
- net GND: no longer C15.2, C17.2, C19.2
- net Ph_a: now also C15.2
- net Ph_b: now also C17.2
- net Ph_c: now also C19.2
Changed lines of the file:
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@@
 	(hierarchical_label "Ph_b"
 		(shape bidirectional)
+		(at 86.614 100.584 270)
+		(effects
+			(font
+				(size 1.27 1.27)
+			)
+			(justify right)
+		)
+	)
+	(hierarchical_label "Ph_b"
+		(shape bidirectional)
 		(at 232.41 27.686 90)
 		(effects
@@
 		)
 	)
+	(hierarchical_label "Ph_c"
+		(shape bidirectional)
+		(at 87.63 155.956 270)
+		(effects
+			(font
+				(size 1.27 1.27)
+			)
+			(justify right)
+		)
+	)
 	(hierarchical_label "H_B"
 		(shape input)
@@
 		)
 	)
+	(hierarchical_label "Ph_a"
+		(shape bidirectional)
+		(at 86.36 49.022 270)
+		(effects
+			(font
+				(size 1.27 1.27)
+			)
+			(justify right)
+		)
+	)
 	(hierarchical_label "SENS_C+"
 		(shape input)
@@
 	)
 	(symbol
-		(lib_id "power:GND")
-		(at 87.63 155.956 0)
-		(unit 1)
-		(exclude_from_sim no)
-		(in_bom yes)
-		(on_board yes)
-		(dnp no)
-		(fields_autoplaced yes)
-		(property "Reference" "#PWR046"
-			(at 87.63 162.306 0)
-			(effects
-				(font
-					(size 1.27 1.27)
-				)
-				(hide yes)
-			)
-		)
-		(property "Value" "GND"
-			(at 87.63 161.036 0)
-			(effects
-				(font
-					(size 1.27 1.27)
-				)
-			)
-		)
-		(property "Footprint" ""
-			(at 87.63 155.956 0)
-			(effects
-				(font
-					(size 1.27 1.27)
-				)
-				(hide yes)
-			)
-		)
-		(property "Datasheet" ""
-			(at 87.63 155.956 0)
-			(effects
-				(font
-					(size 1.27 1.27)
-				)
-				(hide yes)
-			)
-		)
-		(property "Description" ""
-			(at 87.63 155.956 0)
-			(effects
-				(font
-					(size 1.27 1.27)
-				)
-				(hide yes)
-			)
-		)
-		(pin "1"
-		)
-		(instances
-			(project "tolt"
-				(path "/38c63d96-01d7-4159-b7c0-aa8cee77c3e9/ca9cc269-3e36-4e00-8810-1c2cb270ed60"
-					(reference "#PWR046")
-					(unit 1)
-				)
-			)
-		)
-	)
-	(symbol
 		(lib_id "power:GNDPWR")
 		(at 82.042 73.152 0)
@@
 	)
 	(symbol
-		(lib_id "power:GND")
-		(at 86.614 100.584 0)
-		(unit 1)
-		(exclude_from_sim no)
-		(in_bom yes)
-		(on_board yes)
-		(dnp no)
-		(fields_autoplaced yes)
-		(property "Reference" "#PWR041"
-			(at 86.614 106.934 0)
-			(effects
-				(font
-					(size 1.27 1.27)
-				)
-				(hide yes)
-			)
-		)
-		(property "Value" "GND"
-			(at 86.614 105.664 0)
-			(effects
-				(font
-					(size 1.27 1.27)
-				)
-			)
-		)
-		(property "Footprint" ""
-			(at 86.614 100.584 0)
-			(effects
-				(font
-					(size 1.27 1.27)
-				)
-				(hide yes)
-			)
-		)
-		(property "Datasheet" ""
-			(at 86.614 100.584 0)
-			(effects
-				(font
-					(size 1.27 1.27)
-				)
-				(hide yes)
-			)
-		)
-		(property "Description" ""
-			(at 86.614 100.584 0)
-			(effects
-				(font
-					(size 1.27 1.27)
-				)
-				(hide yes)
-			)
-		)
-		(pin "1"
-		)
-		(instances
-			(project "tolt"
-				(path "/38c63d96-01d7-4159-b7c0-aa8cee77c3e9/ca9cc269-3e36-4e00-8810-1c2cb270ed60"
-					(reference "#PWR041")
-					(unit 1)
-				)
-			)
-		)
-	)
-	(symbol
 		(lib_id "Device:C")
 		(at 76.454 120.904 0)
@@
 					(unit 1)
 				)
-			)
-		)
-	)
-	(symbol
-		(lib_id "power:GND")
-		(at 86.36 49.022 0)
-		(unit 1)
-		(exclude_from_sim no)
-		(in_bom yes)
-		(on_board yes)
-		(dnp no)
-		(fields_autoplaced yes)
-		(property "Reference" "#PWR036"
-			(at 86.36 55.372 0)
-			(effects
-				(font
-					(size 1.27 1.27)
-				)
-				(hide yes)
-			)
-		)
-		(property "Value" "GND"
-			(at 86.36 54.102 0)
-			(effects
-				(font
-					(size 1.27 1.27)
-				)
-			)
-		)
-		(property "Footprint" ""
-			(at 86.36 49.022 0)
-			(effects
-				(font
-					(size 1.27 1.27)
-				)
-				(hide yes)
-			)
-		)
-		(property "Datasheet" ""
-			(at 86.36 49.022 0)
-			(effects
-				(font
-					(size 1.27 1.27)
-				)
-				(hide yes)
-			)
-		)
-		(property "Description" ""
-			(at 86.36 49.022 0)
-			(effects
-				(font
-					(size 1.27 1.27)
-				)
-				(hide yes)
-			)
-		)
-		(pin "1"
-		)
-		(instances
-			(project "tolt"
-				(path "/38c63d96-01d7-4159-b7c0-aa8cee77c3e9/ca9cc269-3e36-4e00-8810-1c2cb270ed60"
-					(reference "#PWR036")
-					(unit 1)
-				)
